File: Nova 1200 CPU Home-Brew - MartyG/Nova 1200 CPU Home-Brew - MartyG.kicad_sch (KiCad schematic)
At the start: 0 parts

Commit message: build
Parts:
- added U1: 9601, Package_DIP:DIP-14_W7.62mm, symbol ForgottenMachines:DM9601
- added U2: 7474, Package_DIP:DIP-14_W7.62mm, symbol ForgottenMachines:7474
Changed lines of the file:
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@@
 (kicad_sch (version 20230121) (generator eeschema)
   (paper "E")
+  (symbol (lib_id "ForgottenMachines:DM9601") (at 81.28 66.04 0) (unit 1)
+    (in_bom yes) (on_board yes) (dnp no) (fields_autoplaced)
+    (property "Reference" "U1" (at 84.7724 53.34 0)
+      (effects (font (size 1.27 1.27)))
+    )
+    (property "Value" "9601" (at 84.7724 55.88 0)
+      (effects (font (size 1.27 1.27)))
+    )
+    (property "Footprint" "Package_DIP:DIP-14_W7.62mm" (at 104.14 78.74 0)
+      (effects (font (size 1.27 1.27)) hide)
+    )
+    (property "Datasheet" "" (at 90.17 77.47 0)
+      (effects (font (size 1.27 1.27)) hide)
+    )
+    (pin "1")
+    (pin "2")
+    (pin "3")
+    (pin "4")
+    (pin "6")
+    (pin "8")
+    (pin "11")
+    (pin "13")
+    (pin "14")
+    (pin "7")
+    (instances
+      (project "Nova 1200 CPU Home-Brew - MartyG"
+        (path "/4e23fd18-5064-4456-9bf9-14f3233470c7"
+          (reference "U1") (unit 1)
+        )
+      )
+    )
+  )
+  (symbol (lib_id "ForgottenMachines:DM9601") (at -29.21 63.5 0) (unit 2)
+    (in_bom yes) (on_board yes) (dnp no) (fields_autoplaced)
+    (property "Reference" "U1" (at -8.89 60.325 0)
+      (effects (font (size 1.27 1.27)) (justify left))
+    )
+    (property "Value" "9601" (at -8.89 62.865 0)
+      (effects (font (size 1.27 1.27)) (justify left))
+    )
+    (property "Footprint" "Package_DIP:DIP-14_W7.62mm" (at -6.35 76.2 0)
+      (effects (font (size 1.27 1.27)) hide)
+    )
+    (property "Datasheet" "" (at -20.32 74.93 0)
+      (effects (font (size 1.27 1.27)) hide)
+    )
+    (pin "1")
+    (pin "2")
+    (pin "3")
+    (pin "4")
+    (pin "6")
+    (pin "8")
+    (pin "11")
+    (pin "13")
+    (pin "14")
+    (pin "7")
+    (instances
+      (project "Nova 1200 CPU Home-Brew - MartyG"
+        (path "/4e23fd18-5064-4456-9bf9-14f3233470c7"
+          (reference "U1") (unit 2)
+        )
+      )
+    )
+  )
+  (symbol (lib_id "ForgottenMachines:7474") (at -21.59 93.98 0) (unit 3)
+    (in_bom yes) (on_board yes) (dnp no) (fields_autoplaced)
+    (property "Reference" "U2" (at -13.97 93.345 0)
+      (effects (font (size 1.27 1.27)) (justify left))
+    )
+    (property "Value" "7474" (at -13.97 95.885 0)
+      (effects (font (size 1.27 1.27)) (justify left))
+    )
+    (property "Footprint" "Package_DIP:DIP-14_W7.62mm" (at -2.794 105.41 0)
+      (effects (font (size 1.27 1.27)) hide)
+    )
+    (property "Datasheet" "" (at -21.59 93.98 0)
+      (effects (font (size 1.27 1.27)) hide)
+    )
+    (pin "1")
+    (pin "2")
+    (pin "3")
+    (pin "4")
+    (pin "5")
+    (pin "6")
+    (pin "10")
+    (pin "11")
+    (pin "12")
+    (pin "13")
+    (pin "8")
+    (pin "9")
+    (pin "14")
+    (pin "7")
+    (instances
+      (project "Nova 1200 CPU Home-Brew - MartyG"
+        (path "/4e23fd18-5064-4456-9bf9-14f3233470c7"
+          (reference "U2") (unit 3)
+        )
+      )
+    )
+  )
+  (symbol (lib_id "ForgottenMachines:7474") (at 155.575 78.74 0) (unit 2)
+    (in_bom yes) (on_board yes) (dnp no) (fields_autoplaced)
+    (property "Reference" "U2" (at 158.1405 69.85 0)
+      (effects (font (size 1.27 1.27)) (justify left))
+    )
+    (property "Value" "7474" (at 158.1405 72.39 0)
+      (effects (font (size 1.27 1.27)) (justify left))
+    )
+    (property "Footprint" "Package_DIP:DIP-14_W7.62mm" (at 174.371 90.17 0)
+      (effects (font (size 1.27 1.27)) hide)
+    )
+    (property "Datasheet" "" (at 155.575 78.74 0)
+      (effects (font (size 1.27 1.27)) hide)
+    )
+    (pin "1")
+    (pin "2")
+    (pin "3")
+    (pin "4")
+    (pin "5")
+    (pin "6")
+    (pin "10")
+    (pin "11")
+    (pin "12")
+    (pin "13")
+    (pin "8")
+    (pin "9")
+    (pin "14")
+    (pin "7")
+    (instances
+      (project "Nova 1200 CPU Home-Brew - MartyG"
+        (path "/4e23fd18-5064-4456-9bf9-14f3233470c7"
+          (reference "U2") (unit 2)
+        )
+      )
+    )
+  )
+  (symbol (lib_id "ForgottenMachines:7474") (at 154.94 53.34 0) (unit 1)
+    (in_bom yes) (on_board yes) (dnp no) (fields_autoplaced)
+    (property "Reference" "U2" (at 157.5055 44.45 0)
+      (effects (font (size 1.27 1.27)) (justify left))
+    )
+    (property "Value" "7474" (at 157.5055 46.99 0)
+      (effects (font (size 1.27 1.27)) (justify left))
+    )
+    (property "Footprint" "Package_DIP:DIP-14_W7.62mm" (at 173.736 64.77 0)
+      (effects (font (size 1.27 1.27)) hide)
+    )
+    (property "Datasheet" "" (at 154.94 53.34 0)
+      (effects (font (size 1.27 1.27)) hide)
+    )
+    (pin "1")
+    (pin "2")
+    (pin "3")
+    (pin "4")
+    (pin "5")
+    (pin "6")
+    (pin "10")
+    (pin "11")
+    (pin "12")
+    (pin "13")
+    (pin "8")
+    (pin "9")
+    (pin "14")
+    (pin "7")
+    (instances
+      (project "Nova 1200 CPU Home-Brew - MartyG"
+        (path "/4e23fd18-5064-4456-9bf9-14f3233470c7"
+          (reference "U2") (unit 1)
+        )
+      )
+    )
+  )
   (sheet_instances
     (path "/" (page "1"))
