File: Backplane/Nova 1200 Backplane.kicad_sch (KiCad schematic)
At the start: 48 parts, among them J1 Conn_01x10, J10 Conn_01x10, J11 Conn_01x10, J12 Conn_01x10, J13 Conn_01x10, J14 Conn_01x10, J15 Conn_01x10, J16 Conn_01x10, J17 Conn_01x10, J18 Conn_01x10, J19 Conn_01x10, J1A Conn_01x40, J1A1 Conn_01x40, J1A2 Conn_01x40, J1A3 Conn_01x40, J1A4 Conn_01x40, J1A5 Conn_01x40, J1B Conn_01x40, J1B1 Conn_01x40, J1B2 Conn_01x40, J1B3 Conn_01x40, J1B4 Conn_01x40, J1B5 Conn_01x40, J2 Conn_01x10, J20 Conn_01x10, J21 Conn_01x10, J22 Conn_01x10, J23 Conn_01x10, J24 Conn_01x10, J2A Conn_01x40, J2A1 Conn_01x40, J2A2 Conn_01x40, J2A3 Conn_01x40, J2A4 Conn_01x40, J2A5 Conn_01x40, J2B Conn_01x40, J2B1 Conn_01x40, J2B2 Conn_01x40, J2B3 Conn_01x40, J2B4 Conn_01x40, J2B5 Conn_01x40, J3 Conn_01x10, J4 Conn_01x10, J5 Conn_01x10, J6 Conn_01x10, J7 Conn_01x10, J8 Conn_01x10, J9 Conn_01x10

Commit message: Deep Dives
Parts:
- removed J1, J2, J3, J4: Conn_01x10, symbol Connector_Generic:Conn_01x10
- removed J1A, J1B, J2A, J2B: Conn_01x40, symbol Connector_Generic:Conn_01x40
- added J1, J3: Conn_02x40_Odd_Even, Forgotten Machines:Card_Edge_Entrex_Trapezoid 80, symbol Connector_Generic:Conn_02x40_Odd_Even
- added J2, J4: DG Nova Card-Edge 81-100, Forgotten Machines:Data General Nova Card-Edge 81-100, symbol ForgottenMachines:DG_Nova_Card-Edge_81-100
Connections:
- net +5V: now also J1.3 (Pin_3), J1.4 (Pin_4), J2.97 (Pin_18), J2.98 (Pin_17), J3.3 (Pin_3), J3.4 (Pin_4), J4.97 (Pin_18), J4.98 (Pin_17)
- net +5V OK: now also J1.8 (Pin_8)
- net CLK FLOP: now also J3.48 (Pin_48)
- net CLR: now also J1.50 (Pin_50)
- net DATIA: now also J1.44 (Pin_44)
- net DATIB: now also J1.42 (Pin_42)
- net DATIC: now also J1.54 (Pin_54)
- net DATOA: now also J1.58 (Pin_58)
- net DATOB: now also J1.56 (Pin_56)
- net DATOC: now also J1.48 (Pin_48)
- net DCHI: now also J3.37 (Pin_37)
- net DCHO: now also J3.33 (Pin_33)
- net GND: now also J1.1 (Pin_1), J1.2 (Pin_2), J1.33 (Pin_33), J1.34 (Pin_34), J2.100 (Pin_19), J2.99 (Pin_20), J3.1 (Pin_1), J3.2 (Pin_2), J3.50 (Pin_50), J4.100 (Pin_19), J4.99 (Pin_20)
- net INHIBIT: now also J3.30 (Pin_30)
- net INTA: now also J1.40 (Pin_40)
- net IO PLS: now also J1.74 (Pin_74)
- net IO RST: now also J1.70 (Pin_70)
- net LOAD IR: now also J1.73 (Pin_73)
- net MB LOAD: now also J3.74 (Pin_74)
- net MEM OK: now also J1.9 (Pin_9)
- net OVFLO: now also J3.39 (Pin_39)
- net RESTART ENABLE: now also J1.32 (Pin_32)
- net STROBE: now also J3.20 (Pin_20)
- net STRT: now also J1.52 (Pin_52)
- net ~{CARRY}: now also J1.15 (Pin_15)
- net ~{CON DATA}: now also J1.28 (Pin_28)
- net ~{CON INST}: now also J1.22 (Pin_22)
- net ~{CON RQ}: now also J1.27 (Pin_27)
- net ~{CONT+ISTP+MSTP}: now also J1.25 (Pin_25)
- net ~{DATA0}: now also J3.62 (Pin_62)
- net ~{DATA10}: now also J3.75 (Pin_75)
- net ~{DATA11}: now also J3.58 (Pin_58)
- net ~{DATA12}: now also J3.59 (Pin_59)
- net ~{DATA13}: now also J3.64 (Pin_64)
- net ~{DATA14}: now also J3.56 (Pin_56)
- net ~{DATA15}: now also J3.66 (Pin_66)
- net ~{DATA1}: now also J3.65 (Pin_65)
- net ~{DATA2}: now also J4.82 (Pin_1)
- net ~{DATA3}: now also J3.73 (Pin_73)
- net ~{DATA4}: now also J3.61 (Pin_61)
- net ~{DATA5}: now also J3.57 (Pin_57)
- net ~{DATA6}: now also J4.95 (Pin_16)
- net ~{DATA7}: now also J3.55 (Pin_55)
- net ~{DATA8}: now also J3.60 (Pin_60)
- net ~{DATA9}: now also J3.63 (Pin_63)
- net ~{DCHA}: now also J1.60 (Pin_60)
- net ~{DCHM0}: now also J3.17 (Pin_17)
- net ~{DCHM1}: now also J3.21 (Pin_21)
- net ~{DCHR}: now also J3.35 (Pin_35)
- net ~{DEFER}: now also J1.12 (Pin_12)
- net ~{DIV}: now also J2.91 (Pin_12)
- net ~{DRIVE IO}: now also J4.88 (Pin_7)
- net ~{DS0}: now also J1.72 (Pin_72)
- net ~{DS1}: now also J1.68 (Pin_68)
- net ~{DS2}: now also J1.66 (Pin_66)
- net ~{DS3}: now also J1.46 (Pin_46)
- net ~{DS4}: now also J1.62 (Pin_62)
- net ~{DS5}: now also J1.64 (Pin_64)
- net ~{EXEC}: now also J1.11 (Pin_11)
- net ~{EXT LOAD}: now also J1.47 (Pin_47), J3.49 (Pin_49)
- net ~{FETCH}: now also J1.13 (Pin_13), J1.49 (Pin_49)
- net ~{FORCE LOAD IR}: now also J2.85 (Pin_6)
- net ~{INH TRANS}: now also J3.45 (Pin_45)
- net ~{INTR}: now also J3.29 (Pin_29)
- net ~{ION}: now also J1.16 (Pin_16)
- net ~{ISTP}: now also J1.17 (Pin_17)
- net ~{LOAD AC}: now also J1.77 (Pin_77)
- net ~{MA LOAD}: now also J3.7 (Pin_7)
- net ~{MB CLEAR}: now also J4.86 (Pin_5)
- net ~{MBO0}: now also J3.79 (Pin_79)
- net ~{MBO10}: now also J3.8 (Pin_8)
- net ~{MBO11}: now also J3.5 (Pin_5)
- net ~{MBO12}: now also J1.39 (Pin_39)
- net ~{MBO13}: now also J1.37 (Pin_37)
- net ~{MBO14}: now also J1.43 (Pin_43)
- net ~{MBO15}: now also J1.41 (Pin_41)
- net ~{MBO1}: now also J3.77 (Pin_77)
- net ~{MBO2}: now also J3.44 (Pin_44)
- net ~{MBO3}: now also J3.43 (Pin_43)
- net ~{MBO4}: now also J3.42 (Pin_42)
- net ~{MBO5}: now also J3.32 (Pin_32)
- net ~{MBO6}: now also J3.16 (Pin_16)
- net ~{MBO7}: now also J3.14 (Pin_14)
- net ~{MBO8}: now also J3.12 (Pin_12)
- net ~{MBO9}: now also J3.9 (Pin_9)
- net ~{MD SEL1}: now also J2.87 (Pin_8)
- net ~{MEM0}: now also J3.71 (Pin_71)
- net ~{MEM10}: now also J1.45 (Pin_45)
- net ~{MEM11}: now also J1.51 (Pin_51)
- net ~{MEM12}: now also J1.36 (Pin_36)
- net ~{MEM13}: now also J1.35 (Pin_35)
- net ~{MEM14}: now also J3.76 (Pin_76)
- net ~{MEM15}: now also J3.18 (Pin_18)
- net ~{MEM1}: now also J3.70 (Pin_70)
- net ~{MEM2}: now also J3.47 (Pin_47)
- net ~{MEM3}: now also J3.68 (Pin_68)
- net ~{MEM4}: now also J3.28 (Pin_28)
- net ~{MEM5}: now also J3.26 (Pin_26)
- net ~{MEM6}: now also J3.22 (Pin_22)
- net ~{MEM7}: now also J3.24 (Pin_24)
- net ~{MEM8}: now also J1.55 (Pin_55)
- net ~{MEM9}: now also J1.53 (Pin_53)
- net ~{MSKO}: now also J1.38 (Pin_38)
- net ~{MSTP}: now also J1.20 (Pin_20)
- net ~{PL}: now also J1.19 (Pin_19)
- net ~{POWER FAIL}: now also J1.5 (Pin_5)
- net ~{READ IO}: now also J4.83 (Pin_4)
- net ~{READ1}: now also J4.87 (Pin_8)
- net ~{READ2}: now also J4.90 (Pin_9)
- net ~{RQENB}: now also J3.41 (Pin_41)
- net ~{RST}: now also J1.30 (Pin_30)
- net ~{RUN}: now also J1.14 (Pin_14)
- net ~{SELB}: now also J2.82 (Pin_1)
- net ~{SELD}: now also J1.80 (Pin_80)
- net ~{SHIFT0}: now also J4.94 (Pin_13)
- net ~{SHIFT1}: now also J4.96 (Pin_15)
- net ~{SHIFT2}: now also J4.93 (Pin_14)
- net ~{SHIFT3}: now also J4.91 (Pin_12)
- net ~{SKIP}: now also J3.69 (Pin_69)
- net ~{STOP}: now also J1.31 (Pin_31)
- net ~{TEST}: now also J2.92 (Pin_11)
- net ~{WAS JSR}: now also J2.89 (Pin_10)
- net ~{WHOA}: now also J3.6 (Pin_6)
- no-connect marks 0 -> 471
Other:
- moved on the sheet: J1A2, J1A3, J1B2, J1B3, J2A2, J2A3, J2B2, J2B3

Commit message: Build
Parts:
- added C1, C2: CAP_Disc_Common_-_Entrex_Trapezoid, Forgotten Machines:Disc Capacitor Common Entrex Trapezoid, symbol ForgottenMachines:CAP_Disc_Common_-_Entrex_Trapezoid
Connections:
- net GND: now also C1.1, C2.1
- net ~{CON RQ}: now also C2.2
- net ~{PL}: now also C1.2
- net Entrex P10.19: now reaches J1.24 (Pin_24)
- net Entrex P10.30: now reaches J1.29 (Pin_29)
- no-connect marks 471 -> 469
Other:
- note added: "Entrex P10.11 - GND Entrex P10.37 - Slot 2 #A8"
Changed lines of the file:
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@@
   (no_connect (at 228.6 99.06))
   (no_connect (at 91.44 149.86))
-  (no_connect (at 111.76 302.26))
   (no_connect (at 302.26 86.36))
   (no_connect (at 138.43 35.56))
@@
   (no_connect (at 250.19 187.96))
   (no_connect (at 179.07 99.06))
-  (no_connect (at 119.38 289.56))
   (no_connect (at 280.67 187.96))
   (no_connect (at 223.52 99.06))
@@
     (effects (font (size 1.27 1.27)) (justify right bottom))
   )
+  (text "Entrex P10.11 - GND\nEntrex P10.37 - Slot 2 #A8" (at 90.17 353.06 0)
+    (effects (font (size 1.27 1.27)) (justify left bottom))
+  )
   (text "nova 1200 slot 1 CPU" (at 43.18 294.64 0)
     (effects (font (size 2 2) (thickness 0.4) bold) (justify left bottom))
@@
     )
   )
+  (global_label "Entrex P10.18" (shape input) (at 116.84 279.4 90) (fields_autoplaced)
+    (effects (font (size 1.27 1.27)) (justify left))
+    (property "Intersheetrefs" "${INTERSHEET_REFS}" (at 116.84 263.0928 90)
+      (effects (font (size 1.27 1.27)) (justify left) hide)
+    )
+  )
   (global_label "~{MEM2}" (shape input) (at 274.32 238.76 90) (fields_autoplaced)
     (effects (font (size 1.27 1.27)) (justify left))
@@
     )
   )
+  (global_label "Entrex P10.31" (shape input) (at 88.9 276.86 90) (fields_autoplaced)
+    (effects (font (size 1.27 1.27)) (justify left))
+    (property "Intersheetrefs" "${INTERSHEET_REFS}" (at 88.9 260.5528 90)
+      (effects (font (size 1.27 1.27)) (justify left) hide)
+    )
+  )
   (global_label "~{DS2}" (shape input) (at 165.1 200.66 270) (fields_autoplaced)
     (effects (font (size 1.27 1.27)) (justify right))
@@
     )
   )
+  (global_label "~{PL}" (shape input) (at 62.23 300.99 0) (fields_autoplaced)
+    (effects (font (size 1.27 1.27)) (justify left))
+    (property "Intersheetrefs" "${INTERSHEET_REFS}" (at 67.4339 300.99 0)
+      (effects (font (size 1.27 1.27)) (justify left) hide)
+    )
+  )
   (global_label "-5V" (shape input) (at 87.63 48.26 270) (fields_autoplaced)
     (effects (font (size 1.27 1.27)) (justify right))
@@
     )
   )
+  (global_label "Entrex P10.10" (shape input) (at 119.38 308.61 270) (fields_autoplaced)
+    (effects (font (size 1.27 1.27)) (justify right))
+    (property "Intersheetrefs" "${INTERSHEET_REFS}" (at 119.38 324.9172 90)
+      (effects (font (size 1.27 1.27)) (justify right) hide)
+    )
+  )
   (global_label "DATA RDR" (shape input) (at 259.08 99.06 270) (fields_autoplaced)
     (effects (font (size 1.27 1.27)) (justify right))
@@
     )
   )
+  (global_label "Entrex P10.33" (shape input) (at 99.06 308.61 270) (fields_autoplaced)
+    (effects (font (size 1.27 1.27)) (justify right))
+    (property "Intersheetrefs" "${INTERSHEET_REFS}" (at 99.06 324.9172 90)
+      (effects (font (size 1.27 1.27)) (justify right) hide)
+    )
+  )
   (global_label "GND" (shape input) (at 83.82 289.56 90) (fields_autoplaced)
     (effects (font (size 1.27 1.27)) (justify left))
@@
     )
   )
+  (global_label "Entrex P10.3" (shape input) (at 116.84 313.69 270) (fields_autoplaced)
+    (effects (font (size 1.27 1.27)) (justify right))
+    (property "Intersheetrefs" "${INTERSHEET_REFS}" (at 116.84 328.7877 90)
+      (effects (font (size 1.27 1.27)) (justify right) hide)
+    )
+  )
   (global_label "GND" (shape input) (at 340.36 48.26 270) (fields_autoplaced)
     (effects (font (size 1.27 1.27)) (justify right))
@@
     )
   )
+  (global_label "GND" (shape input) (at 49.53 312.42 180) (fields_autoplaced)
+    (effects (font (size 1.27 1.27)) (justify right))
+    (property "Intersheetrefs" "${INTERSHEET_REFS}" (at 42.7537 312.42 0)
+      (effects (font (size 1.27 1.27)) (justify right) hide)
+    )
+  )
   (global_label "~{MEM4}" (shape input) (at 248.92 251.46 270) (fields_autoplaced)
     (effects (font (size 1.27 1.27)) (justify right))
@@
     )
   )
+  (global_label "Entrex P10.35" (shape input) (at 96.52 311.15 270) (fields_autoplaced)
+    (effects (font (size 1.27 1.27)) (justify right))
+    (property "Intersheetrefs" "${INTERSHEET_REFS}" (at 96.52 327.4572 90)
+      (effects (font (size 1.27 1.27)) (justify right) hide)
+    )
+  )
   (global_label "WB6" (shape input) (at 256.54 48.26 270) (fields_autoplaced)
     (effects (font (size 1.27 1.27)) (justify right))
@@
     )
   )
+  (global_label "~{CON RQ}" (shape input) (at 62.23 312.42 0) (fields_autoplaced)
+    (effects (font (size 1.27 1.27)) (justify left))
+    (property "Intersheetrefs" "${INTERSHEET_REFS}" (at 72.4293 312.42 0)
+      (effects (font (size 1.27 1.27)) (justify left) hide)
+    )
+  )
   (global_label "~{DATA9}" (shape input) (at 294.64 289.56 90) (fields_autoplaced)
     (effects (font (size 1.27 1.27)) (justify left))
@@
     )
   )
+  (global_label "Entrex P10.19" (shape input) (at 111.76 302.26 270) (fields_autoplaced)
+    (effects (font (size 1.27 1.27)) (justify right))
+    (property "Intersheetrefs" "${INTERSHEET_REFS}" (at 111.76 318.5672 90)
+      (effects (font (size 1.27 1.27)) (justify right) hide)
+    )
+  )
   (global_label "+5V OK" (shape input) (at 91.44 302.26 270) (fields_autoplaced)
     (effects (font (size 1.27 1.27)) (justify right))
@@
     )
   )
+  (global_label "Entrex P10.46" (shape input) (at 109.22 313.69 270) (fields_autoplaced)
+    (effects (font (size 1.27 1.27)) (justify right))
+    (property "Intersheetrefs" "${INTERSHEET_REFS}" (at 109.22 329.9972 90)
+      (effects (font (size 1.27 1.27)) (justify right) hide)
+    )
+  )
   (global_label "~{MBO3}" (shape input) (at 269.24 289.56 90) (fields_autoplaced)
     (effects (font (size 1.27 1.27)) (justify left))
@@
     )
   )
+  (global_label "GND" (shape input) (at 49.53 300.99 180) (fields_autoplaced)
+    (effects (font (size 1.27 1.27)) (justify right))
+    (property "Intersheetrefs" "${INTERSHEET_REFS}" (at 42.7537 300.99 0)
+      (effects (font (size 1.27 1.27)) (justify right) hide)
+    )
+  )
   (global_label "OVFLO" (shape input) (at 264.16 86.36 90) (fields_autoplaced)
     (effects (font (size 1.27 1.27)) (justify left))
@@
     )
   )
+  (global_label "Entrex P10.30" (shape input) (at 119.38 289.56 90) (fields_autoplaced)
+    (effects (font (size 1.27 1.27)) (justify left))
+    (property "Intersheetrefs" "${INTERSHEET_REFS}" (at 119.38 273.2528 90)
+      (effects (font (size 1.27 1.27)) (justify left) hide)
+    )
+  )
   (global_label "RWND T" (shape input) (at 302.26 35.56 90) (fields_autoplaced)
     (effects (font (size 1.27 1.27)) (justify left))
@@
     )
   )
+  (symbol (lib_id "ForgottenMachines:CAP_Disc_Common_-_Entrex_Trapezoid") (at 55.88 300.99 90) (unit 1)
+    (in_bom yes) (on_board yes) (dnp no)
+    (property "Reference" "C1" (at 55.88 303.53 90)
+      (effects (font (size 1.27 1.27)))
+    )
+    (property "Value" "CAP_Disc_Common_-_Entrex_Trapezoid" (at 53.34 297.18 0)
+      (effects (font (size 1.27 1.27)) (justify left) hide)
+    )
+    (property "Footprint" "Forgotten Machines:Disc Capacitor Common Entrex Trapezoid" (at 66.04 336.55 0)
+      (effects (font (size 1.27 1.27)) hide)
+    )
+    (property "Datasheet" "~" (at 55.88 300.99 0)
+      (effects (font (size 1.27 1.27)) hide)
+    )
+    (pin "1")
+    (pin "2")
+    (instances
+      (project "Nova 1200 Backplane"
+        (path "/c1f710ce-b3f9-4828-9325-9c2326e8d74c"
+          (reference "C1") (unit 1)
+        )
+      )
+    )
+  )
   (symbol (lib_id "Connector_Generic:Conn_01x10") (at 328.93 195.58 90) (unit 1)
     (in_bom yes) (on_board yes) (dnp no) (fields_autoplaced)
@@
         )
       )
+    )
+  )
+  (symbol (lib_id "ForgottenMachines:CAP_Disc_Common_-_Entrex_Trapezoid") (at 55.88 312.42 90) (unit 1)
+    (in_bom yes) (on_board yes) (dnp no)
+    (property "Reference" "C2" (at 55.88 314.96 90)
+      (effects (font (size 1.27 1.27)))
+    )
+    (property "Value" "CAP_Disc_Common_-_Entrex_Trapezoid" (at 53.34 308.61 0)
+      (effects (font (size 1.27 1.27)) (justify left) hide)
+    )
+    (property "Footprint" "Forgotten Machines:Disc Capacitor Common Entrex Trapezoid" (at 66.04 347.98 0)
+      (effects (font (size 1.27 1.27)) hide)
+    )
+    (property "Datasheet" "~" (at 55.88 312.42 0)
+      (effects (font (size 1.27 1.27)) hide)
+    )
+    (pin "1")
+    (pin "2")
+    (instances
+      (project "Nova 1200 Backplane"
+        (path "/c1f710ce-b3f9-4828-9325-9c2326e8d74c"
+          (reference "C2") (unit 1)
+        )
+      )
