File: Backplane/Nova 1200 Backplane.kicad_sch (KiCad schematic)
At the start: 46 parts, among them J1 Conn_02x40_Odd_Even, J10 Conn_01x10, J11 Conn_01x10, J12 Conn_01x10, J13 Conn_01x10, J14 Conn_01x10, J15 Conn_01x10, J16 Conn_01x10, J17 Conn_01x10, J18 Conn_01x10, J19 Conn_01x10, J1A1 Conn_01x40, J1A2 Conn_01x40, J1A3 Conn_01x40, J1A4 Conn_01x40, J1A5 Conn_01x40, J1B1 Conn_01x40, J1B2 Conn_01x40, J1B3 Conn_01x40, J1B4 Conn_01x40, J1B5 Conn_01x40, J2 DG Nova Card-Edge 81-100, J20 Conn_01x10, J21 Conn_01x10, J22 Conn_01x10, J23 Conn_01x10, J24 Conn_01x10, J2A1 Conn_01x40, J2A2 Conn_01x40, J2A3 Conn_01x40, J2A4 Conn_01x40, J2A5 Conn_01x40, J2B1 Conn_01x40, J2B2 Conn_01x40, J2B3 Conn_01x40, J2B4 Conn_01x40, J2B5 Conn_01x40, J3 Conn_02x40_Odd_Even, J4 DG Nova Card-Edge 81-100, J5 Conn_01x10, J6 Conn_01x10, J7 Conn_01x10, J8 Conn_01x10, J9 Conn_01x10

Commit message: yo
Connections:
- net Entrex Jmp Slot 13 is gone; now on net Entrex Backplane S01B53 to S13B53: J3.53 (Pin_53)
- net Entrex Backplane S01B53 to S13B53: now reaches J2A4.53 (Pin_27)
- no-connect marks 468 -> 467
Changed lines of the file:
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@@
   (no_connect (at 327.66 289.56))
   (no_connect (at 246.38 99.06))
-  (no_connect (at 281.94 137.16))
   (no_connect (at 95.25 35.56))
   (no_connect (at 116.84 137.16))
@@
   )
   (global_label "Entrex P10.18" (shape input) (at 116.84 279.4 90) (fields_autoplaced)
-    (effects (font (size 1.27 1.27)) (justify left))
-    (property "Intersheetrefs" "${INTERSHEET_REFS}" (at 116.84 263.0928 90)
+    (effects (font (size 1 1)) (justify left))
+    (property "Intersheetrefs" "${INTERSHEET_REFS}" (at 116.84 266.5597 90)
       (effects (font (size 1.27 1.27)) (justify left) hide)
     )
@@
     )
   )
+  (global_label "Entrex Backplane S01B53 to S13B53" (shape input) (at 281.94 289.56 90) (fields_autoplaced)
+    (effects (font (size 0.7 0.7)) (justify left))
+    (property "Intersheetrefs" "${INTERSHEET_REFS}" (at 281.94 268.545 90)
+      (effects (font (size 1.27 1.27)) (justify left) hide)
+    )
+  )
   (global_label "~{DS3}" (shape input) (at 139.7 302.26 270) (fields_autoplaced)
     (effects (font (size 1.27 1.27)) (justify right))
@@
   )
   (global_label "Entrex P10.31" (shape input) (at 88.9 276.86 90) (fields_autoplaced)
-    (effects (font (size 1.27 1.27)) (justify left))
-    (property "Intersheetrefs" "${INTERSHEET_REFS}" (at 88.9 260.5528 90)
+    (effects (font (size 1 1)) (justify left))
+    (property "Intersheetrefs" "${INTERSHEET_REFS}" (at 88.9 264.0197 90)
       (effects (font (size 1.27 1.27)) (justify left) hide)
     )
@@
     )
   )
+  (global_label "~{M CON DATA}" (shape input) (at 116.84 325.12 270) (fields_autoplaced)
+    (effects (font (size 1 1)) (justify right))
+    (property "Intersheetrefs" "${INTERSHEET_REFS}" (at 116.84 336.3221 90)
+      (effects (font (size 1.27 1.27)) (justify right) hide)
+    )
+  )
   (global_label "~{DCHA}" (shape input) (at 157.48 200.66 270) (fields_autoplaced)
     (effects (font (size 1.27 1.27)) (justify right))
@@
   )
   (global_label "Entrex P10.10" (shape input) (at 119.38 308.61 270) (fields_autoplaced)
-    (effects (font (size 1.27 1.27)) (justify right))
-    (property "Intersheetrefs" "${INTERSHEET_REFS}" (at 119.38 324.9172 90)
+    (effects (font (size 1 1)) (justify right))
+    (property "Intersheetrefs" "${INTERSHEET_REFS}" (at 119.38 321.4503 90)
       (effects (font (size 1.27 1.27)) (justify right) hide)
     )
@@
   )
   (global_label "Entrex P10.33" (shape input) (at 99.06 308.61 270) (fields_autoplaced)
-    (effects (font (size 1.27 1.27)) (justify right))
-    (property "Intersheetrefs" "${INTERSHEET_REFS}" (at 99.06 324.9172 90)
+    (effects (font (size 1 1)) (justify right))
+    (property "Intersheetrefs" "${INTERSHEET_REFS}" (at 99.06 321.4503 90)
       (effects (font (size 1.27 1.27)) (justify right) hide)
     )
@@
     )
   )
+  (global_label "~{M CON INST}" (shape input) (at 109.22 326.39 270) (fields_autoplaced)
+    (effects (font (size 1 1)) (justify right))
+    (property "Intersheetrefs" "${INTERSHEET_REFS}" (at 109.22 337.3541 90)
+      (effects (font (size 1.27 1.27)) (justify right) hide)
+    )
+  )
   (global_label "~{DATA8}" (shape input) (at 289.56 48.26 270) (fields_autoplaced)
     (effects (font (size 1.27 1.27)) (justify right))
@@
   )
   (global_label "Entrex P10.3" (shape input) (at 116.84 313.69 270) (fields_autoplaced)
-    (effects (font (size 1.27 1.27)) (justify right))
-    (property "Intersheetrefs" "${INTERSHEET_REFS}" (at 116.84 328.7877 90)
+    (effects (font (size 1 1)) (justify right))
+    (property "Intersheetrefs" "${INTERSHEET_REFS}" (at 116.84 325.5779 90)
       (effects (font (size 1.27 1.27)) (justify right) hide)
     )
@@
     )
   )
-  (global_label "Entrex P10.35" (shape input) (at 96.52 311.15 270) (fields_autoplaced)
-    (effects (font (size 1.27 1.27)) (justify right))
-    (property "Intersheetrefs" "${INTERSHEET_REFS}" (at 96.52 327.4572 90)
+  (global_label "Entrex P10.35" (shape input) (at 96.52 310.515 270) (fields_autoplaced)
+    (effects (font (size 1 1)) (justify right))
+    (property "Intersheetrefs" "${INTERSHEET_REFS}" (at 96.52 323.3553 90)
       (effects (font (size 1.27 1.27)) (justify right) hide)
     )
@@
     )
   )
+  (global_label "~{CON INST}" (shape input) (at 111.76 314.96 270) (fields_autoplaced)
+    (effects (font (size 1 1)) (justify right))
+    (property "Intersheetrefs" "${INTERSHEET_REFS}" (at 111.76 324.1812 90)
+      (effects (font (size 1.27 1.27)) (justify right) hide)
+    )
+  )
   (global_label "~{DATA7}" (shape input) (at 284.48 86.36 90) (fields_autoplaced)
     (effects (font (size 1.27 1.27)) (justify left))
@@
     )
   )
+  (global_label "Entrex Backplane S01B53 to S13B53" (shape input) (at 281.94 137.16 90) (fields_autoplaced)
+    (effects (font (size 0.7 0.7)) (justify left))
+    (property "Intersheetrefs" "${INTERSHEET_REFS}" (at 281.94 116.145 90)
+      (effects (font (size 1.27 1.27)) (justify left) hide)
+    )
+  )
   (global_label "INH GND" (shape input) (at 101.6 251.46 270) (fields_autoplaced)
     (effects (font (size 1.27 1.27)) (justify right))
@@
   )
   (global_label "Entrex P10.19" (shape input) (at 111.76 302.26 270) (fields_autoplaced)
-    (effects (font (size 1.27 1.27)) (justify right))
-    (property "Intersheetrefs" "${INTERSHEET_REFS}" (at 111.76 318.5672 90)
+    (effects (font (size 1 1)) (justify right))
+    (property "Intersheetrefs" "${INTERSHEET_REFS}" (at 111.76 315.1003 90)
       (effects (font (size 1.27 1.27)) (justify right) hide)
     )
@@
   )
   (global_label "Entrex P10.46" (shape input) (at 109.22 313.69 270) (fields_autoplaced)
-    (effects (font (size 1.27 1.27)) (justify right))
-    (property "Intersheetrefs" "${INTERSHEET_REFS}" (at 109.22 329.9972 90)
+    (effects (font (size 1 1)) (justify right))
+    (property "Intersheetrefs" "${INTERSHEET_REFS}" (at 109.22 326.5303 90)
       (effects (font (size 1.27 1.27)) (justify right) hide)
     )
@@
     )
   )
-  (global_label "Entrex Jmp Slot 13" (shape input) (at 281.94 289.56 90) (fields_autoplaced)
-    (effects (font (size 1.27 1.27)) (justify left))
-    (property "Intersheetrefs" "${INTERSHEET_REFS}" (at 281.94 268.4633 90)
+  (global_label "~{CON DATA}" (shape input) (at 119.38 277.495 90) (fields_autoplaced)
+    (effects (font (size 1 1)) (justify left))
+    (property "Intersheetrefs" "${INTERSHEET_REFS}" (at 119.38 268.0358 90)
       (effects (font (size 1.27 1.27)) (justify left) hide)
     )
@@
   )
   (global_label "Entrex P10.30" (shape input) (at 119.38 289.56 90) (fields_autoplaced)
-    (effects (font (size 1.27 1.27)) (justify left))
-    (property "Intersheetrefs" "${INTERSHEET_REFS}" (at 119.38 273.2528 90)
+    (effects (font (size 1 1)) (justify left))
+    (property "Intersheetrefs" "${INTERSHEET_REFS}" (at 119.38 276.7197 90)
       (effects (font (size 1.27 1.27)) (justify left) hide)
     )

Commit message: more
Connections:
- net ~{DRIVE IO}: now also J24.88 (Pin_4), J8.88 (Pin_4)
- net ~{READ IO}: now also J23.83, J7.83
- net 60Hz: now reaches J2B5.6
- no-connect marks 467 -> 462
Other:
- note added: "Slot 3 only?"
Changed lines of the file:
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@@
   (no_connect (at 254 238.76))
   (no_connect (at 248.92 149.86))
-  (no_connect (at 320.04 238.76))
   (no_connect (at 248.92 99.06))
   (no_connect (at 269.24 48.26))
@@
   (no_connect (at 279.4 86.36))
   (no_connect (at 251.46 48.26))
-  (no_connect (at 321.31 187.96))
   (no_connect (at 299.72 289.56))
   (no_connect (at 314.96 48.26))
@@
   (no_connect (at 200.66 302.26))
   (no_connect (at 177.8 149.86))
-  (no_connect (at 325.12 251.46))
   (no_connect (at 243.84 149.86))
   (no_connect (at 193.04 251.46))
@@
   (no_connect (at 185.42 137.16))
   (no_connect (at 312.42 35.56))
-  (no_connect (at 326.39 200.66))
   (no_connect (at 304.8 35.56))
   (no_connect (at 196.85 99.06))
@@
   (no_connect (at 300.99 187.96))
   (no_connect (at 228.6 149.86))
-  (no_connect (at 222.25 200.66))
   (no_connect (at 243.84 137.16))
   (no_connect (at 160.02 137.16))
@@
     (effects (font (size 1.27 1.27)) (justify left bottom))
   )
+  (text "Slot 3 only?" (at 222.885 208.28 90)
+    (effects (font (size 1.27 1.27)) (justify right bottom))
+  )
   (text "B" (at 280.035 61.595 0)
     (effects (font (size 1.27 1.27)) (justify right bottom))
@@
     )
   )
+  (global_label "~{READ IO}" (shape input) (at 321.31 187.96 90) (fields_autoplaced)
+    (effects (font (size 1.27 1.27)) (justify left))
+    (property "Intersheetrefs" "${INTERSHEET_REFS}" (at 321.31 177.5793 90)
+      (effects (font (size 1.27 1.27)) (justify left) hide)
+    )
+  )
   (global_label "+5V" (shape input) (at 204.47 99.06 270) (fields_autoplaced)
     (effects (font (size 1.27 1.27)) (justify right))
@@
     )
   )
+  (global_label "60Hz" (shape input) (at 222.25 200.66 270) (fields_autoplaced)
+    (effects (font (size 1.27 1.27)) (justify right))
+    (property "Intersheetrefs" "${INTERSHEET_REFS}" (at 222.25 208.3434 90)
+      (effects (font (size 1.27 1.27)) (justify right) hide)
+    )
+  )
   (global_label "DISK1" (shape input) (at 189.23 86.36 90) (fields_autoplaced)
     (effects (font (size 1.27 1.27)) (justify left))
@@
     )
   )
+  (global_label "~{READ IO}" (shape input) (at 320.04 238.76 90) (fields_autoplaced)
+    (effects (font (size 1.27 1.27)) (justify left))
+    (property "Intersheetrefs" "${INTERSHEET_REFS}" (at 320.04 228.3793 90)
+      (effects (font (size 1.27 1.27)) (justify left) hide)
+    )
+  )
   (global_label "RNIH4" (shape input) (at 99.06 187.96 90) (fields_autoplaced)
     (effects (font (size 1.27 1.27)) (justify left))
@@
     )
   )
+  (global_label "~{DRIVE IO}" (shape input) (at 326.39 200.66 270) (fields_autoplaced)
+    (effects (font (size 1.27 1.27)) (justify right))
+    (property "Intersheetrefs" "${INTERSHEET_REFS}" (at 326.39 211.6455 90)
+      (effects (font (size 1.27 1.27)) (justify right) hide)
+    )
+  )
   (global_label "GND" (shape input) (at 276.86 99.06 270) (fields_autoplaced)
     (effects (font (size 1.27 1.27)) (justify right))
@@
     )
   )
+  (global_label "~{DRIVE IO}" (shape input) (at 325.12 251.46 270) (fields_autoplaced)
+    (effects (font (size 1.27 1.27)) (justify right))
+    (property "Intersheetrefs" "${INTERSHEET_REFS}" (at 325.12 262.4455 90)
+      (effects (font (size 1.27 1.27)) (justify right) hide)
+    )
+  )

Commit message: mega-magic
Parts:
- removed J1, J3: Conn_02x40_Odd_Even, Forgotten Machines:Card_Edge_Entrex_Trapezoid 80, symbol Connector_Generic:Conn_02x40_Odd_Even
- removed J10, J11, J12, J13, J14, J15, J16, J17, J18, J19, J20, J21, J22, J23, J24, J5, J6, J7, J8, J9: Conn_01x10, symbol Connector_Generic:Conn_01x10
- removed J1A1, J1A2, J1A3, J1A4, J1A5, J1B1, J1B2, J1B3, J1B4, J1B5, J2A1, J2A2, J2A3, J2A4, J2A5, J2B1, J2B2, J2B3, J2B4, J2B5: Conn_01x40, symbol Connector_Generic:Conn_01x40
- removed J2, J4: DG Nova Card-Edge 81-100, Forgotten Machines:Data General Nova Card-Edge 81-100, symbol ForgottenMachines:DG_Nova_Card-Edge_81-100
- added J1 (x12): Slot_02x50_Odd_Even, Forgotten Machines:DG NOVA Backplane Connector - Frontside, symbol NovaMem-rescue:Slot_02x50_Odd_Even-_local
Connections:
- net +5V: now also J1.3 (Pin_3), J1.3 (Pin_3), J1.3 (Pin_3), J1.3 (Pin_3), J1.3 (Pin_3), J1.3 (Pin_3), J1.3 (Pin_3), J1.3 (Pin_3), J1.3 (Pin_3), J1.3 (Pin_3), J1.3 (Pin_3), J1.3 (Pin_3), J1.4 (Pin_4), J1.4 (Pin_4), J1.4 (Pin_4), J1.4 (Pin_4), J1.4 (Pin_4), J1.4 (Pin_4), J1.4 (Pin_4), J1.4 (Pin_4), J1.4 (Pin_4), J1.4 (Pin_4), J1.4 (Pin_4), J1.4 (Pin_4), J1.97 (Pin_69), J1.97 (Pin_69), J1.97 (Pin_69), J1.97 (Pin_69), J1.97 (Pin_69), J1.97 (Pin_69), J1.97 (Pin_69), J1.97 (Pin_69), J1.97 (Pin_69), J1.97 (Pin_69), J1.97 (Pin_69), J1.97 (Pin_69), J1.98 (Pin_98), J1.98 (Pin_98), J1.98 (Pin_98), J1.98 (Pin_98), J1.98 (Pin_98), J1.98 (Pin_98), J1.98 (Pin_98), J1.98 (Pin_98), J1.98 (Pin_98), J1.98 (Pin_98), J1.98 (Pin_98), J1.98 (Pin_98)
- net +5V OK: now also J1.8 (Pin_8)
- net +V MEM: now also J1.46 (Pin_46), J1.46 (Pin_46)
- net +V TERM: now also J1.11 (Pin_11), J1.13 (Pin_13)
- net +VINH: now also J1.10 (Pin_10), J1.10 (Pin_10), J1.10 (Pin_10), J1.10 (Pin_10), J1.10 (Pin_10), J1.84 (Pin_84), J1.84 (Pin_84), J1.84 (Pin_84), J1.84 (Pin_84), J1.84 (Pin_84)
- net -5 REMOTE: now also J1.6 (Pin_6)
- net -5V: now also J1.6 (Pin_6), J1.6 (Pin_6), J1.6 (Pin_6), J1.6 (Pin_6), J1.6 (Pin_6), J1.81 (Pin_81), J1.81 (Pin_81), J1.81 (Pin_81), J1.81 (Pin_81), J1.81 (Pin_81)
- net 60Hz: now also J1.6 (Pin_6)
- net 9 CH: now also J1.71 (Pin_71)
- net BOT: now also J1.53 (Pin_53)
- net CLK FLOP: now also J1.48 (Pin_48), J1.48 (Pin_48)
- net CLK RDR: now also J1.38 (Pin_38)
- net CLR: now also J1.50 (Pin_50), J1.50 (Pin_50), J1.50 (Pin_50), J1.50 (Pin_50), J1.50 (Pin_50), J1.50 (Pin_50)
- net DATA RDR: now also J1.36 (Pin_36)
- net DATIA: now also J1.44 (Pin_44), J1.44 (Pin_44), J1.44 (Pin_44), J1.44 (Pin_44), J1.44 (Pin_44), J1.44 (Pin_44)
- net DATIB: now also J1.42 (Pin_42), J1.42 (Pin_42), J1.42 (Pin_42), J1.42 (Pin_42), J1.42 (Pin_42), J1.42 (Pin_42)
- net DATIC: now also J1.54 (Pin_54), J1.54 (Pin_54), J1.54 (Pin_54), J1.54 (Pin_54), J1.54 (Pin_54), J1.54 (Pin_54)
- net DATOA: now also J1.58 (Pin_58), J1.58 (Pin_58), J1.58 (Pin_58), J1.58 (Pin_58), J1.58 (Pin_58), J1.58 (Pin_58)
- net DATOB: now also J1.56 (Pin_56), J1.56 (Pin_56), J1.56 (Pin_56), J1.56 (Pin_56), J1.56 (Pin_56), J1.56 (Pin_56)
- net DATOC: now also J1.48 (Pin_48), J1.48 (Pin_48), J1.48 (Pin_48), J1.48 (Pin_48), J1.48 (Pin_48), J1.48 (Pin_48)
- net DCHI: now also J1.37 (Pin_37), J1.37 (Pin_37), J1.37 (Pin_37), J1.37 (Pin_37), J1.37 (Pin_37), J1.37 (Pin_37)
- net DCHO: now also J1.33 (Pin_33), J1.33 (Pin_33), J1.33 (Pin_33), J1.33 (Pin_33), J1.33 (Pin_33), J1.33 (Pin_33)
- net DISK NEW REQ: now also J1.59 (Pin_59)
- net DISK PRES REQ: now also J1.57 (Pin_57)
- net DISK WR DATA: now also J1.63 (Pin_63), J1.71 (Pin_71)
- net DISK0: now also J1.69 (Pin_69)
- net DISK0 ACT: now also J1.61 (Pin_61)
- net DISK1: now also J1.85 (Pin_85)
- net DISK2: now also J1.81 (Pin_81)
- net DLY CNT: now also J1.47 (Pin_47)
- net DLY1: now also J1.81 (Pin_81)
- net DSK SEL: now also J1.67 (Pin_67)
- net DSK ~{RST}: now also J1.75 (Pin_75)
- net EOT: now also J1.48 (Pin_48)
- net Entrex Backplane S01B53 to S13B53: now also J1.53 (Pin_53), J1.53 (Pin_53)
- net Entrex P10.19: now also J1.24 (Pin_24)
- net Entrex P10.30: now also J1.29 (Pin_29)
- net GND: now also J1.1 (Pin_1), J1.1 (Pin_1), J1.1 (Pin_1), J1.1 (Pin_1), J1.1 (Pin_1), J1.1 (Pin_1), J1.1 (Pin_1), J1.1 (Pin_1), J1.1 (Pin_1), J1.1 (Pin_1), J1.1 (Pin_1), J1.1 (Pin_1), J1.100 (Pin_100), J1.100 (Pin_100), J1.100 (Pin_100), J1.100 (Pin_100), J1.100 (Pin_100), J1.100 (Pin_100), J1.100 (Pin_100), J1.100 (Pin_100), J1.100 (Pin_100), J1.100 (Pin_100), J1.100 (Pin_100), J1.100 (Pin_100), J1.2 (Pin_2), J1.2 (Pin_2), J1.2 (Pin_2), J1.2 (Pin_2), J1.2 (Pin_2), J1.2 (Pin_2), J1.2 (Pin_2), J1.2 (Pin_2), J1.2 (Pin_2), J1.2 (Pin_2), J1.2 (Pin_2), J1.2 (Pin_2), J1.33 (Pin_33), J1.33 (Pin_33), J1.33 (Pin_33), J1.33 (Pin_33), J1.33 (Pin_33), J1.33 (Pin_33), J1.34 (Pin_34), J1.34 (Pin_34), J1.34 (Pin_34), J1.34 (Pin_34), J1.34 (Pin_34), J1.34 (Pin_34), J1.50 (Pin_50), J1.50 (Pin_50), J1.50 (Pin_50), J1.50 (Pin_50), J1.50 (Pin_50), J1.50 (Pin_50), J1.89 (Pin_89), J1.89 (Pin_89), J1.92 (Pin_92), J1.92 (Pin_92), J1.99 (Pin_99), J1.99 (Pin_99), J1.99 (Pin_99), J1.99 (Pin_99), J1.99 (Pin_99), J1.99 (Pin_99), J1.99 (Pin_99), J1.99 (Pin_99), J1.99 (Pin_99), J1.99 (Pin_99), J1.99 (Pin_99), J1.99 (Pin_99)
- net HI DENS: now also J1.49 (Pin_49)
- net INH GND: now also J1.14 (Pin_14), J1.14 (Pin_14), J1.16 (Pin_16), J1.16 (Pin_16), J1.20 (Pin_20), J1.20 (Pin_20), J1.22 (Pin_22), J1.22 (Pin_22), J1.26 (Pin_26), J1.26 (Pin_26), J1.30 (Pin_30), J1.30 (Pin_30), J1.31 (Pin_31), J1.31 (Pin_31), J1.8 (Pin_8), J1.8 (Pin_8)
- net INHIBIT: now also J1.30 (Pin_30), J1.30 (Pin_30), J1.30 (Pin_30)
- net INTA: now also J1.40 (Pin_40), J1.40 (Pin_40), J1.40 (Pin_40), J1.40 (Pin_40), J1.40 (Pin_40), J1.40 (Pin_40)
- net IO PLS: now also J1.74 (Pin_74), J1.74 (Pin_74), J1.74 (Pin_74), J1.74 (Pin_74), J1.74 (Pin_74), J1.74 (Pin_74)
- net IO RST: now also J1.70 (Pin_70), J1.70 (Pin_70), J1.70 (Pin_70), J1.70 (Pin_70), J1.70 (Pin_70), J1.70 (Pin_70)
- net LOAD IR: now also J1.73 (Pin_73), J1.73 (Pin_73)
- net MB LOAD: now also J1.74 (Pin_74), J1.74 (Pin_74), J1.74 (Pin_74)
- net MEM OK: now also J1.9 (Pin_9)
- net OS2: now also J1.90 (Pin_90)
- net OVFLO: now also J1.39 (Pin_39), J1.39 (Pin_39), J1.39 (Pin_39), J1.39 (Pin_39), J1.39 (Pin_39), J1.39 (Pin_39)
- net RB0: now also J1.31 (Pin_31)
- net RB1: now also J1.40 (Pin_40)
- net RB2: now also J1.25 (Pin_25)
- net RB3: now also J1.27 (Pin_27)
- net RB4: now also J1.13 (Pin_13)
- net RB5: now also J1.15 (Pin_15)
- net RB6: now also J1.19 (Pin_19)
- net RB7: now also J1.23 (Pin_23)
- net RBP: now also J1.38 (Pin_38)
- net RD EN: now also J1.76 (Pin_76)
- net RESTART ENABLE: now also J1.32 (Pin_32)
- net RINH12: now also J1.28 (Pin_28), J1.28 (Pin_28)
- net RINH6: now also J1.18 (Pin_18), J1.18 (Pin_18), J1.19 (Pin_19)
- net RINH9: now also J1.24 (Pin_24), J1.24 (Pin_24)
- net ROS: now also J1.78 (Pin_78), J1.78 (Pin_78)
- net RPO: now also J1.49 (Pin_49)
- net RWND T: now also J1.69 (Pin_69)
- net RWNDG: now also J1.11 (Pin_11)
- net SEL 2 (1): now also J1.78 (Pin_78)
- net SEL 2 (2): now also J1.79 (Pin_79)
- net SEL EN: now also J1.76 (Pin_76)
- net SEL2: now also J1.75 (Pin_75)
- net SND CLK: now also J1.63 (Pin_63)
- net SPARE: now also J1.79 (Pin_79)
- net SPC BKD: now also J1.67 (Pin_67)
- net STROBE: now also J1.20 (Pin_20), J1.20 (Pin_20), J1.20 (Pin_20)
- net STRT: now also J1.52 (Pin_52), J1.52 (Pin_52), J1.52 (Pin_52), J1.52 (Pin_52), J1.52 (Pin_52), J1.52 (Pin_52)
- net TRK0: now also J1.84 (Pin_84)
- net TRK1: now also J1.86 (Pin_86)
- net TRK2: now also J1.87 (Pin_87)
- net TRK3: now also J1.83 (Pin_83)
- net TRK4: now also J1.89 (Pin_89)
- net TRK5: now also J1.91 (Pin_91)
- net TRK6: now also J1.73 (Pin_73)
- net TUR: now also J1.54 (Pin_54)
- net WALLOUT: now also J1.65 (Pin_65)
- net WB0: now also J1.87 (Pin_87)
- net WB1: now also J1.85 (Pin_85)
- net WB2: now also J1.89 (Pin_89)
- net WB3: now also J1.84 (Pin_84)
- net WB4: now also J1.91 (Pin_91)
- net WB5: now also J1.86 (Pin_86)
- net WB6: now also J1.34 (Pin_34)
- net WB7: now also J1.83 (Pin_83)
- net WBP: now also J1.59 (Pin_59)
- net WL: now also J1.36 (Pin_36)
- net WRT: now also J1.88 (Pin_88)
- net WRT STROBE: now also J1.77 (Pin_77)
- net WRT ~{RST}: now also J1.57 (Pin_57)
- net WRT7: now also J1.61 (Pin_61)
- net ~{BMA LOAD}: now also J1.10 (Pin_10), J1.10 (Pin_10)
- net ~{CARRY}: now also J1.15 (Pin_15)
- net ~{CON DATA}: now also J1.28 (Pin_28)
- net ~{CON INST}: now also J1.22 (Pin_22)
- net ~{CON RQ}: now also J1.27 (Pin_27)
- net ~{CONT+ISTP+MSTP}: now also J1.25 (Pin_25)
- net ~{DATA0}: now also J1.62 (Pin_62), J1.62 (Pin_62), J1.62 (Pin_62), J1.62 (Pin_62), J1.62 (Pin_62), J1.62 (Pin_62)
- net ~{DATA10}: now also J1.75 (Pin_75), J1.75 (Pin_75), J1.75 (Pin_75), J1.75 (Pin_75), J1.75 (Pin_75), J1.75 (Pin_75)
- net ~{DATA11}: now also J1.58 (Pin_58), J1.58 (Pin_58), J1.58 (Pin_58), J1.58 (Pin_58), J1.58 (Pin_58), J1.58 (Pin_58)
- net ~{DATA12}: now also J1.59 (Pin_59), J1.59 (Pin_59), J1.59 (Pin_59), J1.59 (Pin_59), J1.59 (Pin_59), J1.59 (Pin_59)
- net ~{DATA13}: now also J1.64 (Pin_64), J1.64 (Pin_64), J1.64 (Pin_64), J1.64 (Pin_64), J1.64 (Pin_64), J1.64 (Pin_64)
- net ~{DATA14}: now also J1.56 (Pin_56), J1.56 (Pin_56), J1.56 (Pin_56), J1.56 (Pin_56), J1.56 (Pin_56), J1.56 (Pin_56)
- net ~{DATA15}: now also J1.66 (Pin_66), J1.66 (Pin_66), J1.66 (Pin_66), J1.66 (Pin_66), J1.66 (Pin_66), J1.66 (Pin_66)
- net ~{DATA1}: now also J1.65 (Pin_65), J1.65 (Pin_65), J1.65 (Pin_65), J1.65 (Pin_65), J1.65 (Pin_65), J1.65 (Pin_65)
- net ~{DATA2}: now also J1.82 (Pin_82), J1.82 (Pin_82), J1.82 (Pin_82), J1.82 (Pin_82), J1.82 (Pin_82), J1.82 (Pin_82)
- net ~{DATA3}: now also J1.73 (Pin_73), J1.73 (Pin_73), J1.73 (Pin_73), J1.73 (Pin_73), J1.73 (Pin_73), J1.73 (Pin_73)
- net ~{DATA4}: now also J1.61 (Pin_61), J1.61 (Pin_61), J1.61 (Pin_61), J1.61 (Pin_61), J1.61 (Pin_61), J1.61 (Pin_61)
- net ~{DATA5}: now also J1.57 (Pin_57), J1.57 (Pin_57), J1.57 (Pin_57), J1.57 (Pin_57), J1.57 (Pin_57), J1.57 (Pin_57)
- net ~{DATA6}: now also J1.95 (Pin_95), J1.95 (Pin_95), J1.95 (Pin_95), J1.95 (Pin_95), J1.95 (Pin_95), J1.95 (Pin_95)
- net ~{DATA7}: now also J1.55 (Pin_55), J1.55 (Pin_55), J1.55 (Pin_55), J1.55 (Pin_55), J1.55 (Pin_55), J1.55 (Pin_55)
- net ~{DATA8}: now also J1.60 (Pin_60), J1.60 (Pin_60), J1.60 (Pin_60), J1.60 (Pin_60), J1.60 (Pin_60), J1.60 (Pin_60)
- net ~{DATA9}: now also J1.63 (Pin_63), J1.63 (Pin_63), J1.63 (Pin_63), J1.63 (Pin_63), J1.63 (Pin_63), J1.63 (Pin_63)
- net ~{DCHA}: now also J1.60 (Pin_60), J1.60 (Pin_60), J1.60 (Pin_60), J1.60 (Pin_60), J1.60 (Pin_60), J1.60 (Pin_60)
- net ~{DCHM0}: now also J1.17 (Pin_17), J1.17 (Pin_17), J1.17 (Pin_17), J1.17 (Pin_17), J1.17 (Pin_17), J1.17 (Pin_17)
- net ~{DCHM1}: now also J1.21 (Pin_21), J1.21 (Pin_21), J1.21 (Pin_21), J1.21 (Pin_21), J1.21 (Pin_21), J1.21 (Pin_21)
- net ~{DCHP IN}: now also J1.94 (Pin_94), J1.94 (Pin_94), J1.94 (Pin_94), J1.94 (Pin_94), J1.94 (Pin_94)
- net ~{DCHP OUT}: now also J1.93 (Pin_93), J1.93 (Pin_93), J1.93 (Pin_93), J1.93 (Pin_93), J1.93 (Pin_93)
- net ~{DCHR}: now also J1.35 (Pin_35), J1.35 (Pin_35), J1.35 (Pin_35), J1.35 (Pin_35), J1.35 (Pin_35), J1.35 (Pin_35)
- net ~{DEFER}: now also J1.12 (Pin_12)
- net ~{DIV}: now also J1.91 (Pin_91), J1.91 (Pin_91)
- net ~{DRIVE IO}: now also J1.88 (Pin_88), J1.88 (Pin_88), J1.88 (Pin_88)
- net ~{DS0}: now also J1.72 (Pin_72), J1.72 (Pin_72), J1.72 (Pin_72), J1.72 (Pin_72), J1.72 (Pin_72), J1.72 (Pin_72)
- net ~{DS1}: now also J1.68 (Pin_68), J1.68 (Pin_68), J1.68 (Pin_68), J1.68 (Pin_68), J1.68 (Pin_68), J1.68 (Pin_68)
- net ~{DS2}: now also J1.66 (Pin_66), J1.66 (Pin_66), J1.66 (Pin_66), J1.66 (Pin_66), J1.66 (Pin_66), J1.66 (Pin_66)
- net ~{DS3}: now also J1.46 (Pin_46), J1.46 (Pin_46), J1.46 (Pin_46), J1.46 (Pin_46), J1.46 (Pin_46), J1.46 (Pin_46)
- net ~{DS4}: now also J1.62 (Pin_62), J1.62 (Pin_62), J1.62 (Pin_62), J1.62 (Pin_62), J1.62 (Pin_62), J1.62 (Pin_62)
- net ~{DS5}: now also J1.64 (Pin_64), J1.64 (Pin_64), J1.64 (Pin_64), J1.64 (Pin_64), J1.64 (Pin_64), J1.64 (Pin_64)
- net ~{EXEC}: now also J1.11 (Pin_11)
- net ~{EXT LOAD}: now also J1.47 (Pin_47), J1.47 (Pin_47), J1.49 (Pin_49), J1.49 (Pin_49)
- net ~{EXT SELECT}: now also J1.80 (Pin_80), J1.80 (Pin_80)
- net ~{FETCH}: now also J1.13 (Pin_13), J1.49 (Pin_49), J1.49 (Pin_49)
- net ~{FORCE LOAD IR}: now also J1.85 (Pin_85), J1.85 (Pin_85)
- net ~{INH TRANS}: now also J1.45 (Pin_45), J1.45 (Pin_45), J1.45 (Pin_45)
- net ~{INHIBIT SELECT}: now also J1.85 (Pin_85), J1.85 (Pin_85)
- net ~{INTP IN}: now also J1.96 (Pin_96), J1.96 (Pin_96), J1.96 (Pin_96), J1.96 (Pin_96), J1.96 (Pin_96)
- net ~{INTP OUT}: now also J1.95 (Pin_95), J1.95 (Pin_95), J1.95 (Pin_95), J1.95 (Pin_95), J1.95 (Pin_95)
- net ~{INTR}: now also J1.29 (Pin_29), J1.29 (Pin_29), J1.29 (Pin_29), J1.29 (Pin_29), J1.29 (Pin_29), J1.29 (Pin_29)
- net ~{ION}: now also J1.16 (Pin_16)
- net ~{ISTP}: now also J1.17 (Pin_17)
- net ~{LOAD AC}: now also J1.77 (Pin_77), J1.77 (Pin_77)
- net ~{MA LOAD}: now also J1.7 (Pin_7), J1.7 (Pin_7), J1.7 (Pin_7)
- net ~{MB CLEAR}: now also J1.86 (Pin_86), J1.86 (Pin_86), J1.86 (Pin_86)
- net ~{MBO0}: now also J1.79 (Pin_79), J1.79 (Pin_79), J1.79 (Pin_79)
- net ~{MBO10}: now also J1.8 (Pin_8), J1.8 (Pin_8), J1.8 (Pin_8)
- net ~{MBO11}: now also J1.5 (Pin_5), J1.5 (Pin_5), J1.5 (Pin_5)
- net ~{MBO12}: now also J1.39 (Pin_39), J1.39 (Pin_39), J1.39 (Pin_39)
- net ~{MBO13}: now also J1.37 (Pin_37), J1.37 (Pin_37), J1.37 (Pin_37)
- net ~{MBO14}: now also J1.43 (Pin_43), J1.43 (Pin_43), J1.43 (Pin_43)
- net ~{MBO15}: now also J1.41 (Pin_41), J1.41 (Pin_41), J1.41 (Pin_41)
- net ~{MBO1}: now also J1.77 (Pin_77), J1.77 (Pin_77), J1.77 (Pin_77)
- net ~{MBO2}: now also J1.44 (Pin_44), J1.44 (Pin_44), J1.44 (Pin_44)
- net ~{MBO3}: now also J1.43 (Pin_43), J1.43 (Pin_43), J1.43 (Pin_43)
- net ~{MBO4}: now also J1.42 (Pin_42), J1.42 (Pin_42), J1.42 (Pin_42)
- net ~{MBO5}: now also J1.32 (Pin_32), J1.32 (Pin_32), J1.32 (Pin_32)
- net ~{MBO6}: now also J1.16 (Pin_16), J1.16 (Pin_16), J1.16 (Pin_16)
- net ~{MBO7}: now also J1.14 (Pin_14), J1.14 (Pin_14), J1.14 (Pin_14)
- net ~{MBO8}: now also J1.12 (Pin_12), J1.12 (Pin_12), J1.12 (Pin_12)
- net ~{MBO9}: now also J1.9 (Pin_9), J1.9 (Pin_9), J1.9 (Pin_9)
- net ~{MD SEL1}: now also J1.87 (Pin_87), J1.87 (Pin_87)
- net ~{MEM0}: now also J1.71 (Pin_71), J1.71 (Pin_71), J1.71 (Pin_71)
- net ~{MEM10}: now also J1.45 (Pin_45), J1.45 (Pin_45), J1.45 (Pin_45)
- net ~{MEM11}: now also J1.51 (Pin_51), J1.51 (Pin_51), J1.51 (Pin_51)
- net ~{MEM12}: now also J1.36 (Pin_36), J1.36 (Pin_36), J1.36 (Pin_36)
- net ~{MEM13}: now also J1.35 (Pin_35), J1.35 (Pin_35), J1.35 (Pin_35)
- net ~{MEM14}: now also J1.76 (Pin_76), J1.76 (Pin_76), J1.76 (Pin_76)
- net ~{MEM15}: now also J1.18 (Pin_18), J1.18 (Pin_18), J1.18 (Pin_18)
- net ~{MEM1}: now also J1.70 (Pin_70), J1.70 (Pin_70), J1.70 (Pin_70)
- net ~{MEM2}: now also J1.47 (Pin_47), J1.47 (Pin_47), J1.47 (Pin_47)
- net ~{MEM3}: now also J1.68 (Pin_68), J1.68 (Pin_68), J1.68 (Pin_68)
- net ~{MEM4}: now also J1.28 (Pin_28), J1.28 (Pin_28), J1.28 (Pin_28)
- net ~{MEM5}: now also J1.26 (Pin_26), J1.26 (Pin_26), J1.26 (Pin_26)
- net ~{MEM6}: now also J1.22 (Pin_22), J1.22 (Pin_22), J1.22 (Pin_22)
- net ~{MEM7}: now also J1.24 (Pin_24), J1.24 (Pin_24), J1.24 (Pin_24)
- net ~{MEM8}: now also J1.55 (Pin_55), J1.55 (Pin_55), J1.55 (Pin_55)
- net ~{MEM9}: now also J1.53 (Pin_53), J1.53 (Pin_53), J1.53 (Pin_53)
- net ~{MSKO}: now also J1.38 (Pin_38), J1.38 (Pin_38), J1.38 (Pin_38), J1.38 (Pin_38), J1.38 (Pin_38), J1.38 (Pin_38)
- net ~{MSTP}: now also J1.20 (Pin_20)
- net ~{PL}: now also J1.19 (Pin_19)
- net ~{POWER FAIL}: now also J1.5 (Pin_5)
- net ~{READ IO}: now also J1.83 (Pin_83), J1.83 (Pin_83), J1.83 (Pin_83)
- net ~{READ1}: now also J1.87 (Pin_87), J1.87 (Pin_87), J1.87 (Pin_87)
- net ~{READ2}: now also J1.90 (Pin_90), J1.90 (Pin_90), J1.90 (Pin_90)
- net ~{RELOAD DISABLE}: now also J1.72 (Pin_72), J1.72 (Pin_72)
- net ~{RQENB}: now also J1.41 (Pin_41), J1.41 (Pin_41), J1.41 (Pin_41), J1.41 (Pin_41), J1.41 (Pin_41), J1.41 (Pin_41)
- net ~{RST}: now also J1.30 (Pin_30)
- net ~{RUN}: now also J1.14 (Pin_14), J1.73 (Pin_73)
- net ~{SELB}: now also J1.82 (Pin_82), J1.82 (Pin_82), J1.82 (Pin_82), J1.82 (Pin_82), J1.82 (Pin_82), J1.82 (Pin_82)
- net ~{SELD}: now also J1.80 (Pin_80), J1.80 (Pin_80), J1.80 (Pin_80), J1.80 (Pin_80), J1.80 (Pin_80), J1.80 (Pin_80)
- net ~{SHIFT0}: now also J1.94 (Pin_94), J1.94 (Pin_94)
- net ~{SHIFT1}: now also J1.96 (Pin_96), J1.96 (Pin_96)
- net ~{SHIFT2}: now also J1.93 (Pin_93), J1.93 (Pin_93)
- net ~{SHIFT3}: now also J1.91 (Pin_91), J1.91 (Pin_91)
- net ~{SKIP}: now also J1.69 (Pin_69), J1.69 (Pin_69)
- net ~{STOP}: now also J1.31 (Pin_31)
- net ~{TEST}: now also J1.92 (Pin_92), J1.92 (Pin_92)
- net ~{WAS JSR}: now also J1.89 (Pin_89), J1.89 (Pin_89)
- net ~{WHOA}: now also J1.6 (Pin_6), J1.6 (Pin_6)
- new net RINH0: J1.5 (Pin_5), J1.5 (Pin_5)
- new net RINH1: J1.7 (Pin_7), J1.7 (Pin_7)
- new net RINH10: J1.23 (Pin_23), J1.23 (Pin_23)
- new net RINH11: J1.21 (Pin_21), J1.21 (Pin_21)
- new net RINH13: J1.25 (Pin_25), J1.25 (Pin_25)
- new net RINH14: J1.29 (Pin_29), J1.29 (Pin_29)
- new net RINH15: J1.27 (Pin_27), J1.27 (Pin_27)
- new net RINH2: J1.9 (Pin_9), J1.9 (Pin_9)
- new net RINH3: J1.11 (Pin_11), J1.11 (Pin_11)
- new net RINH4: J1.13 (Pin_13), J1.13 (Pin_13)
- new net RINH5: J1.15 (Pin_15), J1.15 (Pin_15)
- new net RINH7: J1.17 (Pin_17), J1.17 (Pin_17)
- new net RINH8: J1.19 (Pin_19)

Commit message: big build
Other:
- note removed: "* Means original text was unclear ? Also means original source was unclear This for the nova 1200/800 cpu slot 1 only, see other pages for other slots."
- note removed: "Drawn by Jake Utley"
- note removed: "Nixdorf 620 schematic book, Data general 1969 nova and 1200 technical manual were sources"
Changed lines of the file:
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@@
     (effects (font (size 1.27 1.27)) (justify right bottom))
-  )
-  (text "* Means original text was unclear\n? Also means original source was unclear\n\nThis for the nova 1200/800 cpu slot 1 only, see other pages for other slots."
-    (at 281.94 364.49 0)
-    (effects (font (size 1.27 1.27)) (justify left bottom))
-  )
-  (text "Nixdorf 620 schematic book, Data general 1969 nova and 1200 technical manual were sources\n"
-    (at 281.94 367.03 0)
-    (effects (font (size 1.27 1.27)) (justify left bottom))
   )
   (text "B" (at 280.67 276.86 0)
@@
     (effects (font (size 1.27 1.27)) (justify right bottom))
   )
-  (text "Drawn by Jake Utley" (at 281.94 369.57 0)
-    (effects (font (size 1.27 1.27)) (justify left bottom))
-  )
   (text "RUN not inverted (~{RUN}) on \nBack Panel Nova 1200\nDrawing No. 000090"
