File: CPU Pictures/Nova 1200/CPU Card Edge/CPU Card Edge.kicad_sch (KiCad schematic)
At the start: 55 parts, among them J1 Conn_02x40_Odd_Even, J2 DG Nova Card-Edge 81-100, J3 Conn_02x40_Odd_Even, J4 DG Nova Card-Edge 81-100

Commit message: Build
Parts:
- R51: value 220 -> 330
- R51: value 220 -> 470
Connections:
- no-connect marks 57 -> 58
Other:
- note added: "DATA0-DATA15 terminators"
- moved on the sheet: R51
