File: DG Nova PSU Connector Board w_start-up sequence/DG Nova PSU Connector Board w_start-up sequence.kicad_pcb (KiCad board)
At the start: 2 copper layers, 130 x 90.8 mm, 48 parts, among them J1 Conn_02x07_Counter_Clockwise, J10 Conn_01x06, J11 Conn_01x06, J12 Conn_01x06, J13 Conn_01x06, J14 Conn_01x06, J15 Conn_01x06, J16 Conn_01x06, J17 Conn_01x06, J18 Conn_01x06, J19 Conn_01x06, J2 Conn_01x12, J20 Conn_01x06, J21 Conn_01x06, J22 Conn_01x06, J23 Conn_01x11, J24 Conn_01x11, J25 Conn_01x11, J26 Conn_01x11, J3 Conn_01x12, J7 Conn_01x12, J8 Conn_01x06, J9 Conn_01x06, U1 74HC14

Commit message: Add Sync
Parts:
- removed J7: Conn_01x12, Card Edge:PinHeader_1x12_P2.54mm_Vertical
- added .: PinHeader_2x12_P2.54mm_Vertical, Connector_PinHeader_2.54mm:PinHeader_2x12_P2.54mm_Vertical, F.Cu at (92.2, 88.6)
Routing:
- net GND: track 25.8 -> 27.4 mm
Other:
- board text removed: "FORGOTTEN MACHINES"
