File: DG Nova Extender Board/Backplane Socket Board.kicad_pcb (KiCad board)
At the start: 2 copper layers, 379 x 83.8 mm, 6 parts, among them J1 portAB, J2 portCD, X2 Slot 1 A2, X4 Slot 1 B2, X6 Slot 2 A2, X8 Slot 2 B2

Commit message: More Magic
Parts:
- removed X2: Slot 1 A2, Connector_IDC:IDC-Header_2x25_P2.54mm_Vertical
- removed X4: Slot 1 B2, Connector_IDC:IDC-Header_2x25_P2.54mm_Vertical
- removed X6: Slot 2 A2, Connector_IDC:IDC-Header_2x25_P2.54mm_Vertical
- removed X8: Slot 2 B2, Connector_IDC:IDC-Header_2x25_P2.54mm_Vertical
- added J1: Port A, Forgotten Machines:DG NOVA Backplane Connector - Frontside, F.Cu at (308.9, 94.4)
- added J2: Port B, Forgotten Machines:DG NOVA Backplane Connector - Frontside, F.Cu at (119.7, 94.4)
- added X1: A1, Connector_IDC:IDC-Header_2x25_P2.54mm_Vertical, F.Cu at (378.3, 54.7)
- added X3: A2, Connector_IDC:IDC-Header_2x25_P2.54mm_Vertical, F.Cu at (297.1, 54.6)
- added X5: B1, Connector_IDC:IDC-Header_2x25_P2.54mm_Vertical, F.Cu at (195.5, 54.7)
- added X7: B2, Connector_IDC:IDC-Header_2x25_P2.54mm_Vertical, F.Cu at (114.2, 54.7)
Connections:
- J2 pad 100: (no net) -> d50
Routing:
- net (no net): track 8808.0 -> 0.00 mm
- net c50: track 0.00 -> 50.1 mm
- net c48: track 0.00 -> 49.8 mm
- net c46: track 0.00 -> 49.5 mm
- net c44: track 0.00 -> 49.3 mm
- net d50: track 0.00 -> 49.3 mm
- net c42: track 0.00 -> 49.0 mm
- net d48: track 0.00 -> 49.0 mm
- net d46: track 0.00 -> 48.7 mm
- net c40: track 0.00 -> 48.7 mm
- net c38: track 0.00 -> 48.6 mm
- net d44: track 0.00 -> 48.5 mm
- net d42: track 0.00 -> 48.2 mm
- net c36: track 0.00 -> 48.1 mm
- net d40: track 0.00 -> 48.0 mm
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Other:
- board text added: "A1"
- board text added: "A2"
- board text added: "B1"
- board text added: "B2"
- board text added: "Spacing???"
- board text removed: "A1.1"
- board text removed: "A2.1"
- board text removed: "B1.1"
- board text removed: "B2.1"

Commit message: card extender
Parts:
- moved J2 1.44 mm to (118.3, 94.1)
- moved J1 1.44 mm to (307.5, 94.1)
Changed lines of the file:
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@@
   )
   (footprint "Forgotten Machines:DG NOVA Backplane Connector - Frontside" (layer "F.Cu")
-    (at 119.65 94.441)
+    (at 118.253 94.107)
     (property "Sheetfile" "Backplane Socket Board.kicad_sch")
     (property "Sheetname" "")
@@
   )
   (footprint "Forgotten Machines:DG NOVA Backplane Connector - Frontside" (layer "F.Cu")
-    (at 308.88 94.441)
+    (at 307.483 94.107)
     (property "Sheetfile" "Backplane Socket Board.kicad_sch")
     (property "Sheetname" "")
@@
     )
   )
-  (gr_rect (start 193.04 100.076) (end 234.95 108.585)
+  (gr_rect (start 191.643 99.742) (end 233.553 108.251)
     (stroke (width 0.2) (type default)) (fill none) (layer "F.Cu"))
   (gr_line (start 119.634 54.737) (end 115.57 54.737)
@@
   (gr_line (start 196.85 54.864) (end 197.612 53.848)
     (stroke (width 0.12) (type default)) (layer "B.SilkS"))
+  (gr_line (start 229.743 33.401) (end 229.743 83.058)
+    (stroke (width 0.12) (type default)) (layer "F.SilkS"))
   (gr_line (start 201.041 54.7116) (end 197.231 54.7116)
     (stroke (width 0.12) (type default)) (layer "F.SilkS"))
@@
   (gr_line (start 298.831 54.7116) (end 298.323 54.7116)
     (stroke (width 0.12) (type default)) (layer "F.SilkS"))
+  (gr_line (start 195.453 34.29) (end 195.453 82.931)
+    (stroke (width 0.12) (type default)) (layer "F.SilkS"))
   (gr_line (start 380.365 54.2036) (end 380.365 53.9496)
     (stroke (width 0.12) (type default)) (layer "F.SilkS"))
@@
   (gr_arc (start 228.473 27.813) (mid 228.658987 27.363987) (end 229.108 27.178)
     (stroke (width 0.05) (type solid)) (layer "Edge.Cuts"))
-  (gr_text "Spacing???\n" (at 208.28 87.249) (layer "F.Cu")
+  (gr_text "Spacing???\n" (at 206.883 86.915) (layer "F.Cu")
     (effects (font (size 1.5 1.5) (thickness 0.3) bold) (justify left bottom))
   )
@@
     (effects (font (size 1 1) (thickness 0.2) bold) (justify left bottom mirror))
   )
-  (gr_text "A" (at 308.483 81.915) (layer "F.SilkS")
+  (gr_text "A" (at 307.086 81.581) (layer "F.SilkS")
     (effects (font (size 5.08 4.064) (thickness 0.762)))
   )
@@
     (effects (font (size 2.032 1.524) (thickness 0.254)))
   )
-  (gr_text "B" (at 118.999 81.407) (layer "F.SilkS")
+  (gr_text "B" (at 117.602 81.073) (layer "F.SilkS")
     (effects (font (size 5.08 4.064) (thickness 0.762)))
   )
@@
     (effects (font (size 2.032 1.524) (thickness 0.254)))
   )
-  (gr_text "B" (at 118.999 105.537) (layer "F.SilkS")
+  (gr_text "B" (at 117.602 105.203) (layer "F.SilkS")
     (effects (font (size 5.08 4.064) (thickness 0.762)))
   )
@@
     (effects (font (size 2.032 1.524) (thickness 0.254)))
   )
-  (gr_text "A" (at 308.483 106.045) (layer "F.SilkS")
+  (gr_text "A" (at 306.959 105.711) (layer "F.SilkS")
     (effects (font (size 5.08 4.064) (thickness 0.762)))
   )
   (dimension (type aligned) (layer "F.SilkS")
-    (pts (xy 196.85 91.186) (xy 230.505 91.186))
+    (pts (xy 195.453 90.852) (xy 229.108 90.852))
     (height -6.858)
-    (gr_text "33.6550 mm" (at 213.6775 83.178) (layer "F.SilkS")
+    (gr_text "33.6550 mm" (at 212.2805 82.844) (layer "F.SilkS")
       (effects (font (size 1 1) (thickness 0.15)))
     )

Commit message: build
Parts:
- J1: value portAB -> port A
- J2: value portCD -> port B
- moved X1 0.64 mm to (377.7, 54.7)
- moved J1 0.63 mm to (384.7, 31.6)
- moved X3 0.63 mm to (296.4, 54.6)
Routing:
- net c50: track 50.1 -> 80.3 mm
- net c48: track 49.8 -> 79.7 mm
- net c46: track 49.5 -> 79.2 mm
- net c44: track 49.3 -> 78.7 mm
- net d50: track 49.3 -> 78.7 mm
- net d48: track 49.0 -> 78.2 mm
- net c42: track 49.0 -> 78.2 mm
- net d46: track 48.7 -> 77.6 mm
- net c40: track 48.7 -> 77.6 mm
- net a50: track 47.3 -> 75.9 mm
- net d44: track 48.5 -> 77.1 mm
- net c38: track 48.6 -> 77.2 mm
- net a48: track 46.8 -> 75.2 mm
- net c36: track 48.1 -> 76.5 mm
- net d42: track 48.2 -> 76.6 mm
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Other:
- outline, holes or cut-outs redrawn
