File: DG Nova Extender Board/Backplane Socket Board.kicad_pcb (KiCad board)
At the start: 2 copper layers, 379 x 83.8 mm, 8 parts, among them J1 Port A, J1 port A, J2 Port B, J2 port B, X1 A1, X3 A2, X5 B1, X7 B2

Commit message: changes
Other:
- board text added: "PLUG CABLES INTO THIS SIDE OF BOARD"

Commit message: swap connectors
Parts:
- X1, X3, X5, X7: footprint Connector_IDC:IDC-Header_2x25_P2.54mm_Vertical -> Forgotten Machines:IDC-Header_2x25_P2.54mm - Backside
- moved X1 298.3 mm to (115.3, -87.2), turned to 0 degrees
- moved X3 222.8 mm to (115.3, -75.2), turned to 0 degrees
- moved X5 142.6 mm to (115.3, -63.3), turned to 0 degrees
- moved X7 106.0 mm to (115.3, -51.3), turned to 0 degrees

Commit message: yeah
Parts:
- moved X1 273.7 mm to (347.2, 58.2)
Changed lines of the file:
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@@
   )
   (footprint "Forgotten Machines:IDC-Header_2x25_P2.54mm - Backside" (layer "F.Cu")
-    (at 115.316 -87.224)
+    (at 347.218 58.205)
     (descr "Through hole IDC box header, 2x25, 2.54mm pitch, DIN 41651 / IEC 60603-13, double rows, https://docs.google.com/spreadsheets/d/16SsEcesNF15N3Lb4niX7dcUr-NY5_MFPQhobNuNppn4/edit#gid=0")
     (tags "Through hole vertical IDC box header THT 2x25 2.54mm double row")
@@
     (property "ki_keywords" "connector")
     (attr through_hole)
-    (fp_text reference "X1" (at 36.58 0.215 -90) (layer "F.SilkS")
+    (fp_text reference "X1" (at 33.02 0.102 -90) (layer "F.SilkS") hide
         (effects (font (size 1 1) (thickness 0.15)))
     )
-    (fp_text value "A1" (at -18.415 -12.065) (layer "F.Fab")
+    (fp_text value "A1" (at -32.766 0.356) (layer "F.Fab") hide
         (effects (font (size 1 1) (thickness 0.15)))
     )
@@
   (gr_line (start 211.272723 68.503419) (end 211.32118 68.508007)
     (stroke (width 0.0508) (type solid)) (layer "B.SilkS"))
-  (gr_line (start 379.73 54.102) (end 379.73 54.61)
+  (gr_line (start 379.73 59.182) (end 379.73 59.69)
     (stroke (width 0.12) (type default)) (layer "B.SilkS"))
   (gr_line (start 216.020066 71.562774) (end 215.936296 71.555174)
@@
   (gr_line (start 208.192129 72.070748) (end 208.221979 72.021688)
     (stroke (width 0.0508) (type solid)) (layer "B.SilkS"))
-  (gr_line (start 379.73 53.848) (end 379.73 54.102)
+  (gr_line (start 379.73 58.928) (end 379.73 59.182)
     (stroke (width 0.12) (type default)) (layer "B.SilkS"))
   (gr_line (start 219.357501 70.433462) (end 219.320831 70.456282)
@@
   (gr_line (start 212.229185 77.238413) (end 212.186965 77.236213)
     (stroke (width 0.0508) (type solid)) (layer "B.SilkS"))
-  (gr_line (start 379.73 54.61) (end 379.73 55.372)
+  (gr_line (start 379.73 59.69) (end 379.73 60.452)
     (stroke (width 0.12) (type default)) (layer "B.SilkS"))
   (gr_line (start 228.026597 69.200915) (end 228.058257 69.207715)
@@
   (gr_line (start 217.947283 68.764396) (end 217.971133 68.787786)
     (stroke (width 0.0508) (type solid)) (layer "B.SilkS"))
-  (gr_line (start 379.476 54.61) (end 383.286 54.61)
+  (gr_line (start 379.476 59.69) (end 383.286 59.69)
     (stroke (width 0.12) (type default)) (layer "B.SilkS"))
   (gr_line (start 207.342209 73.959313) (end 205.663678 73.959313)
@@
   (gr_line (start 206.166064 75.497059) (end 206.107934 75.520169)
     (stroke (width 0.0508) (type solid)) (layer "B.SilkS"))
-  (gr_line (start 378.968 54.61) (end 379.476 54.61)
+  (gr_line (start 378.968 59.69) (end 379.476 59.69)
     (stroke (width 0.12) (type default)) (layer "B.SilkS"))
   (gr_line (start 219.72412 70.390022) (end 219.6707 70.392322)
@@
   (gr_line (start 223.391232 73.653213) (end 223.417322 73.696583)
     (stroke (width 0.0508) (type solid)) (layer "B.SilkS"))
-  (gr_line (start 379.73 55.372) (end 378.968 54.61)
+  (gr_line (start 379.73 60.452) (end 378.968 59.69)
     (stroke (width 0.12) (type default)) (layer "B.SilkS"))
   (gr_line (start 207.517609 74.824833) (end 207.517609 74.172853)
@@
   (gr_line (start 219.44824 70.591787) (end 219.41054 70.628587)
     (stroke (width 0.0508) (type solid)) (layer "B.SilkS"))
-  (gr_line (start 378.968 54.61) (end 379.73 53.848)
+  (gr_line (start 378.968 59.69) (end 379.73 58.928)
     (stroke (width 0.12) (type default)) (layer "B.SilkS"))
   (gr_line (start 217.341881 73.460841) (end 217.629374 73.460841)
@@
   (gr_line (start 215.142759 66.950376) (end 215.166039 66.924456)
     (stroke (width 0.0508) (type solid)) (layer "F.SilkS"))
-  (gr_line (start 379.73 53.9496) (end 378.968 54.7116)
+  (gr_line (start 379.73 59.0296) (end 378.968 59.7916)
     (stroke (width 0.12) (type default)) (layer "F.SilkS"))
   (gr_line (start 227.146336 73.833083) (end 227.116486 73.807163)
@@
   (gr_line (start 221.101577 67.00665) (end 221.140857 67.03257)
     (stroke (width 0.0508) (type solid)) (layer "F.SilkS"))
-  (gr_line (start 378.968 54.7116) (end 379.73 55.4736)
+  (gr_line (start 378.968 59.7916) (end 379.73 60.5536)
     (stroke (width 0.12) (type default)) (layer "F.SilkS"))
   (gr_line (start 225.279061 70.540282) (end 227.162704 70.540282)
@@
   (gr_line (start 219.416138 75.401951) (end 219.376858 75.427881)
     (stroke (width 0.0508) (type solid)) (layer "F.SilkS"))
-  (gr_line (start 379.73 54.7116) (end 379.73 54.2036)
+  (gr_line (start 379.73 59.7916) (end 379.73 59.2836)
     (stroke (width 0.12) (type default)) (layer "F.SilkS"))
   (gr_line (start 217.76638 66.999878) (end 217.79943 67.024958)
@@
   (gr_line (start 214.241738 73.694887) (end 214.203978 73.703587)
     (stroke (width 0.0508) (type solid)) (layer "F.SilkS"))
-  (gr_line (start 379.73 55.4736) (end 379.73 54.7116)
+  (gr_line (start 379.73 60.5536) (end 379.73 59.7916)
     (stroke (width 0.12) (type default)) (layer "F.SilkS"))
   (gr_curve (pts (xy 203.870327 67.273577) (xy 203.870327 67.273577) (xy 203.887387 67.278077) (xy 203.852117 67.282577))
@@
   (gr_line (start 219.198468 75.338477) (end 219.165868 75.345277)
     (stroke (width 0.0508) (type solid)) (layer "F.SilkS"))
-  (gr_line (start 379.476 54.7116) (end 378.968 54.7116)
+  (gr_line (start 379.476 59.7916) (end 378.968 59.7916)
     (stroke (width 0.12) (type default)) (layer "F.SilkS"))
   (gr_line (start 205.03952 67.381858) (end 205.07801 67.353508)
@@
   (gr_line (start 213.463439 68.160965) (end 214.159398 68.157065)
     (stroke (width 0.0508) (type solid)) (layer "F.SilkS"))
-  (gr_line (start 383.286 54.7116) (end 379.476 54.7116)
+  (gr_line (start 383.286 59.7916) (end 379.476 59.7916)
     (stroke (width 0.12) (type default)) (layer "F.SilkS"))
   (gr_line (start 222.898472 70.201416) (end 222.892272 70.186196)
@@
   (gr_line (start 214.242382 68.359543) (end 214.281262 68.393133)
     (stroke (width 0.0508) (type solid)) (layer "F.SilkS"))
-  (gr_line (start 379.73 54.2036) (end 379.73 53.9496)
+  (gr_line (start 379.73 59.2836) (end 379.73 59.0296)
     (stroke (width 0.12) (type default)) (layer "F.SilkS"))
   (gr_line (start 218.56939 75.320391) (end 218.53326 75.249891)
@@
     (effects (font (size 1.5 1.5) (thickness 0.3) bold) (justify left bottom))
   )
-  (gr_text "A1" (at 235.458 63.6016) (layer "B.SilkS")
+  (gr_text "A1" (at 380.238 65.024) (layer "B.SilkS")
     (effects (font (size 2.032 1.524) (thickness 0.254)) (justify mirror))
   )
@@
     (effects (font (size 2.032 1.524) (thickness 0.254)) (justify mirror))
   )
-  (gr_text "A2" (at 316.865 63.627) (layer "B.SilkS")
+  (gr_text "A2" (at 295.402 65.278) (layer "B.SilkS")
     (effects (font (size 2.032 1.524) (thickness 0.254)) (justify mirror))
   )
@@
     (effects (font (size 2.032 1.524) (thickness 0.254)) (justify mirror))
   )
-  (gr_text "A1" (at 297.815 63.754) (layer "B.SilkS")
+  (gr_text "A1" (at 314.706 65.024) (layer "B.SilkS")
     (effects (font (size 2.032 1.524) (thickness 0.254)) (justify mirror))
   )
@@
     (effects (font (size 2 2) (thickness 0.4) bold) (justify left bottom mirror))
   )
-  (gr_text "Pin 1" (at 386.207 54.8894) (layer "B.SilkS")
+  (gr_text "Pin 1" (at 386.207 59.9694) (layer "B.SilkS")
     (effects (font (size 2.032 1.524) (thickness 0.254)) (justify mirror))
   )
@@
     (effects (font (size 5.08 4.064) (thickness 0.762)) (justify mirror))
   )
-  (gr_text "A2" (at 380.111 63.5) (layer "B.SilkS")
+  (gr_text "A2" (at 238.252 63.754) (layer "B.SilkS")
     (effects (font (size 2.032 1.524) (thickness 0.254)) (justify mirror))
   )
@@
     (effects (font (size 2.032 1.524) (thickness 0.254)))
   )
-  (gr_text "A1" (at 377.19 62.2046) (layer "F.SilkS")
+  (gr_text "A1" (at 380.492 65.024) (layer "F.SilkS")
     (effects (font (size 2.032 1.524) (thickness 0.254)))
   )
@@
     (effects (font (size 2.032 1.524) (thickness 0.254)))
   )
-  (gr_text "A1" (at 314.833 62.357) (layer "F.SilkS")
+  (gr_text "A1" (at 314.96 65.024) (layer "F.SilkS")
     (effects (font (size 2.032 1.524) (thickness 0.254)))
   )
@@
     (effects (font (size 5.08 4.064) (thickness 0.762)))
   )
-  (gr_text "Pin 1" (at 386.207 54.991) (layer "F.SilkS")
+  (gr_text "Pin 1" (at 386.207 60.071) (layer "F.SilkS")
     (effects (font (size 2.032 1.524) (thickness 0.254)))
   )

Commit message: mega-magic
Parts:
- moved X3 201.4 mm to (265.9, 58.5)
- moved X5 131.3 mm to (165.0, 58.3)
- moved X7 114.1 mm to (83.7, 58.3)
Routing:
- net c03: track 60.8 -> 65.3 mm
- net d49: track 71.4 -> 74.7 mm
- net d25: track 65.0 -> 68.4 mm
- net d47: track 70.8 -> 74.2 mm
- net d23: track 64.5 -> 67.8 mm
- net d27: track 65.6 -> 68.8 mm
- net d21: track 64.0 -> 67.2 mm
- net d37: track 68.2 -> 71.4 mm
- net d45: track 70.3 -> 73.4 mm
- net d43: track 69.8 -> 72.8 mm
- net d39: track 68.7 -> 71.8 mm
- net d15: track 62.4 -> 65.5 mm
- net d13: track 61.9 -> 65.0 mm
- net d19: track 63.5 -> 66.4 mm
- net d41: track 69.3 -> 72.2 mm
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