File: DG Nova Extender Board/Card-Edge Adapter.kicad_pcb (KiCad board)
At the start: 2 copper layers, 379 x 83.8 mm, 12 parts, among them J1 portAB, J2 portCD, X1 Slot 1 A1, X2 Slot 1 A2, X3 Slot 1 B1, X4 Slot 1 B2, X5 Slot 2 A1, X6 Slot 2 A2, X7 Slot 2 B1, X8 Slot 2 B2

Commit message: stuff
Parts:
- moved J1 341.4 mm to (379.1, 28.6), turned to 180 degrees
- moved X1 323.0 mm to (372.1, 92.7), turned to -90 degrees
- moved X2 319.2 mm to (372.1, 74.9), turned to -90 degrees
- moved X7 215.9 mm to (108.0, 92.7), turned to -90 degrees
- moved X8 210.2 mm to (108.0, 74.9), turned to -90 degrees
- moved X3 164.7 mm to (290.8, 92.7), turned to -90 degrees
- moved X4 157.1 mm to (290.8, 74.9), turned to -90 degrees
- moved J2 89.5 mm to (189.2, 28.6), turned to 180 degrees
- moved X5 70.1 mm to (189.2, 92.7), turned to -90 degrees
- moved X6 49.8 mm to (189.2, 74.9), turned to -90 degrees
Other:
- outline, holes or cut-outs redrawn
