File: DG Nova Extender Board/Backplane Socket Board.kicad_sch (KiCad schematic)
At the start: 6 parts, among them J1 portAB, J2 portCD, X1 Slot 1 A1, X3 Slot 1 B1, X5 Slot 2 A1, X7 Slot 2 B1

Commit message: More Magic
Parts:
- J1: value portAB -> Port A; footprint Forgotten Machines:DG NOVA Backplane Connector -> Forgotten Machines:DG NOVA Backplane Connector - Frontside
- J2: value portCD -> Port B; footprint Forgotten Machines:DG NOVA Backplane Connector -> Forgotten Machines:DG NOVA Backplane Connector - Frontside
- X1: value Slot 1 A1 -> A1
- X3: value Slot 1 B1 -> A2
- X5: value Slot 2 A1 -> B1
- X7: value Slot 2 B1 -> B2
Changed lines of the file:
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@@
       (effects (font (size 1.27 1.27)))
     )
-    (property "Value" "Slot 1 A1" (at 64.77 29.1846 0)
+    (property "Value" "A1" (at 64.77 29.1846 0)
       (effects (font (size 1.27 1.27) bold))
     )
@@
       (effects (font (size 1.27 1.27)))
     )
-    (property "Value" "Slot 1 B1" (at 120.65 29.1846 0)
+    (property "Value" "A2" (at 120.65 29.1846 0)
       (effects (font (size 1.27 1.27) bold))
     )
@@
       (effects (font (size 1.27 1.27)) (justify left))
     )
-    (property "Value" "portAB" (at 25.908 134.5184 90)
+    (property "Value" "Port A" (at 25.908 134.5184 90)
       (effects (font (size 1.016 1.016)) (justify left))
     )
-    (property "Footprint" "Forgotten Machines:DG NOVA Backplane Connector" (at 76.2 134.62 0)
+    (property "Footprint" "Forgotten Machines:DG NOVA Backplane Connector - Frontside" (at 76.2 134.62 0)
       (effects (font (size 1.27 1.27)) hide)
     )
@@
       (effects (font (size 1.27 1.27)) (justify left))
     )
-    (property "Value" "portCD" (at 191.008 134.5184 90)
+    (property "Value" "Port B" (at 191.008 134.5184 90)
       (effects (font (size 1.016 1.016)) (justify left))
     )
-    (property "Footprint" "Forgotten Machines:DG NOVA Backplane Connector" (at 241.3 134.62 0)
+    (property "Footprint" "Forgotten Machines:DG NOVA Backplane Connector - Frontside" (at 241.3 134.62 0)
       (effects (font (size 1.27 1.27)) hide)
     )
@@
       (effects (font (size 1.27 1.27)))
     )
-    (property "Value" "Slot 2 A1" (at 229.87 29.1846 0)
+    (property "Value" "B1" (at 229.87 29.1846 0)
       (effects (font (size 1.27 1.27) bold))
     )
@@
       (effects (font (size 1.27 1.27)))
     )
-    (property "Value" "Slot 2 B1" (at 285.75 29.1846 0)
+    (property "Value" "B2" (at 285.75 29.1846 0)
       (effects (font (size 1.27 1.27) bold))
     )

Commit message: swap connectors
Parts:
- X1, X3, X5, X7: footprint Connector_IDC:IDC-Header_2x25_P2.54mm_Vertical -> Forgotten Machines:IDC-Header_2x25_P2.54mm - Backside
Changed lines of the file:
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@@
       (effects (font (size 1.27 1.27) bold))
     )
-    (property "Footprint" "Connector_IDC:IDC-Header_2x25_P2.54mm_Vertical" (at 63.5 62.865 0)
+    (property "Footprint" "Forgotten Machines:IDC-Header_2x25_P2.54mm - Backside" (at 63.5 62.865 0)
       (effects (font (size 1.27 1.27)) hide)
     )
@@
       (effects (font (size 1.27 1.27) bold))
     )
-    (property "Footprint" "Connector_IDC:IDC-Header_2x25_P2.54mm_Vertical" (at 119.38 62.865 0)
+    (property "Footprint" "Forgotten Machines:IDC-Header_2x25_P2.54mm - Backside" (at 119.38 62.865 0)
       (effects (font (size 1.27 1.27)) hide)
     )
@@
       (effects (font (size 1.27 1.27) bold))
     )
-    (property "Footprint" "Connector_IDC:IDC-Header_2x25_P2.54mm_Vertical" (at 228.6 62.865 0)
+    (property "Footprint" "Forgotten Machines:IDC-Header_2x25_P2.54mm - Backside" (at 228.6 62.865 0)
       (effects (font (size 1.27 1.27)) hide)
     )
@@
       (effects (font (size 1.27 1.27) bold))
     )
-    (property "Footprint" "Connector_IDC:IDC-Header_2x25_P2.54mm_Vertical" (at 284.48 62.865 0)
-      (effects (font (size 1.27 1.27)) hide)
-    )
+    (property "Footprint" "Forgotten Machines:IDC-Header_2x25_P2.54mm - Backside" (at 284.48 62.865 0)
+      (effects (font (size 1.27 1.27)) hide)
+    )
