File: DG Nova Extender Board/Backplane Wire-Wrap Side Plug.kicad_pcb (KiCad board)
At the start: 2 copper layers, 379 x 76.2 mm, 3 parts, among them J1 Port A, X1 A1, X3 A2

Commit message: Updates
Parts:
- J1: moved to B.Cu
- moved X1 282.5 mm to (65.3, 39.7), turned to 180 degrees
- moved J1 203.1 mm to (109.0, 50.8), turned to 180 degrees
- moved X3 114.0 mm to (153.5, 39.9), turned to 180 degrees
Connections:
- J1 pad 1: a01 -> GND
- J1 pad 100: b50 -> GND
- J1 pad 2: a02 -> GND
- J1 pad 3: a03 -> +5V
- J1 pad 4: a04 -> +5V
- J1 pad 97: b47 -> +5V
- J1 pad 98: b48 -> +5V
- J1 pad 99: b49 -> GND
- X1 pad 1: a01 -> GND
- X1 pad 2: a02 -> GND
- X1 pad 3: a03 -> +5V
- X1 pad 4: a04 -> +5V
- X3 pad 47: b47 -> +5V
- X3 pad 48: b48 -> +5V
- X3 pad 49: b49 -> GND
- X3 pad 50: b50 -> GND
Routing:
- net +5V: track 0.00 -> 87.5 mm
- net GND: track 0.00 -> 72.3 mm
- net a50: track 0.00 -> 18.9 mm
- net a48: track 0.00 -> 18.8 mm
- net b02: track 0.00 -> 18.5 mm
- net b46: track 0.00 -> 17.9 mm
- net a32: track 0.00 -> 17.9 mm
- net a46: track 0.00 -> 17.6 mm
- net b04: track 0.00 -> 17.6 mm
- net a44: track 0.00 -> 17.4 mm
- net b44: track 0.00 -> 17.3 mm
- net a30: track 0.00 -> 17.3 mm
- net b06: track 0.00 -> 17.3 mm
- net a42: track 0.00 -> 17.1 mm
- net b42: track 0.00 -> 17.0 mm
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- added copper zone on B.Cu, net +5V
- added copper zone on F.Cu, net GND
Other:
- board size 379 x 76.2 mm -> 170.8 x 29.3 mm
- board text added: "100"
- board text added: "50"
- board text added: "Data General Nova / DCC D-116 Backplane Wire-Wrap-Side 2.54mm Adapter"
- board text added: "Pin 51"
- board text removed: "A"
- board text removed: "A1"
- board text removed: "A2"
- board text removed: "PLUG CABLES INTO THIS SIDE OF BOARD"
