File: DG_Nova_Front_Panel_Tester_09_1/DG_Nova_Front_Panel_Tester.kicad_sch (KiCad schematic)
At the start: 10 parts, among them J1 Slot_02x26, J2 Conn_01x04, J3 Conn_01x08, J4 Conn_01x08, J5 Conn_01x06, J6 Conn_01x04, J7 Conn_01x02, J8 Conn_01x19, SW1 SW_Push

Commit message: all
Parts:
- XA1: footprint Arduino:Arduino_Mega2560_Shield -> Forgotten Machines:Arduino_Mega2560_Shield
Changed lines of the file:
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@@
+    (stroke (width 0) (type default))
+  )
+  (wire (pts (xy 62.865 59.69) (xy 68.58 59.69))
     (stroke (width 0) (type default))
   )
@@
   )
   (wire (pts (xy 68.58 130.81) (xy 59.69 130.81))
+    (stroke (width 0) (type default))
+  )
+  (wire (pts (xy 62.865 41.91) (xy 68.58 41.91))
     (stroke (width 0) (type default))
   )
@@
     )
   )
-  (global_label "~{CON DATA}" (shape input) (at 68.58 41.91 180) (fields_autoplaced)
-    (effects (font (size 0.9906 0.9906)) (justify right))
-    (property "Intersheetrefs" "${INTERSHEET_REFS}" (at 59.7197 41.91 0)
+  (global_label "~{CON DATA}" (shape input) (at 62.865 41.91 180) (fields_autoplaced)
+    (effects (font (size 0.9906 0.9906)) (justify right))
+    (property "Intersheetrefs" "${INTERSHEET_REFS}" (at 54.0047 41.91 0)
       (effects (font (size 1.27 1.27)) (justify right) hide)
     )
@@
     )
   )
-  (global_label "~{FETCH}" (shape input) (at 139.7 140.97 0) (fields_autoplaced)
-    (effects (font (size 1.27 1.27)) (justify left))
-    (property "Intersheetrefs" "${INTERSHEET_REFS}" (at 147.7573 140.97 0)
+  (global_label "~{FETCH}" (shape input) (at 140.335 140.97 0) (fields_autoplaced)
+    (effects (font (size 1.27 1.27)) (justify left))
+    (property "Intersheetrefs" "${INTERSHEET_REFS}" (at 148.3923 140.97 0)
       (effects (font (size 1.27 1.27)) (justify left) hide)
     )
@@
     )
   )
-  (global_label "~{STOP}" (shape input) (at 68.58 59.69 180) (fields_autoplaced)
-    (effects (font (size 0.9906 0.9906)) (justify right))
-    (property "Intersheetrefs" "${INTERSHEET_REFS}" (at 63.0973 59.69 0)
+  (global_label "~{STOP}" (shape input) (at 62.865 59.69 180) (fields_autoplaced)
+    (effects (font (size 0.9906 0.9906)) (justify right))
+    (property "Intersheetrefs" "${INTERSHEET_REFS}" (at 57.3823 59.69 0)
       (effects (font (size 1.27 1.27)) (justify right) hide)
     )
@@
       (effects (font (size 1.524 1.524)))
     )
-    (property "Footprint" "Arduino:Arduino_Mega2560_Shield" (at 119.38 26.67 0)
+    (property "Footprint" "Forgotten Machines:Arduino_Mega2560_Shield" (at 119.38 26.67 0)
       (effects (font (size 1.524 1.524)) hide)
     )
