File: DG Nova CPU Tester/DG Nova CPU Tester.kicad_sch (KiCad schematic)
At the start: 18 parts, among them J11 Conn_01x16, J4 ATX-24, J6 Conn_01x16, J7 Conn_01x18, J8 Conn_01x16, J9 Conn_01x18, U1 Nova 1200 CPU

Commit message: all
Parts:
- removed U1: Nova 1200 CPU, symbol ForgottenMachines:DG_Nova_1200_CPU
- added C3, C4, C5: C, Capacitor_THT:C_Disc_D6.0mm_W2.5mm_P5.00mm, symbol Device:C
- added D1, D2, D3, D4, D5, D6: 1N4004, Diode_THT:D_DO-41_SOD81_P10.16mm_Horizontal, symbol Diode:1N4004
- added J1 (x2): Slot_02x50_Odd_Even, Forgotten Machines:DG NOVA Backplane Connector - Frontside, symbol NovaMem-rescue:Slot_02x50_Odd_Even-_local
- added J10: Conn_01x18, Connector_PinHeader_2.54mm:PinHeader_1x18_P2.54mm_Horizontal, symbol Connector_Generic:Conn_01x18
- added J12: Conn_01x08, Connector_PinHeader_2.54mm:PinHeader_1x08_P2.54mm_Horizontal, symbol Connector_Generic:Conn_01x08
- added J13, J14: Conn_01x04, Connector_PinHeader_2.54mm:PinHeader_1x04_P2.54mm_Horizontal, symbol Connector_Generic:Conn_01x04
- added JP4: Vipass Ammeter, Connector_PinHeader_2.54mm:PinHeader_1x02_P2.54mm_Vertical, symbol Jumper:Jumper_2_Open
- added R1, R6: 1k, Resistor_THT:R_Axial_DIN0207_L6.3mm_D2.5mm_P10.16mm_Horizontal, symbol Device:R
- added R2, R5: 10k, Resistor_THT:R_Axial_DIN0207_L6.3mm_D2.5mm_P10.16mm_Horizontal, symbol Device:R
- added R3, R4: 4.7k, Resistor_THT:R_Axial_DIN0207_L6.3mm_D2.5mm_P10.16mm_Horizontal, symbol Device:R
- added SW1: SW_Push, Button_Switch_THT:SW_PUSH_6mm, symbol Switch:SW_Push
- added U1: 74HC14, Package_DIP:DIP-14_W7.62mm, symbol 74xx:74HC14
- J?: value Slot_02x26 -> Front Panel Socket - Backside
- XA1: footprint Arduino:Arduino_Mega2560_Shield -> Forgotten Machines:Arduino_Mega2560_Shield
Connections:
- net +5V: now also D1.1 (K), D2.2 (A), D3.1 (K), D4.2 (A), D5.1 (K), D6.2 (A), J1.3 (Pin_3), J1.3 (Pin_3), J1.4 (Pin_4), J1.4 (Pin_4), J1.97 (Pin_69), J1.97 (Pin_69), J1.98 (Pin_98), J1.98 (Pin_98), U1.14 (VCC)
- net +5V OK: now also J14.3 (Pin_3), U1.12
- net CLR: now also J1.50 (Pin_50), J10.14 (Pin_14)
- net DATIA: now also J1.44 (Pin_44), J10.7 (Pin_7)
- net DATIB: now also J1.42 (Pin_42), J10.8 (Pin_8)
- net DATIC: now also J1.54 (Pin_54), J10.9 (Pin_9)
- net DATOA: now also J1.58 (Pin_58), J10.10 (Pin_10)
- net DATOB: now also J1.56 (Pin_56), J10.11 (Pin_11)
- net DATOC: now also J1.48 (Pin_48), J10.12 (Pin_12)
- net DCHI: now also J1.37 (Pin_37), J12.6 (Pin_6)
- net DCHO: now also J1.33 (Pin_33), J12.7 (Pin_7)
- net GND: now also C3.2, C4.2, C5.2, J1.1 (Pin_1), J1.1 (Pin_1), J1.100 (Pin_100), J1.100 (Pin_100), J1.2 (Pin_2), J1.2 (Pin_2), J1.33 (Pin_33), J1.34 (Pin_34), J1.50 (Pin_50), J1.89 (Pin_89), J1.92 (Pin_92), J1.99 (Pin_99), J1.99 (Pin_99), JP4.2 (B), SW1.1, U1.7 (GND)
- net GND After Meter: now also JP4.1 (A)
- net INHIBIT: now also J1.30 (Pin_30)
- net INTA: now also J1.40 (Pin_40), J13.4 (Pin_4)
- net IO PLS: now also J1.74 (Pin_74), J10.15 (Pin_15)
- net IO RST: now also J1.70 (Pin_70), J14.1 (Pin_1)
- net MB LOAD: now also J1.74 (Pin_74)
- net MEM OK: now also XA1.D52, U1.10
- net OVFLO: now also J1.39 (Pin_39), J12.8 (Pin_8)
- net RESTART ENABLE: now also XA1.A7
- net STROBE: now also J1.20 (Pin_20)
- net STRT: now also J1.52 (Pin_52), J10.13 (Pin_13)
- net ~{CARRY}: now also XA1.D32
- net ~{CON DATA}: now also XA1.D0 (D0_RX0)
- net ~{CON INST}: now also XA1.A4
- net ~{CON RQ}: now also XA1.A5
- net ~{CONT+ISTP+MSTP}: now also XA1.D1 (D1_TX0)
- net ~{DATA0}: now also J1.62 (Pin_62)
- net ~{DATA10}: now also J1.75 (Pin_75)
- net ~{DATA11}: now also J1.58 (Pin_58)
- net ~{DATA12}: now also J1.59 (Pin_59)
- net ~{DATA13}: now also J1.64 (Pin_64)
- net ~{DATA14}: now also J1.56 (Pin_56)
- net ~{DATA15}: now also J1.66 (Pin_66)
- net ~{DATA1}: now also J1.65 (Pin_65)
- net ~{DATA2}: now also J1.82 (Pin_82)
- net ~{DATA3}: now also J1.73 (Pin_73)
- net ~{DATA4}: now also J1.61 (Pin_61)
- net ~{DATA5}: now also J1.57 (Pin_57)
- net ~{DATA6}: now also J1.95 (Pin_95)
- net ~{DATA7}: now also J1.55 (Pin_55)
- net ~{DATA8}: now also J1.60 (Pin_60)
- net ~{DATA9}: now also J1.63 (Pin_63)
- net ~{DCHA}: now also J1.60 (Pin_60), J12.3 (Pin_3)
- net ~{DCHM0}: now also J1.17 (Pin_17), J12.4 (Pin_4)
- net ~{DCHM1}: now also J1.21 (Pin_21), J12.5 (Pin_5)
- net ~{DCHR}: now also J1.35 (Pin_35), J12.1 (Pin_1)
- net ~{DEFER}: now also XA1.D50
- net ~{DRIVE IO}: now also J1.88 (Pin_88)
- net ~{DS0}: now also J1.72 (Pin_72), J10.1 (Pin_1)
- net ~{DS1}: now also J1.68 (Pin_68), J10.2 (Pin_2)
- net ~{DS2}: now also J1.66 (Pin_66), J10.3 (Pin_3)
- net ~{DS3}: now also J1.46 (Pin_46), J10.4 (Pin_4)
- net ~{DS4}: now also J1.62 (Pin_62), J10.5 (Pin_5)
- net ~{DS5}: now also J1.64 (Pin_64), J10.6 (Pin_6)
- net ~{EXEC}: now also XA1.D51
- net ~{FETCH}: now also XA1.D49
- net ~{INH TRANS}: now also J1.45 (Pin_45)
- net ~{INTR}: now also J1.29 (Pin_29), J13.1 (Pin_1)
- net ~{ION}: now also XA1.D31
- net ~{ISTP}: now also XA1.A2
- net ~{MA LOAD}: now also J1.7 (Pin_7)
- net ~{MB CLEAR}: now also J1.86 (Pin_86)
- net ~{MBO0}: now also J1.79 (Pin_79)
- net ~{MBO10}: now also XA1.D24, J1.8 (Pin_8)
- net ~{MBO11}: now also XA1.D25, J1.5 (Pin_5)
- net ~{MBO12}: now also XA1.D26, J1.39 (Pin_39)
- net ~{MBO13}: now also XA1.D27, J1.37 (Pin_37)
- net ~{MBO14}: now also XA1.D28, J1.43 (Pin_43)
- net ~{MBO15}: now also XA1.D29, J1.41 (Pin_41)
- net ~{MBO1}: now also XA1.D15 (D15_RX3), J1.77 (Pin_77)
- net ~{MBO2}: now also XA1.D16 (D16_TX2), J1.44 (Pin_44)
- net ~{MBO3}: now also XA1.D17 (D17_RX2), J1.43 (Pin_43)
- net ~{MBO4}: now also XA1.D18 (D18_TX1), J1.42 (Pin_42)
- net ~{MBO5}: now also XA1.D19 (D19_RX1), J1.32 (Pin_32)
- net ~{MBO6}: now also XA1.D20 (D20_SDA), J1.16 (Pin_16)
- net ~{MBO7}: now also XA1.D21 (D21_SCL), J1.14 (Pin_14)
- net ~{MBO8}: now also XA1.D22, J1.12 (Pin_12)
- net ~{MBO9}: now also XA1.D23, J1.9 (Pin_9)
- net ~{MEM0}: now also XA1.D33, J1.71 (Pin_71)
- net ~{MEM10}: now also XA1.D43, J1.45 (Pin_45)
- net ~{MEM11}: now also XA1.D44, J1.51 (Pin_51)
- net ~{MEM12}: now also XA1.D45, J1.36 (Pin_36)
- net ~{MEM13}: now also XA1.D46, J1.35 (Pin_35)
- net ~{MEM14}: now also XA1.D47, J1.76 (Pin_76)
- net ~{MEM15}: now also XA1.D48, J1.18 (Pin_18)
- net ~{MEM1}: now also XA1.D34, J1.70 (Pin_70)
- net ~{MEM2}: now also XA1.D35, J1.47 (Pin_47)
- net ~{MEM3}: now also XA1.D36, J1.68 (Pin_68)
- net ~{MEM4}: now also XA1.D37, J1.28 (Pin_28)
- net ~{MEM5}: now also XA1.D38, J1.26 (Pin_26)
- net ~{MEM6}: now also XA1.D39, J1.22 (Pin_22)
- net ~{MEM7}: now also XA1.D40, J1.24 (Pin_24)
- net ~{MEM8}: now also XA1.D41, J1.55 (Pin_55)
- net ~{MEM9}: now also XA1.D42, J1.53 (Pin_53)
- net ~{MSKO}: now also J1.38 (Pin_38), J13.2 (Pin_2)
- net ~{PL}: now also XA1.A3
- net ~{POWER FAIL}: now also J14.4 (Pin_4), U1.8
- net ~{READ IO}: now also J1.83 (Pin_83)
- net ~{READ1}: now also J1.87 (Pin_87)
- net ~{READ2}: now also J1.90 (Pin_90)
- net ~{RQENB}: now also J1.41 (Pin_41), J14.2 (Pin_2)
- net ~{RST}: now also XA1.A6
- net ~{RUN}: now also XA1.D30
- net ~{SELB}: now also J1.82 (Pin_82), J10.16 (Pin_16)
- net ~{SELD}: now also J1.80 (Pin_80), J10.17 (Pin_17)
- net ~{STOP}: now also XA1.D14 (D14_TX3)
- net at XA1.RST1 (RESET): now also SW1.2
- new net: C5.1, R5.2, R6.1, U1.1
- new net: U1.13, U1.2
- new net: D4.1 (K), R4.2
- new net: C4.1, R3.2, R4.1, U1.3
- new net: U1.11, U1.4
- new net: D5.2 (A), R5.1
- new net: C3.1, R1.2, R2.1, U1.5
- new net: U1.6, U1.9
- new net: D1.2 (A), R1.1
- new net: D6.1 (K), R6.2
- new net: D2.1 (K), R2.2
- new net: D3.2 (A), R3.1
- new net +V MEM: J1.46 (Pin_46)
- new net +VINH: J1.10 (Pin_10), J1.84 (Pin_84)
- new net -5V: J1.6 (Pin_6), J1.81 (Pin_81)
- new net 60Hz: J1.6 (Pin_6)
- new net INH GND: J1.14 (Pin_14), J1.16 (Pin_16), J1.20 (Pin_20), J1.22 (Pin_22), J1.26 (Pin_26), J1.30 (Pin_30), J1.31 (Pin_31), J1.8 (Pin_8)
- new net RINH0: J1.5 (Pin_5)
- new net RINH1: J1.7 (Pin_7)
- new net RINH10: J1.23 (Pin_23)
- new net RINH11: J1.21 (Pin_21)
- new net RINH12: J1.28 (Pin_28)
- new net RINH13: J1.25 (Pin_25)
- new net RINH14: J1.29 (Pin_29)
- new net RINH15: J1.27 (Pin_27)
- new net RINH2: J1.9 (Pin_9)
- new net RINH3: J1.11 (Pin_11)
- new net RINH4: J1.13 (Pin_13)
- new net RINH5: J1.15 (Pin_15)
- new net RINH6: J1.18 (Pin_18)
- new net RINH7: J1.17 (Pin_17)
- new net RINH8: J1.19 (Pin_19)
- new net RINH9: J1.24 (Pin_24)
- new net ROS: J1.78 (Pin_78)
- new net ~{BMA LOAD}: J1.10 (Pin_10)
- new net ~{DCHP IN}: J1.94 (Pin_94)
- new net ~{DCHP OUT}: J1.93 (Pin_93)
- new net ~{EXT SELECT}: J1.80 (Pin_80)
- new net ~{INHIBIT SELECT}: J1.85 (Pin_85)
- new net ~{INTP IN}: J1.96 (Pin_96)
- new net ~{INTP OUT}: J1.95 (Pin_95)
- new net ~{RELOAD DISABLE}: J1.72 (Pin_72)
- no-connect marks 62 -> 115
Other:
- note added: "DCHP"
- note added: "Data Channel"
- note added: "INTP"
- note added: "PWR ON"
- note added: "Program Interrupt"
- note added: "SLOT 3456789101112 4K MEM or IO"
- note added: "Slot 3 only?"
- note added: "Start-Up Power Manager"
- note added: "System Control"
- note removed: "Data Channel DCHR DCHP DCHA DCHM0 DCHM1 DCHI DCHO OVFLO"
- note removed: "Program Interrupt INTR MSKO INTP INTA"
- note removed: "Programmed I/O DS0-DS5 DATIA DATIB DATIC DATOA DATOB DATOC STRT CLR IOPLS SELB SELD"
- note removed: "System Control IORST PWR ON RQENB"
- moved on the sheet: J11, J6, J7, J9, XA1

Commit message: changes
Parts:
- added U2: Pico, Forgotten Machines:RPi_Pico_SMD_TH, symbol ForgottenMachines:Raspberry_Pi_Pico
Other:
- moved on the sheet: SW1, XA1

Commit message: work
Parts:
- J1: footprint Forgotten Machines:DG NOVA Backplane Connector - Frontside -> Forgotten Machines:DG NOVA Backplane Connector - Backside
Connections:
- net +5V: now also U2.39 (VSYS), XA1.5V1 (5V), XA1.5V3 (5V), XA1.5V4 (5V)
- net GND: now also U2.13 (GND), U2.18 (GND), U2.23 (GND), U2.28 (GND), U2.3 (GND), U2.33 (AGND), U2.38 (GND), U2.42 (GND), U2.8 (GND)
- net +3v3: now reaches J4.1 (+3.3V), J4.12 (+3.3V), J4.13 (+3.3V), J4.2 (+3.3V)
- net UART_TX: now reaches U2.1 (GPIO0)
- net UART_RX: now reaches U2.2 (GPIO1)
- no-connect marks 115 -> 114
Other:
- moved on the sheet: C3, C4, C5, D1, D2, D3, D4, D5, D6, J1, R1, R2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

Commit message: yes
Parts:
- added J17: Conn_01x10, Connector_PinHeader_2.54mm:PinHeader_1x10_P2.54mm_Horizontal, symbol Connector_Generic:Conn_01x10
- added TP1: TestPoint, Connector_PinHeader_2.54mm:PinHeader_1x01_P2.54mm_Vertical, symbol Connector:TestPoint
Connections:
- net Entrex Backplane S01B53 to S13B53: now also TP1.1
- net ~{DIV}: now also J17.4 (Pin_4)
- net ~{EXT LOAD}: now also J17.2 (Pin_2)
- net ~{FORCE LOAD IR}: now also J17.3 (Pin_3)
- net ~{SHIFT0}: now also J17.6 (Pin_6)
- net ~{SHIFT1}: now also J17.7 (Pin_7)
- net ~{SHIFT2}: now also J17.8 (Pin_8)
- net ~{SHIFT3}: now also J17.9 (Pin_9)
- net ~{TEST}: now also J17.5 (Pin_5)
- net ~{WHOA}: now also J17.1 (Pin_1)
Other:
- note added: "Orphaned Inputs"
- note removed: "Orphaned Inputs WHOA EXT LOAD FORCE LOAD IR DIV TEST"
- moved on the sheet: J10, J11, J12, J13, J14, J4, J6, J7, J8, JP1, JP4, MES1

Commit message: arrange
Connections:
- net INHIBIT: now also J11.7 (Pin_7); no longer J11.3 (Pin_3)
- net LOAD IR: now also J11.13 (Pin_13); no longer J11.12 (Pin_12)
- net MB LOAD: now also J11.10 (Pin_10); no longer J11.11 (Pin_11)
- net STROBE: now also J11.6 (Pin_6); no longer J11.2 (Pin_2)
- net ~{DIV}: now also J17.2 (Pin_2); no longer J17.4 (Pin_4)
- net ~{DRIVE IO}: now also J11.2 (Pin_2); no longer J11.8 (Pin_8)
- net ~{EXT LOAD}: now also J17.4 (Pin_4); no longer J17.2 (Pin_2)
- net ~{INH TRANS}: now also J11.8 (Pin_8); no longer J11.4 (Pin_4)
- net ~{LOAD AC}: now also J11.12 (Pin_12); no longer J11.13 (Pin_13)
- net ~{MB CLEAR}: now also J11.11 (Pin_11); no longer J11.10 (Pin_10)
- net ~{READ IO}: now also J11.3 (Pin_3); no longer J11.7 (Pin_7)
- net ~{READ1}: now also J11.4 (Pin_4); no longer J11.5 (Pin_5)
- net ~{READ2}: now also J11.5 (Pin_5); no longer J11.6 (Pin_6)
- net ~{SHIFT0}: now also J17.7 (Pin_7); no longer J17.6 (Pin_6)
- net ~{SHIFT1}: now also J17.8 (Pin_8); no longer J17.7 (Pin_7)
- net ~{SHIFT2}: now also J17.9 (Pin_9); no longer J17.8 (Pin_8)
- net ~{SHIFT3}: now also J17.10 (Pin_10); no longer J17.9 (Pin_9)
Changed lines of the file:
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@@
     )
   )
-  (global_label "~{LOAD AC}" (shape input) (at 294.64 59.055 0) (fields_autoplaced)
+  (global_label "~{LOAD AC}" (shape input) (at 294.64 56.515 0) (fields_autoplaced)
     (effects (font (size 1.27 1.27)) (justify left))
-    (property "Intersheetrefs" "${INTERSHEET_REFS}" (at 304.7294 59.055 0)
+    (property "Intersheetrefs" "${INTERSHEET_REFS}" (at 304.7294 56.515 0)
       (effects (font (size 1.27 1.27)) (justify left) hide)
     )
@@
     )
   )
-  (global_label "~{DRIVE IO}" (shape input) (at 294.64 46.355 0) (fields_autoplaced)
+  (global_label "~{DRIVE IO}" (shape input) (at 294.64 31.115 0) (fields_autoplaced)
     (effects (font (size 1.27 1.27)) (justify left))
-    (property "Intersheetrefs" "${INTERSHEET_REFS}" (at 304.9713 46.355 0)
+    (property "Intersheetrefs" "${INTERSHEET_REFS}" (at 304.9713 31.115 0)
       (effects (font (size 1.27 1.27)) (justify left) hide)
     )
@@
     )
   )
-  (global_label "~{SHIFT1}" (shape input) (at 267.335 41.91 180) (fields_autoplaced)
+  (global_label "~{SHIFT1}" (shape input) (at 267.335 44.45 180) (fields_autoplaced)
     (effects (font (size 1.27 1.27)) (justify right))
-    (property "Intersheetrefs" "${INTERSHEET_REFS}" (at 258.6729 41.91 0)
+    (property "Intersheetrefs" "${INTERSHEET_REFS}" (at 258.6729 44.45 0)
       (effects (font (size 1.27 1.27)) (justify right) hide)
     )
@@
     )
   )
-  (global_label "STROBE" (shape input) (at 294.64 31.115 0) (fields_autoplaced)
+  (global_label "STROBE" (shape input) (at 294.64 41.275 0) (fields_autoplaced)
     (effects (font (size 1.27 1.27)) (justify left))
-    (property "Intersheetrefs" "${INTERSHEET_REFS}" (at 304.0882 31.115 0)
+    (property "Intersheetrefs" "${INTERSHEET_REFS}" (at 304.0882 41.275 0)
       (effects (font (size 1.27 1.27)) (justify left) hide)
     )
@@
     )
   )
-  (global_label "MB LOAD" (shape input) (at 294.64 53.975 0) (fields_autoplaced)
+  (global_label "MB LOAD" (shape input) (at 294.64 51.435 0) (fields_autoplaced)
     (effects (font (size 1.27 1.27)) (justify left))
-    (property "Intersheetrefs" "${INTERSHEET_REFS}" (at 305.0922 53.975 0)
+    (property "Intersheetrefs" "${INTERSHEET_REFS}" (at 305.0922 51.435 0)
       (effects (font (size 1.27 1.27)) (justify left) hide)
     )
@@
     )
   )
-  (global_label "~{READ IO}" (shape input) (at 294.64 43.815 0) (fields_autoplaced)
+  (global_label "~{READ IO}" (shape input) (at 294.64 33.655 0) (fields_autoplaced)
     (effects (font (size 1.27 1.27)) (justify left))
-    (property "Intersheetrefs" "${INTERSHEET_REFS}" (at 304.3665 43.815 0)
+    (property "Intersheetrefs" "${INTERSHEET_REFS}" (at 304.3665 33.655 0)
       (effects (font (size 1.27 1.27)) (justify left) hide)
     )
@@
     )
   )
-  (global_label "LOAD IR" (shape input) (at 294.64 56.515 0) (fields_autoplaced)
+  (global_label "LOAD IR" (shape input) (at 294.64 59.055 0) (fields_autoplaced)
     (effects (font (size 1.27 1.27)) (justify left))
-    (property "Intersheetrefs" "${INTERSHEET_REFS}" (at 304.2456 56.515 0)
+    (property "Intersheetrefs" "${INTERSHEET_REFS}" (at 304.2456 59.055 0)
       (effects (font (size 1.27 1.27)) (justify left) hide)
     )
@@
     )
   )
-  (global_label "~{SHIFT0}" (shape input) (at 267.335 39.37 180) (fields_autoplaced)
+  (global_label "~{SHIFT0}" (shape input) (at 267.335 41.91 180) (fields_autoplaced)
     (effects (font (size 1.27 1.27)) (justify right))
-    (property "Intersheetrefs" "${INTERSHEET_REFS}" (at 258.6729 39.37 0)
+    (property "Intersheetrefs" "${INTERSHEET_REFS}" (at 258.6729 41.91 0)
       (effects (font (size 1.27 1.27)) (justify right) hide)
     )
@@
     )
   )
-  (global_label "~{READ1}" (shape input) (at 294.64 38.735 0) (fields_autoplaced)
+  (global_label "~{READ1}" (shape input) (at 294.64 36.195 0) (fields_autoplaced)
     (effects (font (size 1.27 1.27)) (justify left))
-    (property "Intersheetrefs" "${INTERSHEET_REFS}" (at 302.8787 38.735 0)
+    (property "Intersheetrefs" "${INTERSHEET_REFS}" (at 302.8787 36.195 0)
       (effects (font (size 1.27 1.27)) (justify left) hide)
     )
@@
     )
   )
-  (global_label "~{EXT LOAD}" (shape input) (at 267.335 29.21 180) (fields_autoplaced)
+  (global_label "~{EXT LOAD}" (shape input) (at 267.335 34.29 180) (fields_autoplaced)
     (effects (font (size 1.27 1.27)) (justify right))
-    (property "Intersheetrefs" "${INTERSHEET_REFS}" (at 256.2781 29.21 0)
+    (property "Intersheetrefs" "${INTERSHEET_REFS}" (at 256.2781 34.29 0)
       (effects (font (size 1.27 1.27)) (justify right) hide)
     )
@@
     )
   )
-  (global_label "~{SHIFT2}" (shape input) (at 267.335 44.45 180) (fields_autoplaced)
+  (global_label "~{SHIFT2}" (shape input) (at 267.335 46.99 180) (fields_autoplaced)
     (effects (font (size 1.27 1.27)) (justify right))
-    (property "Intersheetrefs" "${INTERSHEET_REFS}" (at 258.6729 44.45 0)
+    (property "Intersheetrefs" "${INTERSHEET_REFS}" (at 258.6729 46.99 0)
       (effects (font (size 1.27 1.27)) (justify right) hide)
     )
@@
     )
   )
-  (global_label "~{DIV}" (shape input) (at 267.335 34.29 180) (fields_autoplaced)
+  (global_label "~{DIV}" (shape input) (at 267.335 29.21 180) (fields_autoplaced)
     (effects (font (size 1.27 1.27)) (justify right))
-    (property "Intersheetrefs" "${INTERSHEET_REFS}" (at 262.12 34.29 0)
+    (property "Intersheetrefs" "${INTERSHEET_REFS}" (at 262.12 29.21 0)
       (effects (font (size 1.27 1.27)) (justify right) hide)
     )
@@
     )
   )
-  (global_label "~{SHIFT3}" (shape input) (at 267.335 46.99 180) (fields_autoplaced)
+  (global_label "~{SHIFT3}" (shape input) (at 267.335 49.53 180) (fields_autoplaced)
     (effects (font (size 1.27 1.27)) (justify right))
-    (property "Intersheetrefs" "${INTERSHEET_REFS}" (at 258.6729 46.99 0)
+    (property "Intersheetrefs" "${INTERSHEET_REFS}" (at 258.6729 49.53 0)
       (effects (font (size 1.27 1.27)) (justify right) hide)
     )
@@
     )
   )
-  (global_label "~{READ2}" (shape input) (at 294.64 41.275 0) (fields_autoplaced)
+  (global_label "~{READ2}" (shape input) (at 294.64 38.735 0) (fields_autoplaced)
     (effects (font (size 1.27 1.27)) (justify left))
-    (property "Intersheetrefs" "${INTERSHEET_REFS}" (at 302.8787 41.275 0)
+    (property "Intersheetrefs" "${INTERSHEET_REFS}" (at 302.8787 38.735 0)
       (effects (font (size 1.27 1.27)) (justify left) hide)
     )
@@
     )
   )
-  (global_label "~{MB CLEAR}" (shape input) (at 294.64 51.435 0) (fields_autoplaced)
+  (global_label "~{MB CLEAR}" (shape input) (at 294.64 53.975 0) (fields_autoplaced)
     (effects (font (size 1.27 1.27)) (justify left))
-    (property "Intersheetrefs" "${INTERSHEET_REFS}" (at 306.1807 51.435 0)
+    (property "Intersheetrefs" "${INTERSHEET_REFS}" (at 306.1807 53.975 0)
       (effects (font (size 1.27 1.27)) (justify left) hide)
     )
@@
     )
   )
-  (global_label "~{INH TRANS}" (shape input) (at 294.64 36.195 0) (fields_autoplaced)
+  (global_label "~{INH TRANS}" (shape input) (at 294.64 46.355 0) (fields_autoplaced)
     (effects (font (size 1.27 1.27)) (justify left))
-    (property "Intersheetrefs" "${INTERSHEET_REFS}" (at 306.7856 36.195 0)
+    (property "Intersheetrefs" "${INTERSHEET_REFS}" (at 306.7856 46.355 0)
       (effects (font (size 1.27 1.27)) (justify left) hide)
     )
@@
     )
   )
-  (global_label "INHIBIT" (shape input) (at 294.64 33.655 0) (fields_autoplaced)
+  (global_label "INHIBIT" (shape input) (at 294.64 43.815 0) (fields_autoplaced)
     (effects (font (size 1.27 1.27)) (justify left))
-    (property "Intersheetrefs" "${INTERSHEET_REFS}" (at 303.6046 33.655 0)
+    (property "Intersheetrefs" "${INTERSHEET_REFS}" (at 303.6046 43.815 0)
       (effects (font (size 1.27 1.27)) (justify left) hide)
     )

Commit message: board
Parts:
- removed J11: Conn_01x16, Connector_PinHeader_2.54mm:PinHeader_1x16_P2.54mm_Horizontal, symbol Connector_Generic:Conn_01x16
- removed J17: Conn_01x10, Connector_PinHeader_2.54mm:PinHeader_1x10_P2.54mm_Horizontal, symbol Connector_Generic:Conn_01x10
- added J11: Conn_01x10, Connector_PinHeader_2.54mm:PinHeader_1x10_P2.54mm_Horizontal, symbol Connector_Generic:Conn_01x10
- added J17: Conn_01x16, Connector_PinHeader_2.54mm:PinHeader_1x16_P2.54mm_Horizontal, symbol Connector_Generic:Conn_01x16
Connections:
- net CLK FLOP: now also J17.1 (Pin_1)
- net LOAD IR: now also J17.13 (Pin_13)
- net ~{DIV}: now also J11.2 (Pin_2)
- net ~{EXT LOAD}: now also J11.4 (Pin_4)
- net ~{FORCE LOAD IR}: now also J11.3 (Pin_3)
- net ~{LOAD AC}: now also J17.12 (Pin_12)
- net ~{MD SEL1}: now also J17.14 (Pin_14)
- net ~{SHIFT0}: now also J11.7 (Pin_7)
- net ~{SHIFT1}: now also J11.8 (Pin_8)
- net ~{SHIFT2}: now also J11.9 (Pin_9)
- net ~{SHIFT3}: now also J11.10 (Pin_10)
- net ~{TEST}: now also J11.5 (Pin_5)
- net ~{WAS JSR}: now also J17.15 (Pin_15)
- net ~{WHOA}: now also J11.1 (Pin_1)
Other:
- note added: "CPU Option Inputs"
- note added: "CPU Option Outputs"
- note added: "MEM Control Outputs"
- note removed: "Orphaned Inputs"
- note removed: "Orphaned Outputs"
- moved on the sheet: J9

Commit message: footprint
Parts:
- MES1: footprint Forgotten Machines:XK-001_Volt-Amp_Meter -> Forgotten Machines:XK-001_Volt-Amp_Meter - Backside
Changed lines of the file:
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@@
       (effects (font (size 1.27 1.27)) (justify right))
     )
-    (property "Footprint" "Forgotten Machines:XK-001_Volt-Amp_Meter" (at 347.98 86.36 0)
+    (property "Footprint" "Forgotten Machines:XK-001_Volt-Amp_Meter - Backside" (at 347.98 86.36 0)
       (effects (font (size 1.27 1.27)) hide)
     )
