File: DG Nova CPU Tester/DG Nova CPU Tester.kicad_sch (KiCad schematic)
At the start: 44 parts, among them J1 Slot_02x50_Odd_Even, J10 Conn_01x18, J11 Conn_01x10, J12 Conn_01x08, J13 Conn_01x04, J14 Conn_01x04, J17 Conn_01x16, J4 ATX-24, J6 Conn_01x16, J7 Conn_01x18, J8 Conn_01x16, J9 Conn_01x18, SW1 SW_Push, U1 74HC14, U2 Pico

Commit message: update
Parts:
- added J18: MEM Control Outputs, Connector_PinHeader_2.54mm:PinHeader_1x10_P2.54mm_Horizontal, symbol Connector_Generic:Conn_01x10
- J10: value Conn_01x18 -> Programmed I/O
- J11: value Conn_01x10 -> CPU Option Inputs
- J12: value Conn_01x08 -> Data Channel
- J13: value Conn_01x04 -> Program Interrupt
- J14: value Conn_01x04 -> System Control
- J17: value Conn_01x16 -> CPU Option Outputs; symbol Connector_Generic:Conn_01x16 -> Connector_Generic:Conn_01x06
- J6: value Conn_01x16 -> MBO
- J7: value Conn_01x18 -> MEM
- J8: value Conn_01x16 -> Data Channel
- J9: value Conn_01x18 -> Front Panel Controls
- TP1: value TestPoint -> Entrex Backplane S01B53 to S13B53
Connections:
- net INHIBIT: now also J18.9 (Pin_9)
- net LOAD IR: now also J17.3 (Pin_3); no longer J17.13 (Pin_13)
- net MB LOAD: now also J18.6 (Pin_6)
- net STROBE: now also J18.8 (Pin_8)
- net ~{DRIVE IO}: now also J18.1 (Pin_1)
- net ~{INH TRANS}: now also J18.10 (Pin_10)
- net ~{LOAD AC}: now also J17.2 (Pin_2); no longer J17.12 (Pin_12)
- net ~{MA LOAD}: now also J18.5 (Pin_5)
- net ~{MB CLEAR}: now also J18.7 (Pin_7)
- net ~{MD SEL1}: now also J17.4 (Pin_4); no longer J17.14 (Pin_14)
- net ~{READ IO}: now also J18.2 (Pin_2)
- net ~{READ1}: now also J18.3 (Pin_3)
- net ~{READ2}: now also J18.4 (Pin_4)
- net ~{WAS JSR}: now also J17.5 (Pin_5); no longer J17.15 (Pin_15)
Other:
- note added: "MEM / MBO"
Changed lines of the file:
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@@
     (fill (type none))
   )
-  (rectangle (start 279.4 19.05) (end 309.88 73.025)
+  (rectangle (start 279.4 19.05) (end 309.88 48.26)
     (stroke (width 0) (type default))
     (fill (type none))
@@
     (effects (font (size 1.27 1.27)) (justify left bottom))
   )
+  (text "MEM / MBO" (at 212.725 21.59 0)
+    (effects (font (size 1.27 1.27)) (justify left bottom))
+  )
   (text "B" (at 274.955 298.45 0)
     (effects (font (size 1.27 1.27)) (justify right bottom))
@@
     )
   )
-  (global_label "MB LOAD" (shape input) (at 323.85 48.26 0) (fields_autoplaced)
+  (global_label "MB LOAD" (shape input) (at 323.85 40.64 0) (fields_autoplaced)
     (effects (font (size 1.27 1.27)) (justify left))
-    (property "Intersheetrefs" "${INTERSHEET_REFS}" (at 334.3022 48.26 0)
+    (property "Intersheetrefs" "${INTERSHEET_REFS}" (at 334.3022 40.64 0)
       (effects (font (size 1.27 1.27)) (justify left) hide)
     )
@@
     )
   )
-  (global_label "INHIBIT" (shape input) (at 323.85 40.64 0) (fields_autoplaced)
+  (global_label "INHIBIT" (shape input) (at 323.85 48.26 0) (fields_autoplaced)
     (effects (font (size 1.27 1.27)) (justify left))
-    (property "Intersheetrefs" "${INTERSHEET_REFS}" (at 332.8146 40.64 0)
+    (property "Intersheetrefs" "${INTERSHEET_REFS}" (at 332.8146 48.26 0)
       (effects (font (size 1.27 1.27)) (justify left) hide)
     )
@@
     )
   )
-  (global_label "~{MD SEL1}" (shape input) (at 290.83 62.23 0) (fields_autoplaced)
+  (global_label "~{MD SEL1}" (shape input) (at 290.83 36.83 0) (fields_autoplaced)
     (effects (font (size 1.27 1.27)) (justify left))
-    (property "Intersheetrefs" "${INTERSHEET_REFS}" (at 301.1611 62.23 0)
+    (property "Intersheetrefs" "${INTERSHEET_REFS}" (at 301.1611 36.83 0)
       (effects (font (size 1.27 1.27)) (justify left) hide)
     )
@@
     )
   )
-  (global_label "STROBE" (shape input) (at 323.85 38.1 0) (fields_autoplaced)
+  (global_label "STROBE" (shape input) (at 323.85 45.72 0) (fields_autoplaced)
     (effects (font (size 1.27 1.27)) (justify left))
-    (property "Intersheetrefs" "${INTERSHEET_REFS}" (at 333.2982 38.1 0)
+    (property "Intersheetrefs" "${INTERSHEET_REFS}" (at 333.2982 45.72 0)
       (effects (font (size 1.27 1.27)) (justify left) hide)
     )
@@
     )
   )
-  (global_label "~{WAS JSR}" (shape input) (at 290.83 64.77 0) (fields_autoplaced)
+  (global_label "~{WAS JSR}" (shape input) (at 290.83 39.37 0) (fields_autoplaced)
     (effects (font (size 1.27 1.27)) (justify left))
-    (property "Intersheetrefs" "${INTERSHEET_REFS}" (at 301.0402 64.77 0)
+    (property "Intersheetrefs" "${INTERSHEET_REFS}" (at 301.0402 39.37 0)
       (effects (font (size 1.27 1.27)) (justify left) hide)
     )
@@
     )
   )
-  (global_label "~{MB CLEAR}" (shape input) (at 323.85 50.8 0) (fields_autoplaced)
+  (global_label "~{MB CLEAR}" (shape input) (at 323.85 43.18 0) (fields_autoplaced)
     (effects (font (size 1.27 1.27)) (justify left))
-    (property "Intersheetrefs" "${INTERSHEET_REFS}" (at 335.3907 50.8 0)
+    (property "Intersheetrefs" "${INTERSHEET_REFS}" (at 335.3907 43.18 0)
       (effects (font (size 1.27 1.27)) (justify left) hide)
     )
@@
     )
   )
-  (global_label "~{LOAD AC}" (shape input) (at 290.83 57.15 0) (fields_autoplaced)
+  (global_label "~{LOAD AC}" (shape input) (at 290.83 31.75 0) (fields_autoplaced)
     (effects (font (size 1.27 1.27)) (justify left))
-    (property "Intersheetrefs" "${INTERSHEET_REFS}" (at 300.9194 57.15 0)
+    (property "Intersheetrefs" "${INTERSHEET_REFS}" (at 300.9194 31.75 0)
       (effects (font (size 1.27 1.27)) (justify left) hide)
     )
@@
     )
   )
-  (global_label "~{INH TRANS}" (shape input) (at 323.85 43.18 0) (fields_autoplaced)
+  (global_label "~{INH TRANS}" (shape input) (at 323.85 50.8 0) (fields_autoplaced)
     (effects (font (size 1.27 1.27)) (justify left))
-    (property "Intersheetrefs" "${INTERSHEET_REFS}" (at 335.9956 43.18 0)
+    (property "Intersheetrefs" "${INTERSHEET_REFS}" (at 335.9956 50.8 0)
       (effects (font (size 1.27 1.27)) (justify left) hide)
     )
@@
     )
   )
-  (global_label "LOAD IR" (shape input) (at 290.83 59.69 0) (fields_autoplaced)
+  (global_label "LOAD IR" (shape input) (at 290.83 34.29 0) (fields_autoplaced)
     (effects (font (size 1.27 1.27)) (justify left))
-    (property "Intersheetrefs" "${INTERSHEET_REFS}" (at 300.4356 59.69 0)
+    (property "Intersheetrefs" "${INTERSHEET_REFS}" (at 300.4356 34.29 0)
       (effects (font (size 1.27 1.27)) (justify left) hide)
     )
@@
     )
   )
-  (global_label "~{MA LOAD}" (shape input) (at 323.85 45.72 0) (fields_autoplaced)
+  (global_label "~{MA LOAD}" (shape input) (at 323.85 38.1 0) (fields_autoplaced)
     (effects (font (size 1.27 1.27)) (justify left))
-    (property "Intersheetrefs" "${INTERSHEET_REFS}" (at 334.1208 45.72 0)
+    (property "Intersheetrefs" "${INTERSHEET_REFS}" (at 334.1208 38.1 0)
       (effects (font (size 1.27 1.27)) (justify left) hide)
     )
@@
       (effects (font (size 1.27 1.27)) (justify left))
     )
-    (property "Value" "Conn_01x16" (at 219.71 46.355 0)
+    (property "Value" "MBO" (at 219.71 46.355 0)
       (effects (font (size 1.27 1.27)) (justify left) hide)
     )
@@
       (effects (font (size 1.27 1.27)) (justify left))
     )
-    (property "Value" "Conn_01x10" (at 271.78 40.64 0)
+    (property "Value" "CPU Option Inputs" (at 271.78 40.64 0)
       (effects (font (size 1.27 1.27)) (justify left) hide)
     )
@@
       (effects (font (size 1.27 1.27)) (justify left))
     )
-    (property "Value" "Conn_01x16" (at 170.815 46.99 0)
+    (property "Value" "Data Channel" (at 170.815 46.99 0)
       (effects (font (size 1.27 1.27)) (justify left) hide)
     )
@@
       (effects (font (size 1.27 1.27)) (justify left))
     )
-    (property "Value" "Conn_01x04" (at 138.43 65.405 0)
+    (property "Value" "System Control" (at 138.43 65.405 0)
       (effects (font (size 1.27 1.27)) (justify left) hide)
     )
@@
       (effects (font (size 1.27 1.27)) (justify left))
     )
-    (property "Value" "Conn_01x18" (at 83.185 45.085 0)
+    (property "Value" "Programmed I/O" (at 83.185 45.085 0)
       (effects (font (size 1.27 1.27)) (justify left) hide)
     )
@@
       (effects (font (size 1.27 1.27)) (justify left))
     )
-    (property "Value" "Conn_01x08" (at 170.18 36.83 0)
+    (property "Value" "Data Channel" (at 170.18 36.83 0)
       (effects (font (size 1.27 1.27)) (justify left) hide)
     )
@@
       (effects (font (size 1.27 1.27)) (justify left))
     )
-    (property "Value" "Conn_01x04" (at 130.81 33.02 0)
+    (property "Value" "Program Interrupt" (at 130.81 33.02 0)
       (effects (font (size 1.27 1.27)) (justify left) hide)
     )
@@
     )
   )
+  (symbol (lib_id "Connector_Generic:Conn_01x10") (at 318.77 38.1 0) (mirror y) (unit 1)
+    (in_bom yes) (on_board yes) (dnp no)
+    (property "Reference" "J18" (at 320.675 53.34 0)
+      (effects (font (size 1.27 1.27)) (justify left))
+    )
+    (property "Value" "MEM Control Outputs" (at 315.595 41.275 0)
+      (effects (font (size 1.27 1.27)) (justify left) hide)
+    )
+    (property "Footprint" "Connector_PinHeader_2.54mm:PinHeader_1x10_P2.54mm_Horizontal" (at 318.77 38.1 0)
+      (effects (font (size 1.27 1.27)) hide)
+    )
+    (property "Datasheet" "~" (at 318.77 38.1 0)
+      (effects (font (size 1.27 1.27)) hide)
+    )
+    (pin "1")
+    (pin "10")
+    (pin "2")
+    (pin "3")
+    (pin "4")
+    (pin "5")
+    (pin "6")
+    (pin "7")
+    (pin "8")
+    (pin "9")
+    (instances
+      (project "DG Nova CPU Tester"
+        (path "/c1f710ce-b3f9-4828-9325-9c2326e8d74c"
+          (reference "J18") (unit 1)
+        )
+      )
+    )
+  )
   (symbol (lib_id "Jumper:Jumper_2_Open") (at 376.555 48.895 270) (mirror x) (unit 1)
     (in_bom yes) (on_board yes) (dnp no)
@@
       (effects (font (size 1.27 1.27)) (justify left))
     )
-    (property "Value" "Conn_01x18" (at 36.83 51.435 0)
+    (property "Value" "Front Panel Controls" (at 36.83 51.435 0)
       (effects (font (size 1.27 1.27)) (justify left) hide)
     )
@@
       (effects (font (size 1.27 1.27)) (justify left))
     )
-    (property "Value" "Conn_01x18" (at 218.44 48.895 0)
+    (property "Value" "MEM" (at 218.44 48.895 0)
       (effects (font (size 1.27 1.27)) (justify left) hide)
     )
@@
     )
   )
-  (symbol (lib_id "Connector_Generic:Conn_01x16") (at 285.75 46.99 0) (mirror y) (unit 1)
+  (symbol (lib_id "Connector_Generic:Conn_01x06") (at 285.75 34.29 0) (mirror y) (unit 1)
     (in_bom yes) (on_board yes) (dnp no)
-    (property "Reference" "J17" (at 287.655 69.85 0)
+    (property "Reference" "J17" (at 287.655 45.085 0)
       (effects (font (size 1.27 1.27)) (justify left))
     )
-    (property "Value" "Conn_01x16" (at 282.575 50.165 0)
+    (property "Value" "CPU Option Outputs" (at 282.575 37.465 0)
       (effects (font (size 1.27 1.27)) (justify left) hide)
     )
-    (property "Footprint" "Connector_PinHeader_2.54mm:PinHeader_1x16_P2.54mm_Horizontal" (at 285.75 46.99 0)
+    (property "Footprint" "Connector_PinHeader_2.54mm:PinHeader_1x16_P2.54mm_Horizontal" (at 285.75 34.29 0)
       (effects (font (size 1.27 1.27)) hide)
     )
-    (property "Datasheet" "~" (at 285.75 46.99 0)
+    (property "Datasheet" "~" (at 285.75 34.29 0)
       (effects (font (size 1.27 1.27)) hide)
     )
     (pin "1")
-    (pin "10")
-    (pin "11")
-    (pin "12")
-    (pin "13")
-    (pin "14")
-    (pin "15")
-    (pin "16")
     (pin "2")
     (pin "3")
@@
     (pin "5")
     (pin "6")
-    (pin "7")
-    (pin "8")
-    (pin "9")
     (instances
       (project "DG Nova CPU Tester"
@@
       (effects (font (size 1.27 1.27)) (justify left))
     )
-    (property "Value" "TestPoint" (at 43.3832 380.9492 0)
+    (property "Value" "Entrex Backplane S01B53 to S13B53" (at 43.3832 380.9492 0)
       (effects (font (size 1.27 1.27)) (justify left))
     )
