File: DG Nova CPU Tester/DG Nova CPU Tester.kicad_pcb (KiCad board)
At the start: 2 copper layers, 1 part

Commit message: PCB
Parts:
- added C1: CAP_Disc_Common_-_Entrex_Trapezoid, Forgotten Machines:Disc Capacitor Common Entrex Trapezoid, F.Cu at (-45.6, 14.7)
- added C2: CAP_Disc_Common_-_Entrex_Trapezoid, Forgotten Machines:Disc Capacitor Common Entrex Trapezoid, F.Cu at (-45.6, 18.8)
- added C3: C, Capacitor_THT:C_Disc_D6.0mm_W2.5mm_P5.00mm, F.Cu at (-48.4, -5.76)
- added C4: C, Capacitor_THT:C_Disc_D6.0mm_W2.5mm_P5.00mm, F.Cu at (-48.4, -1.72)
- added C5: C, Capacitor_THT:C_Disc_D6.0mm_W2.5mm_P5.00mm, F.Cu at (-48.4, 2.33)
- added D1: 1N4004, Diode_THT:D_DO-41_SOD81_P10.16mm_Horizontal, F.Cu at (-50.8, 74.8)
- added D2: 1N4004, Diode_THT:D_DO-41_SOD81_P10.16mm_Horizontal, F.Cu at (-50.8, 79.1)
- added D3: 1N4004, Diode_THT:D_DO-41_SOD81_P10.16mm_Horizontal, F.Cu at (-50.8, 83.3)
- added D4: 1N4004, Diode_THT:D_DO-41_SOD81_P10.16mm_Horizontal, F.Cu at (-50.8, 87.6)
- added D5: 1N4004, Diode_THT:D_DO-41_SOD81_P10.16mm_Horizontal, F.Cu at (-50.8, 91.8)
- added D6: 1N4004, Diode_THT:D_DO-41_SOD81_P10.16mm_Horizontal, F.Cu at (-50.8, 96.1)
- added J1: Front Panel Socket - Backside, Forgotten Machines:DG NOVA Front Pannel Connector - Backside, F.Cu at (-199.7, 9.46)
- added J10: Conn_01x18, Connector_PinHeader_2.54mm:PinHeader_1x18_P2.54mm_Horizontal, F.Cu at (-164.8, 75.0)
- added J11: Conn_01x16, Connector_PinHeader_2.54mm:PinHeader_1x16_P2.54mm_Horizontal, F.Cu at (-124.6, 75.0)
- added J12: Conn_01x08, Connector_PinHeader_2.54mm:PinHeader_1x08_P2.54mm_Horizontal, F.Cu at (-45.2, -29.8)
- added J13: Conn_01x04, Connector_PinHeader_2.54mm:PinHeader_1x04_P2.54mm_Horizontal, F.Cu at (-111.2, 102.5)
- added J14: Conn_01x04, Connector_PinHeader_2.54mm:PinHeader_1x04_P2.54mm_Horizontal, F.Cu at (-111.2, 114.8)
- added J15: Slot_02x50_Odd_Even, Forgotten Machines:DG NOVA Backplane Connector - Backside, F.Cu at (-114.3, 53.9)
- added J16: Slot_02x50_Odd_Even, Forgotten Machines:DG NOVA Backplane Connector - Backside, F.Cu at (-114.3, 66.4)
- added J17: Conn_01x10, Connector_PinHeader_2.54mm:PinHeader_1x10_P2.54mm_Horizontal, F.Cu at (-111.2, 75.0)
- added J2: ~, Forgotten Machines:DG NOVA Backplane Connector - Frontside, F.Cu at (-113.1, 28.9)
- added J3: ~, Forgotten Machines:DG NOVA Backplane Connector - Frontside, F.Cu at (-113.1, 41.4)
- added J4: ATX-24, Forgotten Machines:Connector_2x12_P4.2mmx5.5mm (ATX Plug), F.Cu at (-49.4, 104.3)
- added J5: Front Panel Card Edge, Forgotten Machines:DG Nova Front Panel Card Edge, F.Cu at (-219.3, 25.2)
- added J6: Conn_01x16, Connector_PinHeader_2.54mm:PinHeader_1x16_P2.54mm_Horizontal, F.Cu at (-151.4, 75.0)
- added J7: Conn_01x18, Connector_PinHeader_2.54mm:PinHeader_1x18_P2.54mm_Horizontal, F.Cu at (-191.6, 75.0)
- added J8: Conn_01x16, Connector_PinHeader_2.54mm:PinHeader_1x16_P2.54mm_Horizontal, F.Cu at (-138.0, 75.0)
- added J9: Conn_01x18, Connector_PinHeader_2.54mm:PinHeader_1x18_P2.54mm_Horizontal, F.Cu at (-178.2, 75.0)
- added JP1: Vipass Ammeter, Connector_PinHeader_2.54mm:PinHeader_1x02_P2.54mm_Vertical, F.Cu at (-151.4, 117.8)
- added JP2: Entrex ~{M CON DATA}, Connector_PinHeader_2.54mm:PinHeader_1x02_P2.54mm_Vertical, F.Cu at (-146.8, 117.8)
- added JP3: Entrex ~{M CON INST}, Connector_PinHeader_2.54mm:PinHeader_1x02_P2.54mm_Vertical, F.Cu at (-142.1, 117.8)
- added JP4: Vipass Ammeter, Connector_PinHeader_2.54mm:PinHeader_1x02_P2.54mm_Vertical, F.Cu at (-137.5, 117.8)
- added MES1: XK-001, Forgotten Machines:XK-001_Volt-Amp_Meter, F.Cu at (-76.8, 85.9)
- added R1: 1k, Resistor_THT:R_Axial_DIN0207_L6.3mm_D2.5mm_P10.16mm_Horizontal, F.Cu at (-59.2, -30.1)
- added R2: 10k, Resistor_THT:R_Axial_DIN0207_L6.3mm_D2.5mm_P10.16mm_Horizontal, F.Cu at (-59.2, -26.0)
- added R3: 4.7k, Resistor_THT:R_Axial_DIN0207_L6.3mm_D2.5mm_P10.16mm_Horizontal, F.Cu at (-59.2, -22.0)
- added R4: 4.7k, Resistor_THT:R_Axial_DIN0207_L6.3mm_D2.5mm_P10.16mm_Horizontal, F.Cu at (-59.2, -17.9)
- added R5: 10k, Resistor_THT:R_Axial_DIN0207_L6.3mm_D2.5mm_P10.16mm_Horizontal, F.Cu at (-59.2, -13.9)
- added R6: 1k, Resistor_THT:R_Axial_DIN0207_L6.3mm_D2.5mm_P10.16mm_Horizontal, F.Cu at (-59.2, -9.81)
- added SW1: SW_Push, Button_Switch_THT:SW_PUSH_6mm, F.Cu at (-47.9, 6.38)
- added TP1: TestPoint, Connector_PinHeader_2.54mm:PinHeader_1x01_P2.54mm_Vertical, F.Cu at (-132.8, 117.8)
- added U1: 74HC14, Package_DIP:DIP-14_W7.62mm, F.Cu at (-59.2, -5.71)
- added U2: Pico, Forgotten Machines:RPi_Pico_SMD_TH, F.Cu at (-72.8, -5.53)
- added XA1: Arduino_Mega2560_Shield, Forgotten Machines:Arduino_Mega2560_Shield, F.Cu at (-187.0, 21.8)
Other:
- board outline added: 16 x 114 mm

Commit message: board
Parts:
- removed MES1: XK-001, Forgotten Machines:XK-001_Volt-Amp_Meter
- moved J2 467.8 mm to (345.1, 123.2)
- moved J4 462.3 mm to (409.8, 50.7), turned to 90 degrees
- moved J15 460.7 mm to (343.3, 107.3)
- moved U2 458.1 mm to (378.5, 73.0)
- moved XA1 439.9 mm to (248.3, 85.1)
- moved J3 281.1 mm to (155.8, 123.2)
- moved J16 271.4 mm to (154.0, 107.3)
- moved J1 262.4 mm to (55.1, 72.1)
- moved J5 239.5 mm to (15.7, 71.2)
- moved SW1 80.2 mm to (31.4, 17.6)

Commit message: footprint
Parts:
- added J11: Conn_01x10, Connector_PinHeader_2.54mm:PinHeader_1x10_P2.54mm_Horizontal, F.Cu at (-159.3, 11.2)
- added J17: Conn_01x16, Connector_PinHeader_2.54mm:PinHeader_1x16_P2.54mm_Horizontal, F.Cu at (-172.7, 11.2)
- added MES1: XK-001, Forgotten Machines:XK-001_Volt-Amp_Meter - Backside, F.Cu at (-151.0, -5.02)

Commit message: update
Parts:
- moved MES1 554.5 mm to (402.6, 27.3)
- moved JP1 543.0 mm to (386.7, 45.7), turned to -90 degrees
- moved JP4 528.6 mm to (386.7, 49.5), turned to -90 degrees
- moved TP1 473.0 mm to (328.9, 15.2)
- moved JP3 469.1 mm to (315.6, 15.2)
- moved JP2 458.1 mm to (299.7, 15.2)
- moved C1 451.9 mm to (391.2, 130.6)
- moved C2 439.2 mm to (379.1, 130.6)
- moved R6 201.3 mm to (110.5, 98.4), turned to 90 degrees
- moved R5 200.1 mm to (106.4, 98.4), turned to 90 degrees
- moved R4 199.1 mm to (102.4, 98.4), turned to 90 degrees
- moved R3 198.3 mm to (98.3, 98.4), turned to 90 degrees
- moved R2 197.6 mm to (94.3, 98.4), turned to 90 degrees
- moved R1 190.6 mm to (90.2, 88.3), turned to -90 degrees
- moved D6 162.6 mm to (111.4, 85.1), turned to 90 degrees
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
Commit message: build
Parts:
- removed the J11 at (-124.6, 75.0)
- removed the J11 at (-159.3, 11.2)
- removed the J17 at (-111.2, 75.0)
- removed the J17 at (-172.7, 11.2)
- added J11: CPU Option Inputs, Connector_PinHeader_2.54mm:PinHeader_1x10_P2.54mm_Horizontal, F.Cu at (355.6, 7.62)
- added J17: CPU Option Outputs, Connector_PinHeader_2.54mm:PinHeader_1x06_P2.54mm_Horizontal, F.Cu at (383.5, 7.62)
- added J18: MEM Control Outputs, Connector_PinHeader_2.54mm:PinHeader_1x10_P2.54mm_Horizontal, F.Cu at (215.9, 7.62)
- added J19: Logic 8 CH, Connector_PinHeader_2.54mm:PinHeader_2x05_P2.54mm_Vertical, F.Cu at (80.0, 56.5)
- added J20: Logic 8 CH, Connector_PinHeader_2.54mm:PinHeader_1x08_P2.54mm_Horizontal, F.Cu at (76.2, 42.5)
- J10: value Conn_01x18 -> Programmed I/O
- J12: value Conn_01x08 -> Data Channel
- J13: value Conn_01x04 -> Program Interrupt
- J14: value Conn_01x04 -> System Control
- J6: value Conn_01x16 -> MBO
- J7: value Conn_01x18 -> MEM
- J8: value Conn_01x16 -> Data Channel
- J9: value Conn_01x18 -> Front Panel Controls
- TP1: value TestPoint -> Entrex Backplane S01B53 to S13B53
- moved J14 464.1 mm to (340.4, 7.62), turned to 90 degrees
- moved J6 451.2 mm to (294.6, 7.55), turned to 90 degrees
- moved J7 440.7 mm to (243.8, 7.62), turned to 90 degrees
- moved U1 316.9 mm to (393.7, 81.3)
- moved J8 315.5 mm to (170.2, 7.62), turned to 90 degrees
- moved C3 286.6 mm to (353.1, 87.4)
- moved C4 286.6 mm to (353.1, 91.4)
- moved C5 286.6 mm to (353.1, 95.5)
- moved J12 284.7 mm to (147.3, 7.62), turned to 90 degrees
- moved R3 276.1 mm to (374.4, 96.5)
- moved D1 276.1 mm to (366.2, 83.2)
- moved D2 276.1 mm to (370.4, 83.2)
- moved D3 276.1 mm to (374.7, 83.2)
- moved D4 276.1 mm to (378.9, 83.2)
- moved D5 276.1 mm to (383.2, 83.2)
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Other:
- board text added: "LEDs"

Commit message: b
Parts:
- added D10: LED, LED_THT:LED_D3.0mm, F.Cu at (-36.8, 36.1)
- added D7: LED, LED_THT:LED_D3.0mm, F.Cu at (-36.8, 19.4)
- added D8: LED, LED_THT:LED_D3.0mm, F.Cu at (-36.8, 25.0)
- added D9: LED, LED_THT:LED_D3.0mm, F.Cu at (-36.8, 30.5)
- added R10: 68Ω, Resistor_THT:R_Axial_DIN0204_L3.6mm_D1.6mm_P7.62mm_Horizontal, F.Cu at (-31.1, 27.7)
- added R7: 68Ω, Resistor_THT:R_Axial_DIN0204_L3.6mm_D1.6mm_P7.62mm_Horizontal, F.Cu at (-31.1, 18.2)
- added R8: 68Ω, Resistor_THT:R_Axial_DIN0204_L3.6mm_D1.6mm_P7.62mm_Horizontal, F.Cu at (-31.1, 21.4)
- added R9: 68Ω, Resistor_THT:R_Axial_DIN0204_L3.6mm_D1.6mm_P7.62mm_Horizontal, F.Cu at (-31.1, 24.5)
- J19: footprint Connector_PinHeader_2.54mm:PinHeader_2x05_P2.54mm_Vertical -> Forgotten Machines:PinHeader_2x05_P2.54mm_Vertical - Backside
- moved J1 5.92 mm to (34.0, 72.0)
- moved J19 4.46 mm to (80.3, 52.1)
Other:
- board text added: "Make LEDs smaller (LED bars)"

Commit message: big build
Parts:
- removed D10, D9: LED, LED_THT:LED_D3.0mm
- removed R10, R9: 68Ω, Resistor_THT:R_Axial_DIN0204_L3.6mm_D1.6mm_P7.62mm_Horizontal
- added BAR1: LED Bar 10, Forgotten Machines:LED Bar 10, F.Cu at (33.0, 43.8)
- added BAR2: LED Bar 10, Forgotten Machines:LED Bar 7, F.Cu at (58.4, 43.8)
- added BAR3: LED Bar 10, Forgotten Machines:LED Bar 10, F.Cu at (81.3, 43.8)
- added BAR4: LED Bar 10, Forgotten Machines:LED Bar 6, F.Cu at (106.7, 43.7)
- added BAR5: LED Bar 10, Forgotten Machines:LED Bar 10, F.Cu at (124.5, 43.8)
- added BAR6: LED Bar 10, Forgotten Machines:LED Bar 6, F.Cu at (149.9, 43.8)
- added RN1: R_Network09_US, Resistor_THT:R_Array_SIP10, F.Cu at (30.5, 47.0)
- added RN2: R_Network08_US, Resistor_THT:R_Array_SIP9, F.Cu at (76.2, 47.0)
- added RN3: R_Network09_US, Resistor_THT:R_Array_SIP10, F.Cu at (78.7, 47.0)
- added RN4: R_Network07_US, Resistor_THT:R_Array_SIP8, F.Cu at (121.9, 47.0)
- added RN5: R_Network09_US, Resistor_THT:R_Array_SIP10, F.Cu at (121.9, 47.0)
- added RN6: R_Network07_US, Resistor_THT:R_Array_SIP8, F.Cu at (165.1, 47.0)
- D7, D8: footprint LED_THT:LED_D3.0mm -> LED_THT:LED_D1.8mm_W3.3mm_H2.4mm
- J10: value Programmed I/O -> Front Panel Controls; footprint Connector_PinHeader_2.54mm:PinHeader_1x18_P2.54mm_Horizontal -> Connector_PinHeader_2.54mm:PinHeader_1x17_P2.54mm_Vertical
- J11, J18: footprint Connector_PinHeader_2.54mm:PinHeader_1x10_P2.54mm_Horizontal -> Connector_PinHeader_2.54mm:PinHeader_1x10_P2.54mm_Vertical
- J12, J20: footprint Connector_PinHeader_2.54mm:PinHeader_1x08_P2.54mm_Horizontal -> Connector_PinHeader_2.54mm:PinHeader_1x08_P2.54mm_Vertical
- J13, J14: footprint Connector_PinHeader_2.54mm:PinHeader_1x04_P2.54mm_Horizontal -> Connector_PinHeader_2.54mm:PinHeader_1x04_P2.54mm_Vertical
- J17: footprint Connector_PinHeader_2.54mm:PinHeader_1x06_P2.54mm_Horizontal -> Connector_PinHeader_2.54mm:PinHeader_1x05_P2.54mm_Vertical
- J6, J8: footprint Connector_PinHeader_2.54mm:PinHeader_1x16_P2.54mm_Horizontal -> Connector_PinHeader_2.54mm:PinHeader_1x16_P2.54mm_Vertical
- J7: footprint Connector_PinHeader_2.54mm:PinHeader_1x18_P2.54mm_Horizontal -> Connector_PinHeader_2.54mm:PinHeader_1x18_P2.54mm_Vertical
- J9: footprint Connector_PinHeader_2.54mm:PinHeader_1x18_P2.54mm_Horizontal -> Connector_PinHeader_2.54mm:PinHeader_1x17_P2.54mm_Vertical
- R7, R8: value 68Ω -> R_US; footprint Resistor_THT:R_Axial_DIN0204_L3.6mm_D1.6mm_P7.62mm_Horizontal -> Resistor_THT:R_Axial_DIN0204_L3.6mm_D1.6mm_P5.08mm_Horizontal
- moved FPIMAGE1 639.8 mm to (-309.2, -307.3)
- moved J6 214.8 mm to (81.3, 32.8)
- moved D8 204.5 mm to (167.6, 27.3), turned to -90 degrees
- moved R8 202.6 mm to (170.2, 43.8), turned to 90 degrees
- moved J16 200.9 mm to (335.0, 125.7)
- moved J10 192.2 mm to (271.8, 32.8)
- moved J13 187.1 mm to (317.5, 32.8)
- moved J15 179.4 mm to (145.8, 125.7)
- moved J7 122.0 mm to (124.5, 32.8)
- moved R7 111.0 mm to (76.8, 43.8), turned to 90 degrees
- moved D7 108.2 mm to (71.1, 27.3), turned to -90 degrees
- moved J12 102.2 mm to (246.4, 32.8)
- moved J18 50.0 mm to (172.7, 32.8)
- moved J8 41.5 mm to (203.2, 32.8)
- moved JP2 38.2 mm to (73.0, 56.5)
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Connections:
- D7 pad 2: unconnected-(D7-A-Pad2) -> RESTART ENABLE
- D8 pad 2: unconnected-(D8-A-Pad2) -> MEM OK
- J9 pad 3: ~{CARRY} -> ~{FETCH}
- J9 pad 4: ~{FETCH} -> ~{DEFER}
- J9 pad 5: ~{DEFER} -> ~{EXEC}
- J9 pad 6: ~{EXEC} -> ~{CARRY}
- R7 pad 1: Net-(D7-K) -> GND
- R7 pad 2: GND -> Net-(D7-K)
- R8 pad 1: Net-(D8-K) -> GND
- R8 pad 2: GND -> Net-(D8-K)
Routing:
- net Net-(D7-K): track 0.00 -> 13.8 mm
- net Net-(D8-K): track 0.00 -> 12.5 mm
- net (no net): track 0.00 -> 6.35 mm
- net ~{STOP}: track 0.00 -> 3.81 mm
- net ~{SKIP}: track 0.00 -> 3.81 mm
- net ~{RUN}: track 0.00 -> 3.81 mm
- net ~{RST}: track 0.00 -> 3.81 mm
- net ~{PL}: track 0.00 -> 3.81 mm
- net ~{MSTP}: track 0.00 -> 3.81 mm
- net ~{ISTP}: track 0.00 -> 3.81 mm
- net ~{ION}: track 0.00 -> 3.81 mm
- net ~{FETCH}: track 0.00 -> 3.81 mm
- net ~{EXEC}: track 0.00 -> 3.81 mm
- net ~{DEFER}: track 0.00 -> 3.81 mm
- net ~{CONT+ISTP+MSTP}: track 0.00 -> 3.81 mm
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Other:
- board size 16 x 114 mm -> 414.8 x 131.4 mm
- board text added: "MEM OK"
- board text added: "RESTART ENABLE"
- board text added: "Resistor Blocks Share Pin 1 Hole"
- board text added: "consider putting silkscreen borders for resistor blocks on the backside as well"
- board text added: "~{FETCH}"
- board text added: "~{ION}"
- board text added: "~{RUN}"
- board text removed: "LEDs"
- board text removed: "Make LEDs smaller (LED bars)"
