File: DG Nova CPU Tester/DG Nova CPU Tester.kicad_pcb (KiCad board)
At the start: 2 copper layers, 414.8 x 131.4 mm, 64 parts, among them J1 Front Panel Socket - Backside, J10 Front Panel Controls, J11 CPU Option Inputs, J12 Data Channel, J13 Program Interrupt, J14 System Control, J15 Slot_02x50_Odd_Even, J16 Slot_02x50_Odd_Even, J17 CPU Option Outputs, J18 MEM Control Outputs, J19 Logic 8 CH, J20 Logic 8 CH, J4 ATX-24, J5 Front Panel Card Edge, J6 MBO, J7 MEM, J8 Data Channel, J9 Front Panel Controls, SW1 SW_Push, U1 74HC14, U2 Pico

Commit message: TRACE
Parts:
- added BAR7: LED Bar 10, Forgotten Machines:LED Bar 10, F.Cu at (172.7, 43.8)
- added RN7: R_Network09_US, Resistor_THT:R_Array_SIP10, F.Cu at (170.2, 47.0)
- moved R8 1.27 mm to (168.9, 43.8)
Routing:
- net ~{MSKO}: track 0.00 -> 242.5 mm
- net ~{DATA0}: track 0.00 -> 235.5 mm
- net INTA: track 0.00 -> 234.0 mm
- net ~{DATA8}: track 0.00 -> 228.8 mm
- net DATIB: track 0.00 -> 227.3 mm
- net ~{DATA11}: track 0.00 -> 222.1 mm
- net DATIA: track 0.00 -> 220.6 mm
- net ~{DATA14}: track 0.00 -> 215.3 mm
- net ~{DS3}: track 0.00 -> 213.8 mm
- net DATOC: track 0.00 -> 207.1 mm
- net CLR: track 0.00 -> 200.9 mm
- net DATIC: track 0.00 -> 197.9 mm
- net ~{MEM2}: track 0.00 -> 195.9 mm
- net STRT: track 0.00 -> 194.6 mm
- net DATOB: track 0.00 -> 190.9 mm
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Other:
- board text added: "1"
- board text added: "10"
- board text added: "11"
- board text added: "12"
- board text added: "13"
- board text added: "14"
- board text added: "2"
- board text added: "3"
- board text added: "4"
- board text added: "5"
- board text added: "6"
- board text added: "7"
- board text added: "8"
- board text added: "9"
- board text added: "Address ~{MBO}"
- board text added: "Data Channel"
- board text added: "Data Channel ~{DATA}"
- board text added: "Data ~{MEM}"
- board text added: "Front Panel Controls"
- board text added: "MEM Control Outputs"
- board text added: "~{DATA0}"
- board text added: "~{DATA15}"
- board text added: "~{MBO0}"
- board text added: "~{MBO15}"
- board text added: "~{MEM0}"
- board text added: "~{MEM15}"
- board text added: "~{TRY ME}"

Commit message: w
Parts:
- moved C3 45.3 mm to (368.0, 62.2)
- moved C4 43.5 mm to (365.0, 67.4)
- moved C5 40.2 mm to (365.4, 74.9)
- moved XA1 30.8 mm to (121.7, 102.4)
- moved R1 25.7 mm to (379.0, 81.2)
- moved R2 25.7 mm to (383.1, 91.3)
- moved D1 25.7 mm to (378.9, 78.0)
- moved D2 25.7 mm to (383.2, 78.0)
- moved D3 25.7 mm to (387.4, 78.0)
- moved D4 25.7 mm to (391.7, 78.0)
- moved D5 25.7 mm to (395.9, 78.0)
- moved D6 25.7 mm to (400.2, 78.0)
- moved R3 25.7 mm to (387.1, 91.3)
- moved R4 25.7 mm to (391.2, 91.3)
- moved R5 25.7 mm to (395.2, 91.3)
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Routing:
- net ~{READ2}: track 3.43 -> 392.9 mm
- net ~{DATA6}: track 0.00 -> 352.7 mm
- net ~{READ1}: track 3.43 -> 334.0 mm
- net ~{READ IO}: track 3.43 -> 319.2 mm
- net ~{MBO0}: track 3.43 -> 305.7 mm
- net ~{MBO1}: track 3.43 -> 299.0 mm
- net ~{DATA10}: track 0.00 -> 287.4 mm
- net ~{DATA3}: track 0.00 -> 280.7 mm
- net ~{MEM0}: track 3.43 -> 275.7 mm
- net ~{DATA1}: track 0.00 -> 252.6 mm
- net ~{DATA9}: track 0.00 -> 245.9 mm
- net ~{DATA4}: track 0.00 -> 239.3 mm
- net ~{DATA12}: track 0.00 -> 232.4 mm
- net ~{DATA5}: track 0.00 -> 225.7 mm
- net ~{DATA7}: track 0.00 -> 219.3 mm
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
Commit message: yes
Routing:
- net ~{DATA13}: track 71.8 -> 516.2 mm
- net ~{DATA15}: track 68.2 -> 506.5 mm
- net ~{MEM3}: track 67.4 -> 496.1 mm
- net ~{MEM1}: track 63.6 -> 486.3 mm
- net MB LOAD: track 53.0 -> 462.8 mm
- net ~{DATA2}: track 40.8 -> 422.6 mm
- net ~{MB CLEAR}: track 36.7 -> 409.8 mm
- net ~{MEM14}: track 83.6 -> 456.5 mm
- net ~{DRIVE IO}: track 31.2 -> 383.8 mm, vias 0 -> 2
- net GND: track 37.7 -> 48.2 mm
- net ~{READ2}: track 392.9 -> 383.1 mm
- net ~{DATA6}: track 352.7 -> 358.4 mm, vias 0 -> 2

Commit message: build
Parts:
- added BAR11: LED Bar 10, Forgotten Machines:LED Bar 5, F.Cu at (246.4, 43.8)
- added BAR8: LED Bar 10, Forgotten Machines:LED Bar 10, F.Cu at (203.2, 43.8)
- added BAR9: LED Bar 10, Forgotten Machines:LED Bar 6, F.Cu at (228.6, 43.8)
- added D10: LED, LED_THT:LED_D1.8mm_W3.3mm_H2.4mm, F.Cu at (190.5, 27.3)
- added D11: LED, LED_THT:LED_D1.8mm_W3.3mm_H2.4mm, F.Cu at (193.0, 27.3)
- added D13: LED, LED_THT:LED_D1.8mm_W3.3mm_H2.4mm, F.Cu at (259.1, 27.3)
- added D14: LED, LED_THT:LED_D1.8mm_W3.3mm_H2.4mm, F.Cu at (261.6, 27.3)
- added D15: LED, LED_THT:LED_D1.8mm_W3.3mm_H2.4mm, F.Cu at (264.2, 27.3)
- added D9: LED, LED_THT:LED_D1.8mm_W3.3mm_H2.4mm, F.Cu at (185.4, 27.3)
- added RN10: R_Network05_US, Resistor_THT:R_Array_SIP6, F.Cu at (243.8, 47.0)
- added RN11: R_Network09_US, Resistor_THT:R_Array_SIP10, F.Cu at (212.7, 8.89)
- added RN8: R_Network09_US, Resistor_THT:R_Array_SIP10, F.Cu at (200.7, 47.0)
- added RN9: R_Network07_US, Resistor_THT:R_Array_SIP8, F.Cu at (243.8, 47.0)
- J10: value Front Panel Controls -> Programmed I/O
- moved JP2 425.8 mm to (497.6, 88.6)
- moved JP3 425.8 mm to (515.4, 88.6)
- moved U2 209.2 mm to (536.4, 12.3)
- moved SW1 195.4 mm to (134.5, -123.9)
- moved C4 150.8 mm to (514.6, 48.5)
- moved R3 150.8 mm to (536.7, 72.4)
- moved R5 150.8 mm to (544.8, 72.4)
- moved C5 150.8 mm to (515.0, 56.0)
- moved D1 150.8 mm to (528.5, 59.1)
- moved D2 150.8 mm to (532.8, 59.1)
- moved D3 150.8 mm to (537.0, 59.1)
- moved D4 150.8 mm to (541.3, 59.1)
- moved D5 150.8 mm to (545.5, 59.1)
- moved D6 150.8 mm to (549.8, 59.1)
- moved R4 150.8 mm to (540.8, 72.4)
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Connections:
- BAR7 pad 10: unconnected-(BAR7-Pad10) -> Net-(RN7-R9)
- BAR7 pad 11: unconnected-(BAR7-K-Pad11) -> ~{INH TRANS}
- BAR7 pad 9: Net-(RN7-R9) -> unconnected-(BAR7-Pad9)
- J4 pad 14: unconnected-(J4--12V-Pad14) -> -12v
- J4 pad 20: unconnected-(J4--5v-Pad20) -> -5V
Routing:
- net ~{RUN}: track 3.81 -> 628.7 mm, vias 0 -> 6
- net ~{MBO13}: track 3.32 -> 602.9 mm, vias 0 -> 6
- net ~{EXEC}: track 3.81 -> 600.1 mm, vias 0 -> 8
- net ~{MEM12}: track 14.8 -> 603.2 mm, vias 0 -> 3
- net ~{FETCH}: track 3.81 -> 588.2 mm, vias 0 -> 7
- net ~{MEM13}: track 3.43 -> 587.0 mm, vias 0 -> 5
- net +12V Lamp: track 0.00 -> 558.9 mm, vias 0 -> 1
- net ~{MBO14}: track 3.32 -> 558.4 mm, vias 0 -> 5
- net ~{MEM10}: track 3.43 -> 554.3 mm, vias 0 -> 5
- net ~{MBO12}: track 3.32 -> 551.7 mm, vias 0 -> 5
- net ~{EXT LOAD}: track 0.00 -> 538.3 mm, vias 0 -> 4
- net ~{MBO15}: track 3.31 -> 536.5 mm, vias 0 -> 4
- net ~{MEM11}: track 3.43 -> 536.5 mm, vias 0 -> 5
- net ~{MEM9}: track 3.43 -> 530.5 mm, vias 0 -> 5
- net ~{WHOA}: track 0.00 -> 522.8 mm, vias 0 -> 4
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Other:
- board text added: "DCHI"
- board text added: "DCHO"
- board text added: "DCHP"
- board text added: "Entrex Backplane S01B53 to S13B53"
- board text added: "INHIBIT"
- board text added: "MB LOAD"
- board text added: "MEM Control"
- board text added: "OVFLO"
- board text added: "STROBE"
- board text added: "~{CARRY}"
- board text added: "~{CON DATA}"
- board text added: "~{CON INST}"
- board text added: "~{CON RQ}"
- board text added: "~{CONT+ISTP+MSTP}"
- board text added: "~{DCHA}"
- board text added: "~{DCHM0}"
- board text added: "~{DCHM1}"
- board text added: "~{DCHR}"
- board text added: "~{DEFER}"
- board text added: "~{DRIVE IO}"
- board text added: "~{DS0}"
- board text added: "~{DS0} ~{DS1} ~{DS2} ~{DS3} ~{DS4} ~{DS5} DATIA DATIB DATIC DATOA DATOB DATOC STRT CLR IO PLS ~{SELB} ~{SELD}"
- board text added: "~{DS1}"
- board text added: "~{DS2}"
- board text added: "~{DS3}"
- board text added: "~{DS4}"
- board text added: "~{DS5}"
- board text added: "~{EXEC}"
- board text added: "~{INH TRANS}"
- board text added: "~{ISTP}"
- board text added: "~{MA LOAD}"
- board text added: "~{MB CLEAR}"
- board text added: "~{MSTP}"
- board text added: "~{PL}"
- board text added: "~{READ IO}"
- board text added: "~{READ1}"
- board text added: "~{READ2}"
- board text added: "~{RST}"
- board text added: "~{SELB}"
- board text added: "~{SELD}"
- board text added: "~{SKIP}"
- board text added: "~{STOP}"
- board text removed: "MEM Control Outputs"

Commit message: build
Parts:
- added J21: Arduino Anolog Pins, Connector_PinHeader_2.54mm:PinHeader_1x10_P2.54mm_Vertical, F.Cu at (137.2, 60.7)
Connections:
- XA1 pad A0: unconnected-(XA1-PadA0) -> Net-(J21-Pin_10)
- XA1 pad A1: unconnected-(XA1-PadA1) -> Net-(J21-Pin_9)
- XA1 pad A10: unconnected-(XA1-PadA10) -> Net-(J21-Pin_6)
- XA1 pad A11: unconnected-(XA1-PadA11) -> Net-(J21-Pin_5)
- XA1 pad A12: unconnected-(XA1-PadA12) -> Net-(J21-Pin_4)
- XA1 pad A13: unconnected-(XA1-PadA13) -> Net-(J21-Pin_3)
- XA1 pad A14: unconnected-(XA1-PadA14) -> Net-(J21-Pin_2)
- XA1 pad A15: unconnected-(XA1-PadA15) -> Net-(J21-Pin_1)
- XA1 pad A8: unconnected-(XA1-PadA8) -> Net-(J21-Pin_8)
- XA1 pad A9: unconnected-(XA1-PadA9) -> Net-(J21-Pin_7)
Routing:
- net RESTART ENABLE: track 166.9 -> 588.0 mm, vias 1 -> 4
- net ~{CON RQ}: track 402.6 -> 574.9 mm, vias 3 -> 4
- net ~{CON INST}: track 421.5 -> 590.2 mm, vias 2 -> 3
- net ~{RST}: track 428.2 -> 594.1 mm, vias 2 -> 3
- net ~{PL}: track 428.3 -> 592.1 mm, vias 2 -> 3
- net INHIBIT: track 400.4 -> 502.4 mm, vias 3 -> 4
- net ~{ISTP}: track 410.5 -> 442.5 mm, vias 2 -> 3
- net Net-(J21-Pin_10): track 0.00 -> 24.1 mm, vias 0 -> 1
- net ~{MSTP}: track 162.9 -> 186.5 mm
- net Net-(J21-Pin_9): track 0.00 -> 22.4 mm, vias 0 -> 1
- net ~{RQENB}: track 447.1 -> 435.7 mm
- net ~{CARRY}: track 447.9 -> 456.3 mm
- net ~{MBO13}: track 602.9 -> 595.2 mm
- net ~{EXT LOAD}: track 538.3 -> 532.3 mm
- net ~{INTR}: track 425.0 -> 419.8 mm
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Other:
- board text added: "A15 A14 A13 A12 A11 A10 A09 A08 A01 A00"
- board text added: "Arduino Anolog Pins"
- board text added: "D53"

Commit message: trace
Parts:
- added J22: Arduino Digital Pins, Connector_PinHeader_2.54mm:PinHeader_1x06_P2.54mm_Vertical, F.Cu at (170.2, 104.3)
- added J23: Arduino Digital Pins, Connector_PinHeader_2.54mm:PinHeader_1x06_P2.54mm_Vertical, F.Cu at (186.9, 104.3)
- SW1: value SW_Push -> Arduino Reset
- moved D4 259.0 mm to (283.4, 82.9), turned to -90 degrees
- moved R4 255.1 mm to (286.6, 93.1)
- moved D5 251.6 mm to (296.2, 93.2)
- moved R3 247.3 mm to (289.7, 83.1), turned to -90 degrees
- moved R6 247.2 mm to (302.6, 93.2)
- moved D3 246.5 mm to (292.9, 93.2)
- moved R5 245.6 mm to (299.5, 83.1), turned to -90 degrees
- moved D6 245.2 mm to (305.7, 83.1), turned to -90 degrees
- moved U1 233.0 mm to (325.3, 89.9), turned to 90 degrees
- moved D2 224.9 mm to (309.2, 83.1), turned to -90 degrees
- moved SW1 221.9 mm to (202.1, 87.5), turned to 180 degrees
- moved R2 221.3 mm to (312.3, 93.0)
- moved R1 214.0 mm to (315.5, 82.7)
- moved D1 212.6 mm to (318.7, 93.1)
- moved C5 196.0 mm to (322.0, 90.0), turned to 90 degrees
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Connections:
- XA1 pad D10: unconnected-(XA1-PadD10) -> Net-(J23-Pin_3)
- XA1 pad D11: unconnected-(XA1-PadD11) -> Net-(J23-Pin_4)
- XA1 pad D12: unconnected-(XA1-PadD12) -> Net-(J23-Pin_5)
- XA1 pad D13: unconnected-(XA1-PadD13) -> Net-(J23-Pin_6)
- XA1 pad D2: unconnected-(XA1-D2_INT0-PadD2) -> Net-(J22-Pin_1)
- XA1 pad D3: unconnected-(XA1-D3_INT1-PadD3) -> Net-(J22-Pin_2)
- XA1 pad D4: unconnected-(XA1-PadD4) -> Net-(J22-Pin_3)
- XA1 pad D5: unconnected-(XA1-PadD5) -> Net-(J22-Pin_4)
- XA1 pad D6: unconnected-(XA1-PadD6) -> Net-(J22-Pin_5)
- XA1 pad D7: unconnected-(XA1-PadD7) -> Net-(J22-Pin_6)
- XA1 pad D8: unconnected-(XA1-PadD8) -> Net-(J23-Pin_1)
- XA1 pad D9: unconnected-(XA1-PadD9) -> Net-(J23-Pin_2)
Routing:
- net ~{MSTP}: track 186.5 -> 688.1 mm, vias 1 -> 4
- net ~{MBO1}: track 426.5 -> 809.2 mm, vias 1 -> 6
- net ~{CONT+ISTP+MSTP}: track 148.6 -> 519.3 mm, vias 2 -> 6
- net ~{STOP}: track 133.9 -> 500.4 mm, vias 1 -> 5
- net ~{MEM1}: track 697.0 -> 1028.5 mm
- net ~{CON DATA}: track 159.2 -> 488.1 mm, vias 2 -> 5
- net ~{MEM2}: track 400.5 -> 711.9 mm, vias 2 -> 3
- net ~{MBO3}: track 297.6 -> 600.5 mm, vias 2 -> 7
- net ~{MBO2}: track 331.6 -> 630.2 mm, vias 2 -> 7
- net ~{READ2}: track 440.9 -> 723.2 mm, vias 4 -> 6
- net GND: track 237.8 -> 497.0 mm, vias 8 -> 17
- net ~{MEM0}: track 486.0 -> 735.0 mm, vias 1 -> 3
- net ~{DRIVE IO}: track 437.6 -> 659.4 mm, vias 5 -> 7
- net +5V: track 340.8 -> 529.9 mm, vias 1 -> 2
- net ~{SHIFT1}: track 77.4 -> 266.0 mm
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Other:
- board text added: "Arduino Digital Pins"
- board text added: "D02 D03 D04 D05 D06 D07"
- board text added: "D08 D09 D10 D11 D12 D13"

Commit message: Wow
Parts:
- added BAR10: LED Bar 10, Forgotten Machines:LED Bar 6, F.Cu at (271.8, 43.8)
- added BAR12: LED Bar 2, Forgotten Machines:LED Bar 2, F.Cu at (309.9, 43.8)
- added BAR13: LED Bar 4, Forgotten Machines:LED Bar 4, F.Cu at (317.5, 43.8)
- added BAR14: LED Bar 4, Forgotten Machines:LED Bar 4, F.Cu at (332.7, 43.8)
- added BAR15: LED Bar 10, Forgotten Machines:LED Bar 10, F.Cu at (348.0, 43.8)
- added BAR16: LED Bar 10, Forgotten Machines:LED Bar 6, F.Cu at (375.9, 43.8)
- added D12: LED, LED_THT:LED_D1.8mm_W3.3mm_H2.4mm, F.Cu at (287.0, 27.3)
- added D16: LED, LED_THT:LED_D1.8mm_W3.3mm_H2.4mm, F.Cu at (289.6, 27.3)
- added D17: LED, LED_THT:LED_D1.8mm_W3.3mm_H2.4mm, F.Cu at (292.1, 27.3)
- added D18: LED, LED_THT:LED_D1.8mm_W3.3mm_H2.4mm, F.Cu at (299.7, 27.3)
- added D19: LED, LED_THT:LED_D1.8mm_W3.3mm_H2.4mm, F.Cu at (302.3, 27.3)
- added D20: LED, LED_THT:LED_D1.8mm_W3.3mm_H2.4mm, F.Cu at (304.8, 27.3)
- added D21: LED, LED_THT:LED_D1.8mm_W3.3mm_H2.4mm, F.Cu at (294.6, 27.3)
- added D22: LED, LED_THT:LED_D1.8mm_W3.3mm_H2.4mm, F.Cu at (297.2, 27.3)
- added D23: LED, LED_THT:LED_D1.8mm_W3.3mm_H2.4mm, F.Cu at (307.3, 27.3)
- added D24: LED, LED_THT:LED_D1.8mm_W3.3mm_H2.4mm, F.Cu at (337.8, 27.3)
- added D25: LED, LED_THT:LED_D1.8mm_W3.3mm_H2.4mm, F.Cu at (325.1, 27.3)
- added D26: LED, LED_THT:LED_D1.8mm_W3.3mm_H2.4mm, F.Cu at (332.7, 27.3)
- added D27: LED, LED_THT:LED_D1.8mm_W3.3mm_H2.4mm, F.Cu at (381.0, 27.3)
- added D28: LED, LED_THT:LED_D1.8mm_W3.3mm_H2.4mm, F.Cu at (375.9, 27.3)
- added R10: R_US, Resistor_THT:R_Axial_DIN0204_L3.6mm_D1.6mm_P5.08mm_Horizontal, F.Cu at (304.8, 46.4)
- added R11: R_US, Resistor_THT:R_Axial_DIN0204_L3.6mm_D1.6mm_P5.08mm_Horizontal, F.Cu at (327.7, 37.5)
- added R12: R_US, Resistor_THT:R_Axial_DIN0204_L3.6mm_D1.6mm_P5.08mm_Horizontal, F.Cu at (330.2, 37.5)
- added R13: R_US, Resistor_THT:R_Axial_DIN0204_L3.6mm_D1.6mm_P5.08mm_Horizontal, F.Cu at (391.3, 32.6)
- added R14: R_US, Resistor_THT:R_Axial_DIN0204_L3.6mm_D1.6mm_P5.08mm_Horizontal, F.Cu at (342.9, 37.5)
- added R15: R_US, Resistor_THT:R_Axial_DIN0204_L3.6mm_D1.6mm_P5.08mm_Horizontal, F.Cu at (373.4, 37.5)
- added R9: R_US, Resistor_THT:R_Axial_DIN0204_L3.6mm_D1.6mm_P5.08mm_Horizontal, F.Cu at (312.4, 51.4)
- added RN12: R_Network06_US, Resistor_THT:R_Array_SIP7, F.Cu at (269.2, 47.0)
- added RN13: R_Network09_US, Resistor_THT:R_Array_SIP10, F.Cu at (315.0, 47.0)
- added RN14: R_Network09_US, Resistor_THT:R_Array_SIP10, F.Cu at (284.5, 38.7)
- added RN15: R_Network09_US, Resistor_THT:R_Array_SIP10, F.Cu at (345.4, 47.0)
- added RN16: R_Network05_US, Resistor_THT:R_Array_SIP6, F.Cu at (373.4, 47.0)
- added TP2: ATX PWR_OK, Connector_PinHeader_2.54mm:PinHeader_1x01_P2.54mm_Vertical, F.Cu at (416.6, 94.0)
- J17: footprint Connector_PinHeader_2.54mm:PinHeader_1x05_P2.54mm_Vertical -> Connector_PinHeader_2.54mm:PinHeader_1x06_P2.54mm_Vertical
- SW1: value Arduino Reset -> SW_Push
- moved U2 268.6 mm to (273.3, 66.3)
- moved C3 3.60 mm to (338.5, 94.4)
- moved U1 3.60 mm to (328.4, 91.7)
- moved R5 3.60 mm to (302.6, 84.8)
- moved R6 3.60 mm to (305.7, 95.0)
- moved C4 3.60 mm to (333.5, 94.4)
- moved C5 3.60 mm to (325.1, 91.7)
- moved D1 3.60 mm to (321.8, 94.9)
- moved D4 3.60 mm to (286.5, 84.7)
- moved R2 3.60 mm to (315.5, 94.7)
- moved R4 3.60 mm to (289.7, 94.9)
- moved D2 3.60 mm to (312.3, 84.8)
- moved D3 3.60 mm to (296.0, 95.0)
- moved D5 3.60 mm to (299.3, 95.0)
- moved D6 3.60 mm to (308.9, 84.8)
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Connections:
- BAR1 pad 14: ~{SKIP} -> unconnected-(BAR1-K-Pad14)
- J17 pad 5: ~{WAS JSR} -> ~{SKIP}
- J9 pad 7: ~{SKIP} -> unconnected-(J9-Pin_7-Pad7)
Routing:
- net CLK FLOP: track 0.00 -> 343.5 mm, vias 0 -> 5
- net ~{SKIP}: track 194.9 -> 481.3 mm, vias 3 -> 5
- net ~{DATA0}: track 235.5 -> 375.2 mm, vias 0 -> 2
- net ~{DEFER}: track 517.1 -> 647.6 mm, vias 5 -> 8
- net ~{ION}: track 499.6 -> 616.6 mm, vias 3 -> 5
- net ~{CON DATA}: track 488.1 -> 596.1 mm, vias 5 -> 8
- net +5V: track 529.9 -> 622.2 mm, vias 2 -> 11
- net MB LOAD: track 543.4 -> 633.7 mm, vias 1 -> 2
- net ~{READ IO}: track 405.0 -> 489.0 mm, vias 0 -> 1
- net ~{MB CLEAR}: track 453.8 -> 536.8 mm, vias 1 -> 2
- net GND: track 497.0 -> 578.6 mm, vias 17 -> 18
- net ~{FETCH}: track 587.8 -> 666.8 mm
- net ~{READ1}: track 418.7 -> 490.7 mm, vias 0 -> 1
- net ~{READ2}: track 723.2 -> 659.3 mm, vias 6 -> 7
- net ~{DATA2}: track 498.2 -> 559.1 mm, vias 1 -> 2
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Other:
- board text added: "+5V OK"
- board text added: "CLK FLOP"
- board text added: "CLR"
- board text added: "CPU Option Outputs"
- board text added: "DATIA"
- board text added: "DATIB"
- board text added: "DATIC"
- board text added: "DATOA"
- board text added: "DATOB"
- board text added: "DATOC"
- board text added: "INTA"
- board text added: "INTP"
- board text added: "IO PLS"
- board text added: "IO RST"
- board text added: "LOAD IR"
- board text added: "STRT"
- board text added: "~{DIV}"
- board text added: "~{EXT LOAD}"
- board text added: "~{FORCE LOAD IR}"
- board text added: "~{INTR}"
- board text added: "~{LOAD AC}"
- board text added: "~{MD SEL1}"
- board text added: "~{MSKO}"
- board text added: "~{POWER FAIL}"
- board text added: "~{RQENB}"
- board text added: "~{SHIFT0}"
- board text added: "~{SHIFT1}"
- board text added: "~{SHIFT2}"
- board text added: "~{SHIFT3}"
- board text added: "~{TEST}"
- board text added: "~{WAS JSR}"
- board text added: "~{WHOA}"
- board text removed: "~{DS0} ~{DS1} ~{DS2} ~{DS3} ~{DS4} ~{DS5} DATIA DATIB DATIC DATOA DATOB DATOC STRT CLR IO PLS ~{SELB} ~{SELD}"

Commit message: yeah
Parts:
- moved U2 9.02 mm to (282.3, 66.5)
Routing:
- net ~{DATA3}: track 369.4 -> 440.3 mm
- net ~{DATA4}: track 328.6 -> 398.1 mm, vias 0 -> 1
- net ~{DATA5}: track 312.7 -> 381.7 mm, vias 1 -> 2
- net ~{DATA6}: track 472.5 -> 539.4 mm, vias 2 -> 3
- net ~{DATA7}: track 309.6 -> 374.6 mm, vias 1 -> 2
- net ~{DATA8}: track 251.6 -> 311.8 mm, vias 0 -> 1
- net ~{DATA15}: track 606.4 -> 611.6 mm
- net ~{DATA14}: track 236.1 -> 240.1 mm
- net ~{DATA13}: track 614.1 -> 617.9 mm
- net ~{DATA12}: track 318.2 -> 321.9 mm
- net ~{DATA9}: track 333.2 -> 336.1 mm
- net ~{DATA10}: track 376.0 -> 378.2 mm
- net ~{DATA11}: track 246.0 -> 248.1 mm
