File: DG Nova CPU Tester/Reverts/1.kicad_pcb (KiCad board)
At the start: 2 copper layers, 414.8 x 131.4 mm, 115 parts, among them J1 Front Panel Socket - Backside, J10 Programmed I/O, J11 CPU Option Inputs, J12 Data Channel, J13 Program Interrupt, J14 System Control, J15 Slot_02x50_Odd_Even, J16 Slot_02x50_Odd_Even, J17 CPU Option Outputs, J18 MEM Control Outputs, J19 Logic 8 CH, J20 Logic 8 CH, J21 Arduino Anolog Pins, J22 Arduino Digital Pins, J23 Arduino Digital Pins, J4 ATX-24, J5 Front Panel Card Edge, J6 MBO, J7 MEM, J8 Data Channel, J9 Front Panel Controls, SW1 SW_Push, U1 74HC14, U2 Pico

Commit message: All Traces Removed
Parts:
- removed BAR1, BAR15, BAR3, BAR5, BAR7, BAR8: LED Bar 10, Forgotten Machines:LED Bar 10
- removed BAR10, BAR16, BAR4, BAR6, BAR9: LED Bar 10, Forgotten Machines:LED Bar 6
- removed BAR11: LED Bar 10, Forgotten Machines:LED Bar 5
- removed BAR12: LED Bar 2, Forgotten Machines:LED Bar 2
- removed BAR13, BAR14: LED Bar 4, Forgotten Machines:LED Bar 4
- removed BAR2: LED Bar 10, Forgotten Machines:LED Bar 7
- removed D10, D11, D12, D13, D14, D15, D16, D17, D18, D19, D20, D21, D22, D23, D24, D25, D26, D27, D28, D7, D8, D9: LED, LED_THT:LED_D1.8mm_W3.3mm_H2.4mm
- removed J21: Arduino Anolog Pins, Connector_PinHeader_2.54mm:PinHeader_1x10_P2.54mm_Vertical
- removed J22, J23: Arduino Digital Pins, Connector_PinHeader_2.54mm:PinHeader_1x06_P2.54mm_Vertical
- removed R10, R11, R12, R13, R14, R15, R7, R8, R9: R_US, Resistor_THT:R_Axial_DIN0204_L3.6mm_D1.6mm_P5.08mm_Horizontal
- removed RN1, RN11, RN13, RN14, RN15, RN3, RN5, RN7, RN8: R_Network09_US, Resistor_THT:R_Array_SIP10
- removed RN10, RN16: R_Network05_US, Resistor_THT:R_Array_SIP6
- removed RN12: R_Network06_US, Resistor_THT:R_Array_SIP7
- removed RN2: R_Network08_US, Resistor_THT:R_Array_SIP9
- removed RN4, RN6, RN9: R_Network07_US, Resistor_THT:R_Array_SIP8
- removed TP2: ATX PWR_OK, Connector_PinHeader_2.54mm:PinHeader_1x01_P2.54mm_Vertical
- J10, J9: footprint Connector_PinHeader_2.54mm:PinHeader_1x17_P2.54mm_Vertical -> Connector_PinHeader_2.54mm:PinHeader_1x18_P2.54mm_Horizontal
- J11, J18: footprint Connector_PinHeader_2.54mm:PinHeader_1x10_P2.54mm_Vertical -> Connector_PinHeader_2.54mm:PinHeader_1x10_P2.54mm_Horizontal
- J12, J20: footprint Connector_PinHeader_2.54mm:PinHeader_1x08_P2.54mm_Vertical -> Connector_PinHeader_2.54mm:PinHeader_1x08_P2.54mm_Horizontal
- J13, J14: footprint Connector_PinHeader_2.54mm:PinHeader_1x04_P2.54mm_Vertical -> Connector_PinHeader_2.54mm:PinHeader_1x04_P2.54mm_Horizontal
- J17: footprint Connector_PinHeader_2.54mm:PinHeader_1x06_P2.54mm_Vertical -> Connector_PinHeader_2.54mm:PinHeader_1x06_P2.54mm_Horizontal
- J19: footprint Forgotten Machines:PinHeader_2x05_P2.54mm_Vertical - Backside -> Connector_PinHeader_2.54mm:PinHeader_2x05_P2.54mm_Vertical
- J6, J8: footprint Connector_PinHeader_2.54mm:PinHeader_1x16_P2.54mm_Vertical -> Connector_PinHeader_2.54mm:PinHeader_1x16_P2.54mm_Horizontal
- J7: footprint Connector_PinHeader_2.54mm:PinHeader_1x18_P2.54mm_Vertical -> Connector_PinHeader_2.54mm:PinHeader_1x18_P2.54mm_Horizontal
- moved FPIMAGE1 639.8 mm to (207.0, 70.6)
- moved JP2 441.9 mm to (61.0, 20.3)
- moved JP3 441.9 mm to (78.7, 20.3)
- moved TP1 437.2 mm to (101.6, 22.9)
- moved SW1 271.1 mm to (31.0, 20.3), turned to 0 degrees
- moved XA1 227.3 mm to (149.9, 81.3), turned to 0 degrees
- moved C3 227.1 mm to (353.1, 87.4)
- moved C4 223.0 mm to (353.1, 91.4), turned to 0 degrees
- moved C5 216.4 mm to (353.1, 95.5), turned to 0 degrees
- moved J6 214.8 mm to (294.6, 7.55)
- moved U2 204.6 mm to (323.9, 62.2), turned to 0 degrees
- moved J16 200.9 mm to (135.0, 107.3)
- moved R1 196.9 mm to (366.2, 86.4)
- moved D1 196.9 mm to (366.2, 83.2)
- moved J10 192.2 mm to (81.3, 7.62)
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Connections:
- J17 pad 5: ~{SKIP} -> ~{WAS JSR}
- J17 pad 6: ~{WAS JSR} -> unconnected-(J17-Pin_6-Pad6)
- J4 pad 14: -12v -> unconnected-(J4--12V-Pad14)
- J4 pad 20: -5V -> unconnected-(J4--5v-Pad20)
- J9 pad 3: ~{FETCH} -> ~{CARRY}
- J9 pad 4: ~{DEFER} -> ~{FETCH}
- J9 pad 5: ~{EXEC} -> ~{DEFER}
- J9 pad 6: ~{CARRY} -> ~{EXEC}
- J9 pad 7: unconnected-(J9-Pin_7-Pad7) -> ~{SKIP}
- XA1 pad A0: Net-(J21-Pin_10) -> unconnected-(XA1-PadA0)
- XA1 pad A1: Net-(J21-Pin_9) -> unconnected-(XA1-PadA1)
- XA1 pad A10: Net-(J21-Pin_6) -> unconnected-(XA1-PadA10)
- XA1 pad A11: Net-(J21-Pin_5) -> unconnected-(XA1-PadA11)
- XA1 pad A12: Net-(J21-Pin_4) -> unconnected-(XA1-PadA12)
- XA1 pad A13: Net-(J21-Pin_3) -> unconnected-(XA1-PadA13)
- XA1 pad A14: Net-(J21-Pin_2) -> unconnected-(XA1-PadA14)
- XA1 pad A15: Net-(J21-Pin_1) -> unconnected-(XA1-PadA15)
- XA1 pad A8: Net-(J21-Pin_8) -> unconnected-(XA1-PadA8)
- XA1 pad A9: Net-(J21-Pin_7) -> unconnected-(XA1-PadA9)
- XA1 pad D10: Net-(J23-Pin_3) -> unconnected-(XA1-PadD10)
- XA1 pad D11: Net-(J23-Pin_4) -> unconnected-(XA1-PadD11)
- XA1 pad D12: Net-(J23-Pin_5) -> unconnected-(XA1-PadD12)
- XA1 pad D13: Net-(J23-Pin_6) -> unconnected-(XA1-PadD13)
- XA1 pad D2: Net-(J22-Pin_1) -> unconnected-(XA1-D2_INT0-PadD2)
- XA1 pad D3: Net-(J22-Pin_2) -> unconnected-(XA1-D3_INT1-PadD3)
- XA1 pad D4: Net-(J22-Pin_3) -> unconnected-(XA1-PadD4)
- XA1 pad D5: Net-(J22-Pin_4) -> unconnected-(XA1-PadD5)
- XA1 pad D6: Net-(J22-Pin_5) -> unconnected-(XA1-PadD6)
- XA1 pad D7: Net-(J22-Pin_6) -> unconnected-(XA1-PadD7)
- XA1 pad D8: Net-(J23-Pin_1) -> unconnected-(XA1-PadD8)
- XA1 pad D9: Net-(J23-Pin_2) -> unconnected-(XA1-PadD9)
Routing:
- net GND After Meter: track 147.7 -> 0.00 mm
- net +5V: track 58.2 -> 0.00 mm
- net +12V Lamp: track 57.5 -> 0.00 mm
- net Net-(C4-Pad1): track 48.9 -> 0.00 mm
- net Net-(C3-Pad1): track 30.5 -> 0.00 mm
- net GND: track 27.7 -> 0.00 mm
- net Net-(C5-Pad1): track 27.2 -> 0.00 mm
- net ~{RST}: track 27.0 -> 0.00 mm
- net ~{PL}: track 27.0 -> 0.00 mm
- net ~{MEM9}: track 27.0 -> 0.00 mm
- net ~{MEM12}: track 27.0 -> 0.00 mm
- net ~{MBO9}: track 27.0 -> 0.00 mm
- net ~{MBO8}: track 27.0 -> 0.00 mm
- net ~{MBO7}: track 27.0 -> 0.00 mm
- net ~{MBO4}: track 27.0 -> 0.00 mm
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Other:
- board size 414.8 x 131.4 mm -> 16 x 114 mm
- board text added: "LEDs"
- board text removed: "+5V OK"
- board text removed: "1"
- board text removed: "10"
- board text removed: "11"
- board text removed: "12"
- board text removed: "13"
- board text removed: "14"
- board text removed: "2"
- board text removed: "3"
- board text removed: "4"
- board text removed: "5"
- board text removed: "6"
- board text removed: "7"
- board text removed: "8"
- board text removed: "9"
- board text removed: "A15 A14 A13 A12 A11 A10 A09 A08 A01 A00"
- board text removed: "Address ~{MBO}"
- board text removed: "Arduino Anolog Pins"
- board text removed: "Arduino Digital Pins"
- board text removed: "CLK FLOP"
- board text removed: "CLR"
- board text removed: "CPU Option Outputs"
- board text removed: "D02 D03 D04 D05 D06 D07"
- board text removed: "D08 D09 D10 D11 D12 D13"
- board text removed: "D53"
- board text removed: "DATIA"
- board text removed: "DATIB"
- board text removed: "DATIC"
- board text removed: "DATOA"
- board text removed: "DATOB"
- board text removed: "DATOC"
- board text removed: "DCHI"
- board text removed: "DCHO"
- board text removed: "DCHP"
- board text removed: "Data Channel"
- board text removed: "Data Channel ~{DATA}"
- board text removed: "Data ~{MEM}"
- board text removed: "Entrex Backplane S01B53 to S13B53"
- board text removed: "Front Panel Controls"
- board text removed: "INHIBIT"
- board text removed: "INTA"
- board text removed: "INTP"
- board text removed: "IO PLS"
- board text removed: "IO RST"
- board text removed: "LOAD IR"
- board text removed: "MB LOAD"
- board text removed: "MEM Control"
- board text removed: "MEM OK"
- board text removed: "OVFLO"
- board text removed: "RESTART ENABLE"
- board text removed: "Resistor Blocks Share Pin 1 Hole"
- board text removed: "STROBE"
- board text removed: "STRT"
- board text removed: "consider putting silkscreen borders for resistor blocks on the backside as well"
- board text removed: "~{CARRY}"
- board text removed: "~{CON DATA}"
- board text removed: "~{CON INST}"
- board text removed: "~{CON RQ}"
- board text removed: "~{CONT+ISTP+MSTP}"
- board text removed: "~{DATA0}"
- board text removed: "~{DATA15}"
- board text removed: "~{DCHA}"
- board text removed: "~{DCHM0}"
- board text removed: "~{DCHM1}"
- board text removed: "~{DCHR}"
- board text removed: "~{DEFER}"
- board text removed: "~{DIV}"
- board text removed: "~{DRIVE IO}"
- board text removed: "~{DS0}"
- board text removed: "~{DS1}"
- board text removed: "~{DS2}"
- board text removed: "~{DS3}"
- board text removed: "~{DS4}"
- board text removed: "~{DS5}"
- board text removed: "~{EXEC}"
- board text removed: "~{EXT LOAD}"
- board text removed: "~{FETCH}"
- board text removed: "~{FORCE LOAD IR}"
- board text removed: "~{INH TRANS}"
- board text removed: "~{INTR}"
- board text removed: "~{ION}"
- board text removed: "~{ISTP}"
- board text removed: "~{LOAD AC}"
- board text removed: "~{MA LOAD}"
- board text removed: "~{MB CLEAR}"
- board text removed: "~{MBO0}"
- board text removed: "~{MBO15}"
- board text removed: "~{MD SEL1}"
- board text removed: "~{MEM0}"
- board text removed: "~{MEM15}"
- board text removed: "~{MSKO}"
- board text removed: "~{MSTP}"
- board text removed: "~{PL}"
- board text removed: "~{POWER FAIL}"
- board text removed: "~{READ IO}"
- board text removed: "~{READ1}"
- board text removed: "~{READ2}"
- board text removed: "~{RQENB}"
- board text removed: "~{RST}"
- board text removed: "~{RUN}"
- board text removed: "~{SELB}"
- board text removed: "~{SELD}"
- board text removed: "~{SHIFT0}"
- board text removed: "~{SHIFT1}"
- board text removed: "~{SHIFT2}"
- board text removed: "~{SHIFT3}"
- board text removed: "~{SKIP}"
- board text removed: "~{STOP}"
- board text removed: "~{TEST}"
- board text removed: "~{TRY ME}"
- board text removed: "~{WAS JSR}"
- board text removed: "~{WHOA}"
