File: DG Nova CPU Tester/Reverts/3.kicad_pcb (KiCad board)
At the start: 2 copper layers, 414.8 x 131.4 mm, 115 parts, among them J1 Front Panel Socket - Backside, J10 Programmed I/O, J11 CPU Option Inputs, J12 Data Channel, J13 Program Interrupt, J14 System Control, J15 Slot_02x50_Odd_Even, J16 Slot_02x50_Odd_Even, J17 CPU Option Outputs, J18 MEM Control Outputs, J19 Logic 8 CH, J20 Logic 8 CH, J21 Arduino Anolog Pins, J22 Arduino Digital Pins, J23 Arduino Digital Pins, J4 ATX-24, J5 Front Panel Card Edge, J6 MBO, J7 MEM, J8 Data Channel, J9 Front Panel Controls, SW1 SW_Push, U1 74HC14, U2 Pico

Commit message: All Traces Removed
Parts:
- removed BAR10, BAR16, BAR9: LED Bar 10, Forgotten Machines:LED Bar 6
- removed BAR11: LED Bar 10, Forgotten Machines:LED Bar 5
- removed BAR12: LED Bar 2, Forgotten Machines:LED Bar 2
- removed BAR13, BAR14: LED Bar 4, Forgotten Machines:LED Bar 4
- removed BAR15, BAR8: LED Bar 10, Forgotten Machines:LED Bar 10
- removed D10, D11, D12, D13, D14, D15, D16, D17, D18, D19, D20, D21, D22, D23, D24, D25, D26, D27, D28, D9: LED, LED_THT:LED_D1.8mm_W3.3mm_H2.4mm
- removed J21: Arduino Anolog Pins, Connector_PinHeader_2.54mm:PinHeader_1x10_P2.54mm_Vertical
- removed J22, J23: Arduino Digital Pins, Connector_PinHeader_2.54mm:PinHeader_1x06_P2.54mm_Vertical
- removed R10, R11, R12, R13, R14, R15, R9: R_US, Resistor_THT:R_Axial_DIN0204_L3.6mm_D1.6mm_P5.08mm_Horizontal
- removed RN10, RN16: R_Network05_US, Resistor_THT:R_Array_SIP6
- removed RN11, RN13, RN14, RN15, RN8: R_Network09_US, Resistor_THT:R_Array_SIP10
- removed RN12: R_Network06_US, Resistor_THT:R_Array_SIP7
- removed RN9: R_Network07_US, Resistor_THT:R_Array_SIP8
- removed TP2: ATX PWR_OK, Connector_PinHeader_2.54mm:PinHeader_1x01_P2.54mm_Vertical
- J10: value Programmed I/O -> Front Panel Controls
- J17: footprint Connector_PinHeader_2.54mm:PinHeader_1x06_P2.54mm_Vertical -> Connector_PinHeader_2.54mm:PinHeader_1x05_P2.54mm_Vertical
- moved JP2 425.8 mm to (73.0, 56.5)
- moved JP3 425.8 mm to (90.8, 56.5)
- moved TP1 419.1 mm to (113.7, 59.1)
- moved SW1 269.2 mm to (48.3, 51.4), turned to 0 degrees
- moved XA1 244.5 mm to (152.0, 107.3), turned to 0 degrees
- moved C3 228.9 mm to (355.6, 105.8)
- moved C4 225.3 mm to (355.6, 109.9), turned to 0 degrees
- moved C5 219.4 mm to (355.6, 113.9), turned to 0 degrees
- moved U2 210.3 mm to (326.4, 80.6), turned to 0 degrees
- moved R1 200.3 mm to (368.8, 104.8)
- moved D1 198.9 mm to (368.7, 101.6)
- moved R2 193.5 mm to (372.9, 114.9)
- moved D2 189.2 mm to (373.0, 101.6), turned to 90 degrees
- moved U1 179.5 mm to (396.2, 99.7), turned to 0 degrees
- moved R5 174.9 mm to (385.1, 114.9), turned to 90 degrees
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Connections:
- BAR1 pad 14: unconnected-(BAR1-K-Pad14) -> ~{SKIP}
- BAR7 pad 10: Net-(RN7-R9) -> unconnected-(BAR7-Pad10)
- BAR7 pad 11: ~{INH TRANS} -> unconnected-(BAR7-K-Pad11)
- BAR7 pad 9: unconnected-(BAR7-Pad9) -> Net-(RN7-R9)
- J17 pad 5: ~{SKIP} -> ~{WAS JSR}
- J4 pad 14: -12v -> unconnected-(J4--12V-Pad14)
- J4 pad 20: -5V -> unconnected-(J4--5v-Pad20)
- J9 pad 7: unconnected-(J9-Pin_7-Pad7) -> ~{SKIP}
- XA1 pad A0: Net-(J21-Pin_10) -> unconnected-(XA1-PadA0)
- XA1 pad A1: Net-(J21-Pin_9) -> unconnected-(XA1-PadA1)
- XA1 pad A10: Net-(J21-Pin_6) -> unconnected-(XA1-PadA10)
- XA1 pad A11: Net-(J21-Pin_5) -> unconnected-(XA1-PadA11)
- XA1 pad A12: Net-(J21-Pin_4) -> unconnected-(XA1-PadA12)
- XA1 pad A13: Net-(J21-Pin_3) -> unconnected-(XA1-PadA13)
- XA1 pad A14: Net-(J21-Pin_2) -> unconnected-(XA1-PadA14)
- XA1 pad A15: Net-(J21-Pin_1) -> unconnected-(XA1-PadA15)
- XA1 pad A8: Net-(J21-Pin_8) -> unconnected-(XA1-PadA8)
- XA1 pad A9: Net-(J21-Pin_7) -> unconnected-(XA1-PadA9)
- XA1 pad D10: Net-(J23-Pin_3) -> unconnected-(XA1-PadD10)
- XA1 pad D11: Net-(J23-Pin_4) -> unconnected-(XA1-PadD11)
- XA1 pad D12: Net-(J23-Pin_5) -> unconnected-(XA1-PadD12)
- XA1 pad D13: Net-(J23-Pin_6) -> unconnected-(XA1-PadD13)
- XA1 pad D2: Net-(J22-Pin_1) -> unconnected-(XA1-D2_INT0-PadD2)
- XA1 pad D3: Net-(J22-Pin_2) -> unconnected-(XA1-D3_INT1-PadD3)
- XA1 pad D4: Net-(J22-Pin_3) -> unconnected-(XA1-PadD4)
- XA1 pad D5: Net-(J22-Pin_4) -> unconnected-(XA1-PadD5)
- XA1 pad D6: Net-(J22-Pin_5) -> unconnected-(XA1-PadD6)
- XA1 pad D7: Net-(J22-Pin_6) -> unconnected-(XA1-PadD7)
- XA1 pad D8: Net-(J23-Pin_1) -> unconnected-(XA1-PadD8)
- XA1 pad D9: Net-(J23-Pin_2) -> unconnected-(XA1-PadD9)
Routing:
- net ~{MSKO}: track 3.43 -> 242.5 mm
- net ~{DATA0}: track 3.43 -> 235.5 mm
- net INTA: track 2.92 -> 234.0 mm
- net ~{DATA8}: track 3.43 -> 228.8 mm
- net DATIB: track 2.92 -> 227.3 mm
- net ~{DATA11}: track 3.43 -> 222.1 mm
- net DATIA: track 2.92 -> 220.6 mm
- net ~{DATA14}: track 3.43 -> 215.3 mm
- net ~{DS3}: track 3.43 -> 213.8 mm
- net DATOC: track 2.92 -> 207.1 mm
- net CLR: track 2.92 -> 200.9 mm
- net DATIC: track 2.92 -> 197.9 mm
- net STRT: track 2.92 -> 194.6 mm
- net DATOB: track 2.92 -> 190.9 mm
- net ~{INH TRANS}: track 3.43 -> 185.7 mm
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Other:
- board text added: "MEM Control Outputs"
- board text removed: "+5V OK"
- board text removed: "A15 A14 A13 A12 A11 A10 A09 A08 A01 A00"
- board text removed: "Arduino Anolog Pins"
- board text removed: "Arduino Digital Pins"
- board text removed: "CLK FLOP"
- board text removed: "CLR"
- board text removed: "CPU Option Outputs"
- board text removed: "D02 D03 D04 D05 D06 D07"
- board text removed: "D08 D09 D10 D11 D12 D13"
- board text removed: "D53"
- board text removed: "DATIA"
- board text removed: "DATIB"
- board text removed: "DATIC"
- board text removed: "DATOA"
- board text removed: "DATOB"
- board text removed: "DATOC"
- board text removed: "DCHI"
- board text removed: "DCHO"
- board text removed: "DCHP"
- board text removed: "Entrex Backplane S01B53 to S13B53"
- board text removed: "INHIBIT"
- board text removed: "INTA"
- board text removed: "INTP"
- board text removed: "IO PLS"
- board text removed: "IO RST"
- board text removed: "LOAD IR"
- board text removed: "MB LOAD"
- board text removed: "MEM Control"
- board text removed: "OVFLO"
- board text removed: "STROBE"
- board text removed: "STRT"
- board text removed: "~{CARRY}"
- board text removed: "~{CON DATA}"
- board text removed: "~{CON INST}"
- board text removed: "~{CON RQ}"
- board text removed: "~{CONT+ISTP+MSTP}"
- board text removed: "~{DCHA}"
- board text removed: "~{DCHM0}"
- board text removed: "~{DCHM1}"
- board text removed: "~{DCHR}"
- board text removed: "~{DEFER}"
- board text removed: "~{DIV}"
- board text removed: "~{DRIVE IO}"
- board text removed: "~{DS0}"
- board text removed: "~{DS1}"
- board text removed: "~{DS2}"
- board text removed: "~{DS3}"
- board text removed: "~{DS4}"
- board text removed: "~{DS5}"
- board text removed: "~{EXEC}"
- board text removed: "~{EXT LOAD}"
- board text removed: "~{FORCE LOAD IR}"
- board text removed: "~{INH TRANS}"
- board text removed: "~{INTR}"
- board text removed: "~{ISTP}"
- board text removed: "~{LOAD AC}"
- board text removed: "~{MA LOAD}"
- board text removed: "~{MB CLEAR}"
- board text removed: "~{MD SEL1}"
- board text removed: "~{MSKO}"
- board text removed: "~{MSTP}"
- board text removed: "~{PL}"
- board text removed: "~{POWER FAIL}"
- board text removed: "~{READ IO}"
- board text removed: "~{READ1}"
- board text removed: "~{READ2}"
- board text removed: "~{RQENB}"
- board text removed: "~{RST}"
- board text removed: "~{SELB}"
- board text removed: "~{SELD}"
- board text removed: "~{SHIFT0}"
- board text removed: "~{SHIFT1}"
- board text removed: "~{SHIFT2}"
- board text removed: "~{SHIFT3}"
- board text removed: "~{SKIP}"
- board text removed: "~{STOP}"
- board text removed: "~{TEST}"
- board text removed: "~{WAS JSR}"
- board text removed: "~{WHOA}"
