File: DG Nova CPU Tester/Reverts/Before Track Delete.kicad_pcb (KiCad board)
At the start: 2 copper layers, 414.8 x 131.4 mm, 115 parts, among them J1 Front Panel Socket - Backside, J10 Programmed I/O, J11 CPU Option Inputs, J12 Data Channel, J13 Program Interrupt, J14 System Control, J15 Slot_02x50_Odd_Even, J16 Slot_02x50_Odd_Even, J17 CPU Option Outputs, J18 MEM Control Outputs, J19 Logic 8 CH, J20 Logic 8 CH, J21 Arduino Anolog Pins, J22 Arduino Digital Pins, J23 Arduino Digital Pins, J4 ATX-24, J5 Front Panel Card Edge, J6 MBO, J7 MEM, J8 Data Channel, J9 Front Panel Controls, SW1 SW_Push, U1 74HC14, U2 Pico

Commit message: All Traces Removed
Parts:
- moved TP1 440.4 mm to (88.6, 105.3)
- moved D3 242.7 mm to (296.0, 95.0)
- moved D4 242.7 mm to (286.5, 84.7)
- moved D5 242.7 mm to (299.3, 95.0)
- moved D6 242.7 mm to (308.9, 84.8)
- moved R1 242.7 mm to (318.6, 84.5)
- moved R3 242.7 mm to (292.8, 84.8)
- moved C4 242.7 mm to (333.5, 94.4)
- moved C5 242.7 mm to (325.1, 91.7)
- moved D1 242.7 mm to (321.8, 94.9)
- moved D2 242.7 mm to (312.3, 84.8)
- moved R4 242.7 mm to (289.7, 94.9)
- moved U1 242.7 mm to (328.4, 91.7)
- moved C3 242.7 mm to (338.5, 94.4)
- moved R2 242.7 mm to (315.5, 94.7)
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Routing:
- net ~{MEM1}: track 19.7 -> 1029.8 mm, vias 0 -> 2
- net ~{MBO1}: track 27.0 -> 809.2 mm, vias 0 -> 6
- net ~{MEM14}: track 27.0 -> 768.9 mm, vias 0 -> 5
- net ~{MEM3}: track 19.7 -> 759.8 mm, vias 0 -> 6
- net ~{MEM0}: track 18.7 -> 735.0 mm, vias 0 -> 3
- net ~{DATA6}: track 3.43 -> 696.2 mm, vias 0 -> 4
- net ~{MEM2}: track 27.0 -> 711.9 mm, vias 0 -> 3
- net ~{MBO0}: track 3.43 -> 687.6 mm, vias 0 -> 1
- net ~{EXT LOAD}: track 3.56 -> 681.2 mm, vias 0 -> 5
- net ~{MSTP}: track 19.7 -> 688.1 mm, vias 0 -> 4
- net ~{DRIVE IO}: track 3.43 -> 659.4 mm, vias 0 -> 7
- net ~{READ2}: track 3.43 -> 659.3 mm, vias 0 -> 7
- net ~{FETCH}: track 20.2 -> 666.8 mm, vias 0 -> 7
- net MB LOAD: track 2.92 -> 633.7 mm, vias 0 -> 2
- net ~{DEFER}: track 19.7 -> 647.6 mm, vias 0 -> 8
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