File: DG Nova CPU Tester/Reverts/Arduino Placed - right before undoing Front Panel Connectors.kicad_pcb (KiCad board)
At the start: 2 copper layers, 414.8 x 131.4 mm, 115 parts, among them J1 Front Panel Socket - Backside, J10 Programmed I/O, J11 CPU Option Inputs, J12 Data Channel, J13 Program Interrupt, J14 System Control, J15 Slot_02x50_Odd_Even, J16 Slot_02x50_Odd_Even, J17 CPU Option Outputs, J18 MEM Control Outputs, J19 Logic 8 CH, J20 Logic 8 CH, J21 Arduino Anolog Pins, J22 Arduino Digital Pins, J23 Arduino Digital Pins, J4 ATX-24, J5 Front Panel Card Edge, J6 MBO, J7 MEM, J8 Data Channel, J9 Front Panel Controls, SW1 SW_Push, U1 74HC14, U2 Pico

Commit message: Intense
Routing:
- net ~{CONT+ISTP+MSTP}: track 458.2 -> 194.8 mm
- net ~{CON DATA}: track 464.4 -> 201.8 mm, vias 2 -> 3
- net ~{STOP}: track 397.9 -> 177.8 mm, vias 2 -> 1
- net ~{CARRY}: track 402.8 -> 197.4 mm
- net ~{ION}: track 416.2 -> 211.2 mm, vias 1 -> 0
- net ~{RUN}: track 415.9 -> 214.9 mm, vias 1 -> 0
- net ~{ISTP}: track 106.3 -> 223.7 mm, vias 0 -> 1
- net ~{MBO11}: track 314.8 -> 200.4 mm, vias 3 -> 0
- net ~{PL}: track 104.4 -> 218.1 mm, vias 0 -> 2
- net ~{MSTP}: track 102.6 -> 214.5 mm, vias 0 -> 2
- net ~{MEM6}: track 348.2 -> 242.2 mm, vias 2 -> 1
- net RESTART ENABLE: track 106.8 -> 207.6 mm, vias 0 -> 1
- net ~{MEM7}: track 341.3 -> 243.5 mm, vias 2 -> 1
- net ~{MEM4}: track 351.6 -> 258.4 mm, vias 2 -> 1
- net ~{MEM5}: track 344.1 -> 251.8 mm, vias 2 -> 1
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