File: Quantx-DG-Nova-1200-CPU/DG Nova 1200 CPU.kicad_sch (KiCad schematic)
At the start: 241 parts, among them Q1 MPS3640, U1 74LS122, U10 74LS20, U100 045, U101 74LS04, U102 74LS179, U103 74LS179, U105 74LS179, U106 74LS179, U107 74LS179, U108 74LS179, U109 74LS00, U11 74LS03, U110 74LS20, U111 74LS10, U112 74LS51, U113 74LS114, U114 74LS51, U115 74LS179, U116 74LS157, U117 74LS181, U118 74LS00, U119 74LS170, U12 74LS00, U120 8264, U121 74LS157, U122 74LS179, U123 8225, U124 8225, U125 8264, U13 045, U14 74LS20, U15 74LS20, U16 74LS04, U17 74LS179, U18 74LS20, U19 74LS00, U2 74LS74, U20 74LS74, U21 74LS00, U22 74LS04, U23 74LS179, U24 74LS51, U25 74LS139, U26 74LS04, U27 74LS04, U28 74LS179, U29 74LS179, U3 74LS00, U30 82S23, U31 82S23, U32 74LS179, U33 74LS179, U34 045, U35 74LS10, U36 74LS00, U37 74LS179, U38 74LS179, U39 74LS179, U4 045, U40 74LS179, U41 045, U42 74LS179, U43 74H54, U44 74LS51, U45 74LS51, U46 74H54, U47 74H54, U48 045, U49 74LS03, U5 74LS04, U50 74LS10, U51 74LS139, U52 74LS139, U53 045, U54 74LS179, U55 74LS51, U56 74LS20, U57 74LS00, U58 045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

Commit message: QuantX schematic update
Parts:
- added C?: 220pf, symbol Device:C_Small
Connections:
- net GNDREF: now also C?.2
- net at U118.6, U119.15 (D1): now also C?.1
