File: Quantx-DG-Nova-1200-CPU/DG Nova 1200 CPU.kicad_sch (KiCad schematic)
At the start: 242 parts, among them Q1 MPS3640, U1 74LS122, U10 74LS20, U100 045, U101 74LS04, U102 74LS179, U103 74LS179, U105 74LS179, U106 74LS179, U107 74LS179, U108 74LS179, U109 74LS00, U11 74LS03, U110 74LS20, U111 74LS10, U112 74LS51, U113 74LS114, U114 74LS51, U115 74LS179, U116 74LS157, U117 74LS181, U118 74LS00, U119 74LS170, U12 74LS00, U120 8264, U121 74LS157, U122 74LS179, U123 8225, U124 8225, U125 8264, U13 045, U14 74LS20, U15 74LS20, U16 74LS04, U17 74LS179, U18 74LS20, U19 74LS00, U2 74LS74, U20 74LS74, U21 74LS00, U22 74LS04, U23 74LS179, U24 74LS51, U25 74LS139, U26 74LS04, U27 74LS04, U28 74LS179, U29 74LS179, U3 74LS00, U30 82S23, U31 82S23, U32 74LS179, U33 74LS179, U34 045, U35 74LS10, U36 74LS00, U37 74LS179, U38 74LS179, U39 74LS179, U4 045, U40 74LS179, U41 045, U42 74LS179, U43 74H54, U44 74LS51, U45 74LS51, U46 74H54, U47 74H54, U48 045, U49 74LS03, U5 74LS04, U50 74LS10, U51 74LS139, U52 74LS139, U53 045, U54 74LS179, U55 74LS51, U56 74LS20, U57 74LS00, U58 045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

Commit message: updates
Parts:
- added U104: 8271, Package_DIP:DIP-16_W7.62mm, symbol ForgottenMachines:8271
Other:
- note added: "KEY Output"
- note added: "Signetics N8271"
- note added: "~{LOOP} Output"
Changed lines of the file:
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@@
     )
   )
+  (text "~{LOOP} Output" (at 626.745 18.415 0)
+    (effects (font (size 5 5) (thickness 1) bold (color 255 0 0 1)) (justify left bottom))
+  )
   (text "These were labeled as\nPTG0•TS0 and ~{PTG0•TS0}" (at 160.02 153.67 0)
     (effects (font (size 1.27 1.27)) (justify left bottom))
@@
     (effects (font (size 1.27 1.27)) (justify left bottom))
   )
+  (text "Signetics\nN8271" (at 137.795 89.535 0)
+    (effects (font (size 1.27 1.27) (thickness 0.254) bold) (justify left bottom))
+  )
   (text "Program Load Option" (at 731.52 447.04 0)
     (effects (font (size 1.27 1.27)) (justify left bottom))
@@
     (effects (font (size 1.27 1.27)) (justify left bottom))
   )
+  (text "KEY Output" (at 109.22 83.82 0)
+    (effects (font (size 5 5) (thickness 1) bold (color 255 0 0 1)) (justify left bottom))
+  )
   (text "Jumpers are set for REV 107-000083-02 (1970)" (at 744.22 518.16 0)
     (effects (font (size 1.27 1.27)) (justify left bottom))
@@
     )
   )
+  (symbol (lib_id "ForgottenMachines:8271") (at -67.945 46.99 0) (unit 2)
+    (in_bom yes) (on_board yes) (dnp no) (fields_autoplaced)
+    (property "Reference" "U104" (at -59.69 46.355 0)
+      (effects (font (size 1.27 1.27)) (justify left))
+    )
+    (property "Value" "8271" (at -59.69 48.895 0)
+      (effects (font (size 1.27 1.27)) (justify left))
+    )
+    (property "Footprint" "Package_DIP:DIP-16_W7.62mm" (at -110.49 18.415 0)
+      (effects (font (size 1.27 1.27)) hide)
+    )
+    (property "Datasheet" "https://github.com/ForgottenMachines/Universal-9-Track-Reader/blob/main/8271%20Datasheet.pdf" (at -106.045 5.08 0)
+      (effects (font (size 1.27 1.27)) hide)
+    )
+    (pin "8")
+    (pin "1")
+    (pin "15")
+    (pin "10")
+    (pin "4")
+    (pin "14")
+    (pin "13")
+    (pin "2")
+    (pin "12")
+    (pin "11")
+    (pin "16")
+    (pin "7")
+    (pin "3")
+    (pin "6")
+    (pin "5")
+    (pin "9")
+    (instances
+      (project "DG Nova 1200 CPU"
+        (path "/77a6f450-7f0b-4119-87aa-c085c3b42cb7"
+          (reference "U104") (unit 2)
+        )
+      )
+    )
+  )
   (symbol (lib_id "power:+5V") (at 25.4 316.23 90) (mirror x) (unit 1)
     (in_bom yes) (on_board yes) (dnp no) (fields_autoplaced)
@@
         )
       )
+    )
+  )
+  (symbol (lib_id "ForgottenMachines:8271") (at -34.29 45.72 0) (unit 1)
+    (in_bom yes) (on_board yes) (dnp no) (fields_autoplaced)
+    (property "Reference" "U104" (at -32.0959 68.58 0)
+      (effects (font (size 1.27 1.27)) (justify left))
+    )
+    (property "Value" "8271" (at -32.0959 71.12 0)
+      (effects (font (size 1.27 1.27)) (justify left))
+    )
+    (property "Footprint" "Package_DIP:DIP-16_W7.62mm" (at -76.835 17.145 0)
+      (effects (font (size 1.27 1.27)) hide)
+    )
+    (property "Datasheet" "https://github.com/ForgottenMachines/Universal-9-Track-Reader/blob/main/8271%20Datasheet.pdf" (at -72.39 3.81 0)
+      (effects (font (size 1.27 1.27)) hide)
+    )
+    (pin "8")
+    (pin "1")
+    (pin "15")
+    (pin "10")
+    (pin "4")
+    (pin "14")
+    (pin "13")
+    (pin "2")
+    (pin "12")
+    (pin "11")
+    (pin "16")
+    (pin "7")
+    (pin "3")
+    (pin "6")
+    (pin "5")
+    (pin "9")
+    (instances
+      (project "DG Nova 1200 CPU"
+        (path "/77a6f450-7f0b-4119-87aa-c085c3b42cb7"
+          (reference "U104") (unit 1)
+        )
+      )
