File: Quantx-DG-Nova-1200-CPU/DG Nova 1200 CPU - CON_RQ to CON_INST extract.kicad_sch (KiCad schematic)
At the start: 36 parts, among them U101 74LS04, U103 74LS179, U2 74LS74, U21 74LS00, U22 74LS04, U23 74LS179, U24 74LS51, U3 74LS00, U34 045, U36 74LS00, U4 045, U41 045, U43 74H54, U55 74LS51, U6 74LS00, U62 74LS10, U70 045, U82 74LS00, U83 74LS04, U84 74LS20, U85 045, U86 74LS00, U87 74LS00, U89 74LS20, U92 74LS00, U99 74LS20

Commit message: yikes
Parts:
- renumbered U36 to U37
Connections:
- net TP1: now reaches U21.3, U21.4, U43.4
- net TP2: now reaches U23.2 (B), U41.6
Other:
- moved on the sheet: R3, R73, U24A
