File: DG Nova CPU Tester/Piggyback MEM0-7/Piggyback MEM0-7.kicad_pcb (KiCad board)
At the start: 2 copper layers, 59.6 x 62 mm, 4 parts, among them J1 Conn_02x18_Odd_Even, J3 Conn_01x17, U2 74LS08, U3 74LS08

Commit message: yeah
Parts:
- added C1: CAP_Disc_Common_-_Entrex_Trapezoid, Forgotten Machines:Disc Capacitor Common Entrex Trapezoid, F.Cu at (67.5, 42.0)
- added C2: CAP_Disc_Common_-_Entrex_Trapezoid, Forgotten Machines:Disc Capacitor Common Entrex Trapezoid, F.Cu at (46.7, 41.9)
Routing:
- net +5V: track 8.89 -> 5.46 mm, vias 3 -> 2
- net ~{CON INST}: track 76.3 -> 74.9 mm
- net ~{MEM2}: track 50.8 -> 52.1 mm
- net ~{MEM1}: track 29.8 -> 31.0 mm
Other:
- board size 59.6 x 62 mm -> 59.6 x 58 mm
- board text added: "74xx08"
- board text added: "Nova 1200 CPU Tester Arduino Mega MEM0 - MEM7 Output Manager"

Commit message: more
Routing:
- net A13: track 0.00 -> 8.99 mm
Other:
- board size 59.6 x 58 mm -> 55.4 x 57 mm
- board text added: "74xx38"
- board text removed: "74xx08"
Changed lines of the file:
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@@
   (gr_line (start 46.228 36.068) (end 43.688 36.068)
     (stroke (width 0.1) (type default)) (layer "Dwgs.User"))
-  (gr_rect (start 50.038 55.499) (end 93.726 90.678)
+  (gr_rect (start 50.038 55.499) (end 89.535 90.678)
     (stroke (width 0.1) (type default)) (fill none) (layer "Edge.Cuts"))
-  (gr_rect (start 34.163 32.639) (end 93.726 90.678)
+  (gr_rect (start 34.163 33.655) (end 89.535 90.678)
     (stroke (width 0.1) (type default)) (fill none) (layer "Edge.Cuts"))
-  (gr_text "74xx08" (at 79.883 43.815) (layer "F.SilkS")
+  (gr_text "74xx38" (at 79.883 43.815) (layer "F.SilkS")
     (effects (font (size 1 1) (thickness 0.15)) (justify left bottom))
   )
-  (gr_text "74xx08" (at 58.674 43.815) (layer "F.SilkS")
+  (gr_text "74xx38" (at 58.674 43.815) (layer "F.SilkS")
     (effects (font (size 1 1) (thickness 0.15)) (justify left bottom))
   )
@@
   (segment (start 48.768 36.068) (end 50.165 37.465) (width 0.25) (layer "B.Cu") (net 36))
   (segment (start 50.165 37.465) (end 50.165 40.107991) (width 0.25) (layer "B.Cu") (net 36))
+  (segment (start 57.803 38.245) (end 58.928 39.37) (width 0.25) (layer "B.Cu") (net 37))
+  (segment (start 51.308 36.068) (end 53.485 38.245) (width 0.25) (layer "B.Cu") (net 37))
+  (segment (start 53.485 38.245) (end 57.803 38.245) (width 0.25) (layer "B.Cu") (net 37))
   (segment (start 51.308 38.608) (end 51.308 39.37) (width 0.25) (layer "F.Cu") (net 38))
   (segment (start 53.848 36.068) (end 51.308 38.608) (width 0.25) (layer "F.Cu") (net 38))

Commit message: m
Other:
- board text added: "74xx32"
- board text removed: "74xx38"
Changed lines of the file:
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@@
   (gr_rect (start 34.163 33.655) (end 89.535 90.678)
     (stroke (width 0.1) (type default)) (fill none) (layer "Edge.Cuts"))
-  (gr_text "74xx38" (at 79.883 43.815) (layer "F.SilkS")
+  (gr_text "74xx32" (at 79.883 43.815) (layer "F.SilkS")
     (effects (font (size 1 1) (thickness 0.15)) (justify left bottom))
   )
-  (gr_text "74xx38" (at 58.674 43.815) (layer "F.SilkS")
+  (gr_text "74xx32" (at 58.674 43.815) (layer "F.SilkS")
     (effects (font (size 1 1) (thickness 0.15)) (justify left bottom))
   )

Commit message: 74LS32
Parts:
- removed U3: 74LS08, Package_DIP:DIP-14_W7.62mm
- added U1: 74LS32, Package_DIP:DIP-14_W7.62mm, F.Cu at (48.8, 47.0)
- U2: value 74LS08 -> 74LS32
- moved U2 21.7 mm to (70.5, 47.0)
Connections:
- U2 pad 10: A13 -> A09
- U2 pad 11: ~{MEM3} -> ~{MEM7}
- U2 pad 13: A12 -> A08
- U2 pad 2: A15 -> A11
- U2 pad 3: ~{MEM0} -> ~{MEM4}
- U2 pad 5: A14 -> A10
- U2 pad 6: ~{MEM1} -> ~{MEM5}
- U2 pad 8: ~{MEM2} -> ~{MEM6}
Changed lines of the file:
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@@
   (net 51 "A00")
   (footprint "Package_DIP:DIP-14_W7.62mm" (layer "F.Cu")
-    (at 70.485 46.99 90)
+    (at 48.768 46.99 90)
     (descr "14-lead though-hole mounted DIP package, row spacing 7.62 mm (300 mils)")
     (tags "THT DIP DIL PDIP 2.54mm 7.62mm 300mil")
     (property "Sheetfile" "Piggyback MEM0-7.kicad_sch")
     (property "Sheetname" "")
-    (property "ki_description" "Quad And2")
-    (property "ki_keywords" "TTL and2")
-    (attr through_hole)
-    (fp_text reference "U3" (at 3.81 -2.33 90) (layer "F.SilkS") hide
-        (effects (font (size 1 1) (thickness 0.15)))
-    )
-    (fp_text value "74LS08" (at 3.81 17.57 90) (layer "F.Fab")
+    (property "ki_description" "Quad 2-input OR")
+    (property "ki_keywords" "TTL Or2")
+    (attr through_hole)
+    (fp_text reference "U1" (at 3.81 -2.33 90) (layer "F.SilkS")
+        (effects (font (size 1 1) (thickness 0.15)))
+    )
+    (fp_text value "74LS32" (at 3.81 17.57 90) (layer "F.Fab")
         (effects (font (size 1 1) (thickness 0.15)))
     )
@@
       (net 47 "~{CON INST}") (pintype "input"))
     (pad "2" thru_hole oval (at 0 2.54 90) (size 1.6 1.6) (drill 0.8) (layers "*.Cu" "*.Mask")
-      (net 39 "A11") (pintype "input"))
+      (net 35 "A15") (pintype "input"))
     (pad "3" thru_hole oval (at 0 5.08 90) (size 1.6 1.6) (drill 0.8) (layers "*.Cu" "*.Mask")
-      (net 18 "~{MEM4}") (pintype "output"))
+      (net 22 "~{MEM0}") (pintype "output"))
     (pad "4" thru_hole oval (at 0 7.62 90) (size 1.6 1.6) (drill 0.8) (layers "*.Cu" "*.Mask")
       (net 47 "~{CON INST}") (pintype "input"))
     (pad "5" thru_hole oval (at 0 10.16 90) (size 1.6 1.6) (drill 0.8) (layers "*.Cu" "*.Mask")
-      (net 40 "A10") (pintype "input"))
+      (net 36 "A14") (pintype "input"))
     (pad "6" thru_hole oval (at 0 12.7 90) (size 1.6 1.6) (drill 0.8) (layers "*.Cu" "*.Mask")
-      (net 17 "~{MEM5}") (pintype "output"))
+      (net 21 "~{MEM1}") (pintype "output"))
     (pad "7" thru_hole oval (at 0 15.24 90) (size 1.6 1.6) (drill 0.8) (layers "*.Cu" "*.Mask")
       (net 1 "GND") (pinfunction "GND") (pintype "power_in"))
     (pad "8" thru_hole oval (at 7.62 15.24 90) (size 1.6 1.6) (drill 0.8) (layers "*.Cu" "*.Mask")
-      (net 16 "~{MEM6}") (pintype "output"))
+      (net 20 "~{MEM2}") (pintype "output"))
     (pad "9" thru_hole oval (at 7.62 12.7 90) (size 1.6 1.6) (drill 0.8) (layers "*.Cu" "*.Mask")
       (net 47 "~{CON INST}") (pintype "input"))
     (pad "10" thru_hole oval (at 7.62 10.16 90) (size 1.6 1.6) (drill 0.8) (layers "*.Cu" "*.Mask")
-      (net 41 "A09") (pintype "input"))
+      (net 37 "A13") (pintype "input"))
     (pad "11" thru_hole oval (at 7.62 7.62 90) (size 1.6 1.6) (drill 0.8) (layers "*.Cu" "*.Mask")
-      (net 15 "~{MEM7}") (pintype "output"))
+      (net 19 "~{MEM3}") (pintype "output"))
     (pad "12" thru_hole oval (at 7.62 5.08 90) (size 1.6 1.6) (drill 0.8) (layers "*.Cu" "*.Mask")
       (net 47 "~{CON INST}") (pintype "input"))
     (pad "13" thru_hole oval (at 7.62 2.54 90) (size 1.6 1.6) (drill 0.8) (layers "*.Cu" "*.Mask")
-      (net 42 "A08") (pintype "input"))
+      (net 38 "A12") (pintype "input"))
     (pad "14" thru_hole oval (at 7.62 0 90) (size 1.6 1.6) (drill 0.8) (layers "*.Cu" "*.Mask")
       (net 34 "+5V") (pinfunction "VCC") (pintype "power_in"))
@@
   )
   (footprint "Package_DIP:DIP-14_W7.62mm" (layer "F.Cu")
-    (at 48.768 46.99 90)
+    (at 70.485 46.99 90)
     (descr "14-lead though-hole mounted DIP package, row spacing 7.62 mm (300 mils)")
     (tags "THT DIP DIL PDIP 2.54mm 7.62mm 300mil")
     (property "Sheetfile" "Piggyback MEM0-7.kicad_sch")
     (property "Sheetname" "")
-    (property "ki_description" "Quad And2")
-    (property "ki_keywords" "TTL and2")
-    (attr through_hole)
-    (fp_text reference "U2" (at 3.81 -2.33 90) (layer "F.SilkS") hide
-        (effects (font (size 1 1) (thickness 0.15)))
-    )
-    (fp_text value "74LS08" (at 3.81 17.57 90) (layer "F.Fab")
+    (property "ki_description" "Quad 2-input OR")
+    (property "ki_keywords" "TTL Or2")
+    (attr through_hole)
+    (fp_text reference "U2" (at 3.81 -2.33 90) (layer "F.SilkS")
+        (effects (font (size 1 1) (thickness 0.15)))
+    )
+    (fp_text value "74LS32" (at 3.81 17.57 90) (layer "F.Fab")
         (effects (font (size 1 1) (thickness 0.15)))
     )
@@
       (net 47 "~{CON INST}") (pintype "input"))
     (pad "2" thru_hole oval (at 0 2.54 90) (size 1.6 1.6) (drill 0.8) (layers "*.Cu" "*.Mask")
-      (net 35 "A15") (pintype "input"))
+      (net 39 "A11") (pintype "input"))
     (pad "3" thru_hole oval (at 0 5.08 90) (size 1.6 1.6) (drill 0.8) (layers "*.Cu" "*.Mask")
-      (net 22 "~{MEM0}") (pintype "output"))
+      (net 18 "~{MEM4}") (pintype "output"))
     (pad "4" thru_hole oval (at 0 7.62 90) (size 1.6 1.6) (drill 0.8) (layers "*.Cu" "*.Mask")
       (net 47 "~{CON INST}") (pintype "input"))
     (pad "5" thru_hole oval (at 0 10.16 90) (size 1.6 1.6) (drill 0.8) (layers "*.Cu" "*.Mask")
-      (net 36 "A14") (pintype "input"))
+      (net 40 "A10") (pintype "input"))
     (pad "6" thru_hole oval (at 0 12.7 90) (size 1.6 1.6) (drill 0.8) (layers "*.Cu" "*.Mask")
-      (net 21 "~{MEM1}") (pintype "output"))
+      (net 17 "~{MEM5}") (pintype "output"))
     (pad "7" thru_hole oval (at 0 15.24 90) (size 1.6 1.6) (drill 0.8) (layers "*.Cu" "*.Mask")
       (net 1 "GND") (pinfunction "GND") (pintype "power_in"))
     (pad "8" thru_hole oval (at 7.62 15.24 90) (size 1.6 1.6) (drill 0.8) (layers "*.Cu" "*.Mask")
-      (net 20 "~{MEM2}") (pintype "output"))
+      (net 16 "~{MEM6}") (pintype "output"))
     (pad "9" thru_hole oval (at 7.62 12.7 90) (size 1.6 1.6) (drill 0.8) (layers "*.Cu" "*.Mask")
       (net 47 "~{CON INST}") (pintype "input"))
     (pad "10" thru_hole oval (at 7.62 10.16 90) (size 1.6 1.6) (drill 0.8) (layers "*.Cu" "*.Mask")
-      (net 37 "A13") (pintype "input"))
+      (net 41 "A09") (pintype "input"))
     (pad "11" thru_hole oval (at 7.62 7.62 90) (size 1.6 1.6) (drill 0.8) (layers "*.Cu" "*.Mask")
-      (net 19 "~{MEM3}") (pintype "output"))
+      (net 15 "~{MEM7}") (pintype "output"))
     (pad "12" thru_hole oval (at 7.62 5.08 90) (size 1.6 1.6) (drill 0.8) (layers "*.Cu" "*.Mask")
       (net 47 "~{CON INST}") (pintype "input"))
     (pad "13" thru_hole oval (at 7.62 2.54 90) (size 1.6 1.6) (drill 0.8) (layers "*.Cu" "*.Mask")
-      (net 38 "A12") (pintype "input"))
+      (net 42 "A08") (pintype "input"))
     (pad "14" thru_hole oval (at 7.62 0 90) (size 1.6 1.6) (drill 0.8) (layers "*.Cu" "*.Mask")
       (net 34 "+5V") (pinfunction "VCC") (pintype "power_in"))
