File: DG Nova CPU Tester/Piggyback MEM0-7/Piggyback MEM0-7.kicad_sch (KiCad schematic)
At the start: 4 parts, among them J1 Conn_02x18_Odd_Even, J3 Conn_01x17, U2 74LS08, U3 74LS08

Commit message: yeah
Parts:
- added C1, C2: CAP_Disc_Common_-_Entrex_Trapezoid, Forgotten Machines:Disc Capacitor Common Entrex Trapezoid, symbol ForgottenMachines:CAP_Disc_Common_-_Entrex_Trapezoid
Connections:
- net +5V: now also C1.1, C2.1
- net GND: now also C1.2, C2.2
Changed lines of the file:
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@@
+    )
+  )
+  (global_label "GND" (shape input) (at 46.99 142.875 270) (fields_autoplaced)
+    (effects (font (size 1.27 1.27)) (justify right))
+    (property "Intersheetrefs" "${INTERSHEET_REFS}" (at 46.99 149.6513 90)
+      (effects (font (size 1.27 1.27)) (justify right) hide)
     )
   )
@@
     (effects (font (size 1.27 1.27)) (justify left))
     (property "Intersheetrefs" "${INTERSHEET_REFS}" (at 54.3821 94.615 0)
+      (effects (font (size 1.27 1.27)) (justify left) hide)
+    )
+  )
+  (global_label "+5V" (shape input) (at 24.13 130.81 90) (fields_autoplaced)
+    (effects (font (size 1.27 1.27)) (justify left))
+    (property "Intersheetrefs" "${INTERSHEET_REFS}" (at 24.13 124.0337 90)
       (effects (font (size 1.27 1.27)) (justify left) hide)
     )
@@
     )
   )
+  (global_label "GND" (shape input) (at 24.13 143.51 270) (fields_autoplaced)
+    (effects (font (size 1.27 1.27)) (justify right))
+    (property "Intersheetrefs" "${INTERSHEET_REFS}" (at 24.13 150.2863 90)
+      (effects (font (size 1.27 1.27)) (justify right) hide)
+    )
+  )
   (global_label "GND" (shape input) (at 22.86 188.595 270) (fields_autoplaced)
     (effects (font (size 1.27 1.27)) (justify right))
@@
     (effects (font (size 1.27 1.27)) (justify left))
     (property "Intersheetrefs" "${INTERSHEET_REFS}" (at 116.0979 54.61 0)
+      (effects (font (size 1.27 1.27)) (justify left) hide)
+    )
+  )
+  (global_label "+5V" (shape input) (at 46.99 130.175 90) (fields_autoplaced)
+    (effects (font (size 1.27 1.27)) (justify left))
+    (property "Intersheetrefs" "${INTERSHEET_REFS}" (at 46.99 123.3987 90)
       (effects (font (size 1.27 1.27)) (justify left) hide)
     )
@@
     )
   )
+  (symbol (lib_id "ForgottenMachines:CAP_Disc_Common_-_Entrex_Trapezoid") (at 24.13 137.16 0) (unit 1)
+    (in_bom yes) (on_board yes) (dnp no) (fields_autoplaced)
+    (property "Reference" "C1" (at 29.21 137.16 0)
+      (effects (font (size 1.27 1.27)) (justify left))
+    )
+    (property "Value" "CAP_Disc_Common_-_Entrex_Trapezoid" (at 27.94 134.62 0)
+      (effects (font (size 1.27 1.27)) (justify left) hide)
+    )
+    (property "Footprint" "Forgotten Machines:Disc Capacitor Common Entrex Trapezoid" (at -11.43 147.32 0)
+      (effects (font (size 1.27 1.27)) hide)
+    )
+    (property "Datasheet" "~" (at 24.13 137.16 0)
+      (effects (font (size 1.27 1.27)) hide)
+    )
+    (pin "2")
+    (pin "1")
+    (instances
+      (project "Piggyback MEM0-7"
+        (path "/fe0be92e-1d85-43cc-bb82-88d36766eebc"
+          (reference "C1") (unit 1)
+        )
+      )
+    )
+  )
   (symbol (lib_id "74xx:74LS08") (at 99.06 136.525 0) (unit 2)
     (in_bom yes) (on_board yes) (dnp no) (fields_autoplaced)
@@
         )
       )
+    )
+  )
+  (symbol (lib_id "ForgottenMachines:CAP_Disc_Common_-_Entrex_Trapezoid") (at 46.99 136.525 0) (unit 1)
+    (in_bom yes) (on_board yes) (dnp no) (fields_autoplaced)
+    (property "Reference" "C2" (at 52.07 136.525 0)
+      (effects (font (size 1.27 1.27)) (justify left))
+    )
+    (property "Value" "CAP_Disc_Common_-_Entrex_Trapezoid" (at 50.8 133.985 0)
+      (effects (font (size 1.27 1.27)) (justify left) hide)
+    )
+    (property "Footprint" "Forgotten Machines:Disc Capacitor Common Entrex Trapezoid" (at 11.43 146.685 0)
+      (effects (font (size 1.27 1.27)) hide)
+    )
+    (property "Datasheet" "~" (at 46.99 136.525 0)
+      (effects (font (size 1.27 1.27)) hide)
+    )
+    (pin "2")
+    (pin "1")
+    (instances
+      (project "Piggyback MEM0-7"
+        (path "/fe0be92e-1d85-43cc-bb82-88d36766eebc"
+          (reference "C2") (unit 1)
+        )
+      )

Commit message: 74LS32
Parts:
- removed U2, U3: 74LS08, Package_DIP:DIP-14_W7.62mm, symbol 74xx:74LS08
- added U1, U2: 74LS32, Package_DIP:DIP-14_W7.62mm, symbol 74xx:74LS32
Connections:
- net +5V: now also U1.14 (VCC), U2.14 (VCC)
- net A08: now also U2.13
- net A09: now also U2.10
- net A10: now also U2.5
- net A11: now also U2.2
- net A12: now also U1.13
- net A13: now also U1.10
- net A14: now also U1.5
- net A15: now also U1.2
- net GND: now also U1.7 (GND), U2.7 (GND)
- net ~{CON INST}: now also U1.1, U1.12, U1.4, U1.9, U2.1, U2.12, U2.4, U2.9
- net ~{MEM0}: now also U1.3
- net ~{MEM1}: now also U1.6
- net ~{MEM2}: now also U1.8
- net ~{MEM3}: now also U1.11
- net ~{MEM4}: now also U2.3
- net ~{MEM5}: now also U2.6
- net ~{MEM6}: now also U2.8
- net ~{MEM7}: now also U2.11
