File: DG Nova CPU Tester/Piggyback MEM0-7/Piggyback MEM0-7 + Addr.kicad_sch (KiCad schematic)
At the start: 7 parts, among them J1 Conn_02x18_Odd_Even, J3 Conn_01x17, U1 74LS03, U2 74LS03, U3 74LS04

Commit message: Advance the test
Parts:
- added C3, C4, C5: CAP_Disc_Common_-_Entrex_Trapezoid, Forgotten Machines:Disc Capacitor Common Entrex Trapezoid, symbol ForgottenMachines:CAP_Disc_Common_-_Entrex_Trapezoid
- added U4, U9: 74HC595, symbol 74xx:74HC595
- added U5, U6, U7, U8: 74LS03, symbol 74xx:74LS03
Connections:
- net +5V: now also U2.14 (VCC), C3.1, C4.1, C5.1, U4.16 (VCC), U9.16 (VCC)
- net A08: now also U2.13
- net A09: now also U2.10
- net A10: now also U2.5
- net A11: now also U2.2
- net A12: now also U1.13
- net A13: now also U1.10
- net CON DATA: now also U5.1, U5.12, U5.4, U5.9, U6.1, U6.12, U6.4, U6.9, U7.1, U7.12, U7.4, U7.9, U8.1, U8.12, U8.4, U8.9
- net CON INST: now also U1.12, U1.9, U2.1, U2.12, U2.4, U2.9
- net GND: now also U2.7 (GND), C3.2, C4.2, C5.2, U4.8 (GND), U9.8 (GND)
- net ~{MEM0}: now also U6.3
- net ~{MEM10}: now also U8.8
- net ~{MEM11}: now also U8.11
- net ~{MEM12}: now also U7.3
- net ~{MEM13}: now also U7.6
- net ~{MEM14}: now also U7.8
- net ~{MEM15}: now also U7.11
- net ~{MEM1}: now also U6.6
- net ~{MEM2}: now also U1.8, U6.8
- net ~{MEM3}: now also U1.11, U6.11
- net ~{MEM4}: now also U2.3, U5.3
- net ~{MEM5}: now also U2.6, U5.6
- net ~{MEM6}: now also U2.8, U5.8
- net ~{MEM7}: now also U2.11, U5.11
- net ~{MEM8}: now also U8.3
- net ~{MEM9}: now also U8.6
- new net Addr00: U4.15 (QA), U6.2
- new net Addr01: U4.1 (QB), U6.5
- new net Addr02: U4.2 (QC), U6.10
- new net Addr03: U4.3 (QD), U6.13
- new net Addr04: U4.4 (QE), U5.2
- new net Addr05: U4.5 (QF), U5.5
- new net Addr06: U4.6 (QG), U5.10
- new net Addr07: U4.7 (QH), U5.13
- new net Addr08: U8.2, U9.15 (QA)
- new net Addr09: U8.5, U9.1 (QB)
- new net Addr10: U8.10, U9.2 (QC)
- new net Addr11: U8.13, U9.3 (QD)
- new net Addr12: U7.2, U9.4 (QE)
- new net Addr13: U7.5, U9.5 (QF)
- new net Addr14: U7.10, U9.6 (QG)
- new net Addr15: U7.13, U9.7 (QH)
Other:
- note added: "Use this to increase output ports: https://www.instructables.com/Extend-the-Ports-of-Arduino-Using-IC-74HC595N/ https://content.instructables.com/FSH/JDT7/IVO3HSBC/FSHJDT7IVO3HSBC.txt"
- moved on the sheet: J3, U1A, U1B, U1C, U1D, U2A, U2B, U2C, U2D, U2E, U3A, U3B

Commit message: more mem
Parts:
- added C6, C7, C8, C9: CAP_Disc_Common_-_Entrex_Trapezoid, Forgotten Machines:Disc Capacitor Common Entrex Trapezoid, symbol ForgottenMachines:CAP_Disc_Common_-_Entrex_Trapezoid
- added J22: Arduino Digital Pins, Connector_PinHeader_2.54mm:PinHeader_1x05_P2.54mm_Vertical, symbol Connector_Generic:Conn_01x05
- added J23: Arduino Digital Pins, Connector_PinHeader_2.54mm:PinHeader_1x06_P2.54mm_Vertical, symbol Connector_Generic:Conn_01x06
- added SW1: Arduino Mega Reset, Button_Switch_THT:SW_PUSH_6mm, symbol Switch:SW_Push
- added SW4: SW_DIP_x04, Package_DIP:DIP-8_W7.62mm, symbol Switch:SW_DIP_x04
- added unit 5 of U1
- added unit 5 of U5
- added unit 5 of U7
- added unit 5 of U8
- U2, U3, U5, U6, U7, U8: footprint (none) -> Package_DIP:DIP-14_W7.62mm
- U4, U9: footprint (none) -> Package_DIP:DIP-16_W7.62mm
- U6: renamed from U1; footprint (none) -> Package_DIP:DIP-14_W7.62mm
Connections:
- net +5V: now also U4.10 (~{SRCLR}), U9.10 (~{SRCLR}), C6.1, C7.1, C8.1, C9.1, U1.14 (VCC), U5.14 (VCC), U7.14 (VCC), U8.14 (VCC)
- net GND: now also C6.2, C7.2, C8.2, C9.2, SW1.1, SW4.5, SW4.6, SW4.7, SW4.8, U1.7 (GND), U5.7 (GND), U7.7 (GND), U8.7 (GND)
- net ClockPin2: now reaches U9.11 (SRCLK)
- net ClockPin2: now also J23.4 (Pin_4)
- net LatchPin2: now reaches U9.12 (RCLK)
- net LatchPin2: now also J23.5 (Pin_5)
- net DataPin2: now reaches U9.14 (SER)
- net DataPin2: now also J22.4 (Pin_4)
- net ClockPin1: now reaches U4.11 (SRCLK)
- net ClockPin1: now also J22.2 (Pin_2)
- net LatchPin1: now reaches U4.12 (RCLK)
- net LatchPin1: now also J22.3 (Pin_3)
- net DataPin1: now reaches U4.14 (SER)
- net DataPin1: now also J22.1 (Pin_1)
- new net +5V OK: J23.6 (Pin_6)
- new net DIP1: J23.3 (Pin_3), SW4.4
- new net DIP2: J23.2 (Pin_2), SW4.3
- new net DIP3: J23.1 (Pin_1), SW4.2
- new net DIP4: J22.5 (Pin_5), SW4.1
- new net RST1: SW1.2
Other:
- note added: "ClockPin"
- note added: "DataPin"
- note added: "Invert all arduino signals and swap these OR gates for NAND gates"
- note added: "LatchPin"
- note removed: "Invert all arduino signals and swap these or gates for NAND gates"
- moved on the sheet: C1, C2, C3, C4, C5, U2E, U3G, U6E

Commit message: more
Parts:
- C1, C2, C3, C4, C5, C6, C7, C8, C9: footprint Forgotten Machines:Disc Capacitor Common Entrex Trapezoid -> Forgotten Machines:Disc Capacitor Entrex Trapezoid .10

Commit message: Done?
Parts:
- added J5, J6: Conn_01x08, Connector_PinHeader_2.54mm:PinHeader_1x08_P2.54mm_Vertical, symbol Connector_Generic:Conn_01x08
Connections:
- net ClockPin1: now also J6.5 (Pin_5)
- net DIP4: now also J6.8 (Pin_8)
- net DataPin1: now also J6.4 (Pin_4)
- net DataPin2: now also J6.7 (Pin_7)
- net LatchPin1: now also J6.6 (Pin_6)
- net ~{CON DATA}: now also J6.1 (Pin_1)
- new net ~{CONT+ISTP+MSTP}: J6.2 (Pin_2)
- new net ~{MBO1}: J5.7 (Pin_7)
- new net ~{MBO2}: J5.6 (Pin_6)
- new net ~{MBO3}: J5.5 (Pin_5)
- new net ~{MBO4}: J5.4 (Pin_4)
- new net ~{MBO5}: J5.3 (Pin_3)
- new net ~{MBO6}: J5.2 (Pin_2)
- new net ~{MBO7}: J5.1 (Pin_1)
- new net ~{MSTP}: J6.3 (Pin_3)
- new net ~{STOP}: J5.8 (Pin_8)
Changed lines of the file:
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@@
+    (stroke (width 0) (type default))
+  )
+  (wire (pts (xy 148.59 295.91) (xy 166.37 295.91))
     (stroke (width 0) (type default))
   )
@@
     (effects (font (size 1.27 1.27)) (justify left bottom))
   )
+  (label "DIP4" (at 148.59 295.91 0) (fields_autoplaced)
+    (effects (font (size 1.27 1.27)) (justify left bottom))
+  )
   (label "D3" (at 52.07 112.395 0) (fields_autoplaced)
     (effects (font (size 1.27 1.27)) (justify left bottom))
@@
     (property "Intersheetrefs" "${INTERSHEET_REFS}" (at 246.946 283.21 0)
       (effects (font (size 1.27 1.27)) (justify left) hide)
+    )
+  )
+  (global_label "~{CON DATA}" (shape input) (at 166.37 278.13 180) (fields_autoplaced)
+    (effects (font (size 0.9906 0.9906)) (justify right))
+    (property "Intersheetrefs" "${INTERSHEET_REFS}" (at 157.5097 278.13 0)
+      (effects (font (size 1.27 1.27)) (justify right) hide)
     )
   )
@@
     )
   )
+  (global_label "~{MBO2}" (shape input) (at 166.37 266.065 180) (fields_autoplaced)
+    (effects (font (size 1.27 1.27)) (justify right))
+    (property "Intersheetrefs" "${INTERSHEET_REFS}" (at 158.857 266.065 0)
+      (effects (font (size 1.27 1.27)) (justify right) hide)
+    )
+  )
   (global_label "~{MEM2}" (shape input) (at 35.56 76.835 180) (fields_autoplaced)
     (effects (font (size 1.27 1.27)) (justify right))
@@
     )
   )
+  (global_label "~{MBO7}" (shape input) (at 166.37 253.365 180) (fields_autoplaced)
+    (effects (font (size 1.27 1.27)) (justify right))
+    (property "Intersheetrefs" "${INTERSHEET_REFS}" (at 158.857 253.365 0)
+      (effects (font (size 1.27 1.27)) (justify right) hide)
+    )
+  )
   (global_label "LatchPin1" (shape input) (at 27.94 117.475 180) (fields_autoplaced)
     (effects (font (size 1.27 1.27)) (justify right))
@@
     )
   )
+  (global_label "~{MSTP}" (shape input) (at 166.37 283.21 180) (fields_autoplaced)
+    (effects (font (size 0.9906 0.9906)) (justify right))
+    (property "Intersheetrefs" "${INTERSHEET_REFS}" (at 160.221 283.21 0)
+      (effects (font (size 1.27 1.27)) (justify right) hide)
+    )
+  )
   (global_label "~{MEM0}" (shape input) (at 240.03 48.895 0) (fields_autoplaced)
     (effects (font (size 1.27 1.27)) (justify left))
@@
     )
   )
+  (global_label "~{CONT+ISTP+MSTP}" (shape input) (at 166.37 280.67 180) (fields_autoplaced)
+    (effects (font (size 0.9906 0.9906)) (justify right))
+    (property "Intersheetrefs" "${INTERSHEET_REFS}" (at 151.3587 280.67 0)
+      (effects (font (size 1.27 1.27)) (justify right) hide)
+    )
+  )
   (global_label "~{RST}" (shape input) (at 49.53 28.575 270) (fields_autoplaced)
     (effects (font (size 0.9906 0.9906)) (justify right))
@@
     (effects (font (size 1.27 1.27)) (justify right))
     (property "Intersheetrefs" "${INTERSHEET_REFS}" (at 26.1834 66.675 0)
+      (effects (font (size 1.27 1.27)) (justify right) hide)
+    )
+  )
+  (global_label "LatchPin1" (shape input) (at 166.37 290.83 180) (fields_autoplaced)
+    (effects (font (size 1.27 1.27)) (justify right))
+    (property "Intersheetrefs" "${INTERSHEET_REFS}" (at 154.0111 290.83 0)
       (effects (font (size 1.27 1.27)) (justify right) hide)
     )
@@
     )
   )
+  (global_label "ClockPin1" (shape input) (at 166.37 288.29 180) (fields_autoplaced)
+    (effects (font (size 1.27 1.27)) (justify right))
+    (property "Intersheetrefs" "${INTERSHEET_REFS}" (at 153.9506 288.29 0)
+      (effects (font (size 1.27 1.27)) (justify right) hide)
+    )
+  )
   (global_label "GND" (shape input) (at 146.685 222.885 270) (fields_autoplaced)
     (effects (font (size 1.27 1.27)) (justify right))
@@
     )
   )
+  (global_label "~{MBO1}" (shape input) (at 166.37 268.605 180) (fields_autoplaced)
+    (effects (font (size 1.27 1.27)) (justify right))
+    (property "Intersheetrefs" "${INTERSHEET_REFS}" (at 158.857 268.605 0)
+      (effects (font (size 1.27 1.27)) (justify right) hide)
+    )
+  )
   (global_label "Addr12" (shape input) (at 127.635 107.315 0) (fields_autoplaced)
     (effects (font (size 1.27 1.27)) (justify left))
@@
     )
   )
+  (global_label "~{MBO4}" (shape input) (at 166.37 260.985 180) (fields_autoplaced)
+    (effects (font (size 1.27 1.27)) (justify right))
+    (property "Intersheetrefs" "${INTERSHEET_REFS}" (at 158.857 260.985 0)
+      (effects (font (size 1.27 1.27)) (justify right) hide)
+    )
+  )
   (global_label "~{ISTP}" (shape input) (at 59.69 28.575 270) (fields_autoplaced)
     (effects (font (size 0.9906 0.9906)) (justify right))
@@
     )
   )
+  (global_label "DataPin2" (shape input) (at 166.37 293.37 180) (fields_autoplaced)
+    (effects (font (size 1.27 1.27)) (justify right))
+    (property "Intersheetrefs" "${INTERSHEET_REFS}" (at 154.8578 293.37 0)
+      (effects (font (size 1.27 1.27)) (justify right) hide)
+    )
+  )
   (global_label "~{MEM2}" (shape input) (at 239.395 83.82 0) (fields_autoplaced)
     (effects (font (size 1.27 1.27)) (justify left))
@@
     )
   )
+  (global_label "~{STOP}" (shape input) (at 166.37 271.145 180) (fields_autoplaced)
+    (effects (font (size 0.9906 0.9906)) (justify right))
+    (property "Intersheetrefs" "${INTERSHEET_REFS}" (at 160.8873 271.145 0)
+      (effects (font (size 1.27 1.27)) (justify right) hide)
+    )
+  )
   (global_label "A10" (shape input) (at 36.83 28.575 270) (fields_autoplaced)
     (effects (font (size 1.27 1.27)) (justify right))
@@
     )
   )
+  (global_label "DataPin1" (shape input) (at 166.37 285.75 180) (fields_autoplaced)
+    (effects (font (size 1.27 1.27)) (justify right))
+    (property "Intersheetrefs" "${INTERSHEET_REFS}" (at 154.8578 285.75 0)
+      (effects (font (size 1.27 1.27)) (justify right) hide)
+    )
+  )
   (global_label "ClockPin1" (shape input) (at 27.94 114.935 180) (fields_autoplaced)
     (effects (font (size 1.27 1.27)) (justify right))
@@
     )
   )
+  (global_label "~{MBO6}" (shape input) (at 166.37 255.905 180) (fields_autoplaced)
+    (effects (font (size 1.27 1.27)) (justify right))
+    (property "Intersheetrefs" "${INTERSHEET_REFS}" (at 158.857 255.905 0)
+      (effects (font (size 1.27 1.27)) (justify right) hide)
+    )
+  )
   (global_label "~{MBO15}" (shape input) (at 35.56 84.455 180) (fields_autoplaced)
     (effects (font (size 1.27 1.27)) (justify right))
@@
     )
   )
+  (global_label "~{MBO3}" (shape input) (at 166.37 263.525 180) (fields_autoplaced)
+    (effects (font (size 1.27 1.27)) (justify right))
+    (property "Intersheetrefs" "${INTERSHEET_REFS}" (at 158.857 263.525 0)
+      (effects (font (size 1.27 1.27)) (justify right) hide)
+    )
+  )
   (global_label "~{MEM6}" (shape input) (at 35.56 71.755 180) (fields_autoplaced)
     (effects (font (size 1.27 1.27)) (justify right))
@@
     (effects (font (size 1.27 1.27)) (justify right))
     (property "Intersheetrefs" "${INTERSHEET_REFS}" (at 26.8485 59.055 0)
+      (effects (font (size 1.27 1.27)) (justify right) hide)
+    )
+  )
+  (global_label "~{MBO5}" (shape input) (at 166.37 258.445 180) (fields_autoplaced)
+    (effects (font (size 1.27 1.27)) (justify right))
+    (property "Intersheetrefs" "${INTERSHEET_REFS}" (at 158.857 258.445 0)
       (effects (font (size 1.27 1.27)) (justify right) hide)
     )
@@
     )
     (property "Value" "Conn_02x18_Odd_Even" (at 41.91 49.0761 0)
-      (effects (font (size 1.27 1.27)))
+      (effects (font (size 1.27 1.27)) hide)
     )
     (property "Footprint" "Connector_PinHeader_2.54mm:PinHeader_2x18_P2.54mm_Vertical" (at 40.64 71.755 0)
@@
     )
   )
+  (symbol (lib_id "Connector_Generic:Conn_01x08") (at 171.45 285.75 0) (unit 1)
+    (in_bom yes) (on_board yes) (dnp no) (fields_autoplaced)
+    (property "Reference" "J6" (at 173.99 285.75 0)
+      (effects (font (size 1.27 1.27)) (justify left))
+    )
+    (property "Value" "Conn_01x08" (at 173.99 288.29 0)
+      (effects (font (size 1.27 1.27)) (justify left) hide)
+    )
+    (property "Footprint" "Connector_PinHeader_2.54mm:PinHeader_1x08_P2.54mm_Vertical" (at 171.45 285.75 0)
+      (effects (font (size 1.27 1.27)) hide)
+    )
+    (property "Datasheet" "~" (at 171.45 285.75 0)
+      (effects (font (size 1.27 1.27)) hide)
+    )
+    (pin "2")
+    (pin "1")
+    (pin "3")
+    (pin "8")
+    (pin "7")
+    (pin "6")
+    (pin "4")
+    (pin "5")
+    (instances
+      (project "Piggyback MEM0-7 + Addr"
+        (path "/fe0be92e-1d85-43cc-bb82-88d36766eebc"
+          (reference "J6") (unit 1)
+        )
+      )
+    )
+  )
   (symbol (lib_id "ForgottenMachines:CAP_Disc_Common_-_Entrex_Trapezoid") (at 30.48 172.085 0) (unit 1)
     (in_bom yes) (on_board yes) (dnp no) (fields_autoplaced)
@@
         (path "/fe0be92e-1d85-43cc-bb82-88d36766eebc"
           (reference "SW1") (unit 1)
+        )
+      )
+    )
+  )
+  (symbol (lib_id "Connector_Generic:Conn_01x08") (at 171.45 260.985 0) (unit 1)
+    (in_bom yes) (on_board yes) (dnp no) (fields_autoplaced)
+    (property "Reference" "J5" (at 173.99 262.255 0)
+      (effects (font (size 1.27 1.27)) (justify left))
+    )
+    (property "Value" "Conn_01x08" (at 173.99 263.525 0)
+      (effects (font (size 1.27 1.27)) (justify left) hide)
+    )
+    (property "Footprint" "Connector_PinHeader_2.54mm:PinHeader_1x08_P2.54mm_Vertical" (at 171.45 260.985 0)
+      (effects (font (size 1.27 1.27)) hide)
+    )
+    (property "Datasheet" "~" (at 171.45 260.985 0)
+      (effects (font (size 1.27 1.27)) hide)
+    )
+    (pin "2")
+    (pin "1")
+    (pin "3")
+    (pin "8")
+    (pin "7")
+    (pin "6")
+    (pin "4")
+    (pin "5")
+    (instances
+      (project "Piggyback MEM0-7 + Addr"
+        (path "/fe0be92e-1d85-43cc-bb82-88d36766eebc"
+          (reference "J5") (unit 1)
         )
       )
@@
     )
     (property "Value" "Conn_01x17" (at 44.45 21.1361 90)
-      (effects (font (size 1.27 1.27)))
+      (effects (font (size 1.27 1.27)) hide)
     )
     (property "Footprint" "Connector_PinHeader_2.54mm:PinHeader_1x17_P2.54mm_Vertical" (at 44.45 23.495 0)
