File: El Classico ONLY RAM/nova_modern.kicad_pcb (KiCad board)
At the start: 2 copper layers, 379 x 139.7 mm, 49 parts, among them J1 PORTA, J2 PORTB, SW1 SW_SPDT, U1 74LS14, U10 62256P, U11 62256P, U12 27C256, U13 7496, U14 7496, U15 7496, U16 7496, U17 74ALS00, U18 74LS241, U19 74LS241, U2 74LS14, U3 74LS14, U4 74LS14, U5 74LS14, U6 74LS148, U7 74LS148, U8 74LS148, U9 27C256

Commit message: update schematic to work with KiCad correctly
Parts:
- moved C20 0.80 mm to (49.5, 83.0)
Connections:
- J1 pad 10: (no net) -> unconnected-(J1-Pin_10-Pad10)
- J1 pad 11: (no net) -> unconnected-(J1-Pin_11-Pad11)
- J1 pad 12: (no net) -> unconnected-(J1-Pin_12-Pad12)
- J1 pad 13: (no net) -> unconnected-(J1-Pin_13-Pad13)
- J1 pad 14: (no net) -> unconnected-(J1-Pin_14-Pad14)
- J1 pad 15: (no net) -> unconnected-(J1-Pin_15-Pad15)
- J1 pad 25: (no net) -> unconnected-(J1-Pin_25-Pad25)
- J1 pad 34: (no net) -> unconnected-(J1-Pin_34-Pad34)
- J1 pad 35: (no net) -> unconnected-(J1-Pin_35-Pad35)
- J1 pad 36: (no net) -> unconnected-(J1-Pin_36-Pad36)
- J1 pad 37: (no net) -> unconnected-(J1-Pin_37-Pad37)
- J1 pad 38: (no net) -> unconnected-(J1-Pin_38-Pad38)
- J1 pad 39: (no net) -> unconnected-(J1-Pin_39-Pad39)
- J1 pad 40: (no net) -> unconnected-(J1-Pin_40-Pad40)
- J1 pad 41: (no net) -> unconnected-(J1-Pin_41-Pad41)
- J1 pad 42: (no net) -> unconnected-(J1-Pin_42-Pad42)
- J1 pad 43: (no net) -> unconnected-(J1-Pin_43-Pad43)
- J1 pad 44: (no net) -> unconnected-(J1-Pin_44-Pad44)
- J1 pad 45: (no net) -> unconnected-(J1-Pin_45-Pad45)
- J1 pad 46: (no net) -> unconnected-(J1-Pin_46-Pad46)
- J1 pad 47: (no net) -> unconnected-(J1-Pin_47-Pad47)
- J1 pad 48: (no net) -> unconnected-(J1-Pin_48-Pad48)
- J1 pad 49: (no net) -> unconnected-(J1-Pin_49-Pad49)
- J1 pad 5: (no net) -> unconnected-(J1-Pin_5-Pad5)
- J1 pad 50: (no net) -> unconnected-(J1-Pin_50-Pad50)
- J1 pad 51: (no net) -> unconnected-(J1-Pin_51-Pad51)
- J1 pad 52: (no net) -> unconnected-(J1-Pin_52-Pad52)
- J1 pad 53: (no net) -> unconnected-(J1-Pin_53-Pad53)
- J1 pad 54: (no net) -> unconnected-(J1-Pin_54-Pad54)
- J1 pad 55: (no net) -> unconnected-(J1-Pin_55-Pad55)
- J1 pad 56: (no net) -> unconnected-(J1-Pin_56-Pad56)
- J1 pad 57: (no net) -> unconnected-(J1-Pin_57-Pad57)
- J1 pad 58: (no net) -> unconnected-(J1-Pin_58-Pad58)
- J1 pad 59: (no net) -> unconnected-(J1-Pin_59-Pad59)
- J1 pad 6: (no net) -> unconnected-(J1-Pin_6-Pad6)
- J1 pad 60: (no net) -> unconnected-(J1-Pin_60-Pad60)
- J1 pad 61: (no net) -> unconnected-(J1-Pin_61-Pad61)
- J1 pad 62: (no net) -> unconnected-(J1-Pin_62-Pad62)
- J1 pad 63: (no net) -> unconnected-(J1-Pin_63-Pad63)
- J1 pad 64: (no net) -> unconnected-(J1-Pin_64-Pad64)
- J1 pad 65: (no net) -> unconnected-(J1-Pin_65-Pad65)
- J1 pad 66: (no net) -> unconnected-(J1-Pin_66-Pad66)
- J1 pad 67: (no net) -> unconnected-(J1-Pin_67-Pad67)
- J1 pad 68: (no net) -> unconnected-(J1-Pin_68-Pad68)
- J1 pad 69: (no net) -> unconnected-(J1-Pin_69-Pad69)
- J1 pad 7: (no net) -> unconnected-(J1-Pin_7-Pad7)
- J1 pad 70: (no net) -> unconnected-(J1-Pin_70-Pad70)
- J1 pad 71: (no net) -> unconnected-(J1-Pin_71-Pad71)
- J1 pad 72: (no net) -> unconnected-(J1-Pin_72-Pad72)
- J1 pad 73: (no net) -> unconnected-(J1-Pin_73-Pad73)
- J1 pad 74: (no net) -> unconnected-(J1-Pin_74-Pad74)
- J1 pad 75: (no net) -> unconnected-(J1-Pin_75-Pad75)
- J1 pad 76: (no net) -> unconnected-(J1-Pin_76-Pad76)
- J1 pad 77: (no net) -> unconnected-(J1-Pin_77-Pad77)
- J1 pad 78: (no net) -> unconnected-(J1-Pin_78-Pad78)
- J1 pad 79: (no net) -> unconnected-(J1-Pin_79-Pad79)
- J1 pad 8: (no net) -> unconnected-(J1-Pin_8-Pad8)
- J1 pad 80: (no net) -> unconnected-(J1-Pin_80-Pad80)
- J1 pad 81: (no net) -> unconnected-(J1-Pin_81-Pad81)
- J1 pad 82: (no net) -> unconnected-(J1-Pin_82-Pad82)
- J1 pad 83: (no net) -> unconnected-(J1-Pin_83-Pad83)
- J1 pad 84: (no net) -> unconnected-(J1-Pin_84-Pad84)
- J1 pad 85: (no net) -> unconnected-(J1-Pin_85-Pad85)
- J1 pad 86: (no net) -> unconnected-(J1-Pin_86-Pad86)
- J1 pad 87: (no net) -> unconnected-(J1-Pin_87-Pad87)
- J1 pad 88: (no net) -> unconnected-(J1-Pin_88-Pad88)
- J1 pad 89: (no net) -> unconnected-(J1-Pin_89-Pad89)
- J1 pad 9: (no net) -> unconnected-(J1-Pin_9-Pad9)
- J1 pad 90: (no net) -> unconnected-(J1-Pin_90-Pad90)
- J1 pad 91: (no net) -> unconnected-(J1-Pin_91-Pad91)
- J1 pad 92: (no net) -> unconnected-(J1-Pin_92-Pad92)
- J1 pad 93: (no net) -> unconnected-(J1-Pin_93-Pad93)
- J1 pad 94: (no net) -> unconnected-(J1-Pin_94-Pad94)
- J1 pad 95: (no net) -> unconnected-(J1-Pin_95-Pad95)
- J1 pad 96: (no net) -> unconnected-(J1-Pin_96-Pad96)
- J2 pad 11: (no net) -> unconnected-(J2-Pin_11-Pad11)
- J2 pad 13: (no net) -> unconnected-(J2-Pin_13-Pad13)
- J2 pad 15: (no net) -> unconnected-(J2-Pin_15-Pad15)
- J2 pad 17: (no net) -> unconnected-(J2-Pin_17-Pad17)
- J2 pad 19: (no net) -> unconnected-(J2-Pin_19-Pad19)
- J2 pad 21: (no net) -> unconnected-(J2-Pin_21-Pad21)
- J2 pad 23: (no net) -> unconnected-(J2-Pin_23-Pad23)
- J2 pad 25: (no net) -> unconnected-(J2-Pin_25-Pad25)
- J2 pad 27: (no net) -> unconnected-(J2-Pin_27-Pad27)
- J2 pad 29: (no net) -> unconnected-(J2-Pin_29-Pad29)
- J2 pad 31: (no net) -> unconnected-(J2-Pin_31-Pad31)
- J2 pad 33: (no net) -> unconnected-(J2-Pin_33-Pad33)
- J2 pad 34: (no net) -> unconnected-(J2-Pin_34-Pad34)
- J2 pad 35: (no net) -> unconnected-(J2-Pin_35-Pad35)
- J2 pad 36: (no net) -> unconnected-(J2-Pin_36-Pad36)
- J2 pad 37: (no net) -> unconnected-(J2-Pin_37-Pad37)
- J2 pad 38: (no net) -> unconnected-(J2-Pin_38-Pad38)
- J2 pad 39: (no net) -> unconnected-(J2-Pin_39-Pad39)
- J2 pad 40: (no net) -> unconnected-(J2-Pin_40-Pad40)
- J2 pad 41: (no net) -> unconnected-(J2-Pin_41-Pad41)
- J2 pad 42: (no net) -> unconnected-(J2-Pin_42-Pad42)
- J2 pad 43: (no net) -> unconnected-(J2-Pin_43-Pad43)
- J2 pad 44: (no net) -> unconnected-(J2-Pin_44-Pad44)
- J2 pad 45: (no net) -> unconnected-(J2-Pin_45-Pad45)
- J2 pad 46: (no net) -> unconnected-(J2-Pin_46-Pad46)
- J2 pad 47: (no net) -> unconnected-(J2-Pin_47-Pad47)
- J2 pad 48: (no net) -> unconnected-(J2-Pin_48-Pad48)
- J2 pad 49: (no net) -> unconnected-(J2-Pin_49-Pad49)
- J2 pad 5: (no net) -> unconnected-(J2-Pin_5-Pad5)
- J2 pad 50: (no net) -> unconnected-(J2-Pin_50-Pad50)
- J2 pad 51: (no net) -> unconnected-(J2-Pin_51-Pad51)
- J2 pad 52: (no net) -> unconnected-(J2-Pin_52-Pad52)
- J2 pad 53: (no net) -> unconnected-(J2-Pin_53-Pad53)
- J2 pad 54: (no net) -> unconnected-(J2-Pin_54-Pad54)
- J2 pad 55: (no net) -> unconnected-(J2-Pin_55-Pad55)
- J2 pad 56: (no net) -> unconnected-(J2-Pin_56-Pad56)
- J2 pad 57: (no net) -> unconnected-(J2-Pin_57-Pad57)
- J2 pad 58: (no net) -> unconnected-(J2-Pin_58-Pad58)
- J2 pad 59: (no net) -> unconnected-(J2-Pin_59-Pad59)
- J2 pad 6: (no net) -> unconnected-(J2-Pin_6-Pad6)
- J2 pad 60: (no net) -> unconnected-(J2-Pin_60-Pad60)
- J2 pad 61: (no net) -> unconnected-(J2-Pin_61-Pad61)
- J2 pad 62: (no net) -> unconnected-(J2-Pin_62-Pad62)
- J2 pad 63: (no net) -> unconnected-(J2-Pin_63-Pad63)
- J2 pad 64: (no net) -> unconnected-(J2-Pin_64-Pad64)
- J2 pad 65: (no net) -> unconnected-(J2-Pin_65-Pad65)
- J2 pad 66: (no net) -> unconnected-(J2-Pin_66-Pad66)
- J2 pad 67: (no net) -> unconnected-(J2-Pin_67-Pad67)
- J2 pad 69: (no net) -> unconnected-(J2-Pin_69-Pad69)
- J2 pad 7: (no net) -> unconnected-(J2-Pin_7-Pad7)
- J2 pad 70: (no net) -> unconnected-(J2-Pin_70-Pad70)
- J2 pad 71: (no net) -> unconnected-(J2-Pin_71-Pad71)
- J2 pad 73: (no net) -> unconnected-(J2-Pin_73-Pad73)
- J2 pad 75: (no net) -> unconnected-(J2-Pin_75-Pad75)
- J2 pad 77: (no net) -> unconnected-(J2-Pin_77-Pad77)
- J2 pad 8: (no net) -> unconnected-(J2-Pin_8-Pad8)
- J2 pad 80: (no net) -> unconnected-(J2-Pin_80-Pad80)
- J2 pad 81: (no net) -> unconnected-(J2-Pin_81-Pad81)
- J2 pad 82: (no net) -> unconnected-(J2-Pin_82-Pad82)
- J2 pad 83: (no net) -> unconnected-(J2-Pin_83-Pad83)
- J2 pad 84: (no net) -> unconnected-(J2-Pin_84-Pad84)
- J2 pad 9: (no net) -> unconnected-(J2-Pin_9-Pad9)
- J2 pad 91: (no net) -> unconnected-(J2-Pin_91-Pad91)
- J2 pad 92: (no net) -> unconnected-(J2-Pin_92-Pad92)
- J2 pad 94: (no net) -> unconnected-(J2-Pin_94-Pad94)
- J2 pad 95: (no net) -> unconnected-(J2-Pin_95-Pad95)
- U13 pad 10: (no net) -> unconnected-(U13-Q4-Pad10)
- U14 pad 10: (no net) -> unconnected-(U14-Q4-Pad10)
- U15 pad 10: (no net) -> unconnected-(U15-Q4-Pad10)
- U16 pad 10: (no net) -> unconnected-(U16-Q4-Pad10)
- U6 pad 14: (no net) -> unconnected-(U6-GS-Pad14)
- U6 pad 15: (no net) -> unconnected-(U6-EO-Pad15)
- U7 pad 14: (no net) -> unconnected-(U7-GS-Pad14)
- U7 pad 15: (no net) -> unconnected-(U7-EO-Pad15)
- U8 pad 14: (no net) -> unconnected-(U8-GS-Pad14)
- U8 pad 15: (no net) -> unconnected-(U8-EO-Pad15)
Other:
- net class Default removed
- net class Power removed
