File: El Classico ONLY RAM/nova_modern.kicad_sch (KiCad schematic)
At the start: 45 parts, among them J1 PORTA, J2 PORTB, SW1 SW_SPDT, U1 74LS14, U10 62256P, U11 62256P, U12 27C256, U13 7496, U14 7496, U15 7496, U16 7496, U17 74ALS00, U18 74LS241, U19 74LS241, U2 74LS14, U3 74LS14, U4 74LS14, U5 74LS14, U6 74LS148, U7 74LS148, U8 74LS148, U9 27C256

Commit message: update schematic to work with KiCad correctly
Parts:
- removed C20: 10uF/25V, Capacitor_THT:CP_Radial_D8.0mm_P3.50mm, symbol Device:CP1
- added C20: 10uF/25V, Capacitor_THT:CP_Radial_D8.0mm_P3.50mm, symbol Device:C_Polarized_US
Connections:
- net GND: now also U13.12 (GND), U13.7 (P4), U14.12 (GND), U14.7 (P4), U15.12 (GND), U15.7 (P4), U16.12 (GND), U16.7 (P4), C20.2
- net IO00: now also U13.2 (P0)
- net IO01: now also U13.3 (P1)
- net IO02: now also U13.4 (P2)
- net IO03: now also U13.6 (P3)
- net IO04: now also U14.2 (P0)
- net IO05: now also U14.3 (P1)
- net IO06: now also U14.4 (P2)
- net IO07: now also U14.6 (P3)
- net IO08: now also U15.2 (P0)
- net IO09: now also U15.3 (P1)
- net IO10: now also U15.4 (P2)
- net IO11: now also U15.6 (P3)
- net IO12: now also U16.2 (P0)
- net IO13: now also U16.3 (P1)
- net IO14: now also U16.4 (P2)
- net IO15: now also U16.6 (P3)
- net SUM0: now also U13.9 (Ser); no longer J2.74 (Pin_74), J2.76 (Pin_76), J2.79 (Pin_79), U13.1 (CK), U13.8 (PE), U14.1 (CK), U14.8 (PE), U15.1 (CK), U15.8 (PE), U16.1 (CK), U16.8 (PE), U5.4 (2Y)
- net VCC: now also U13.5 (VCC), U14.5 (VCC), U15.5 (VCC), U16.5 (VCC), C20.1
- net WD00: now also U13.15 (Q0)
- net WD01: now also U13.14 (Q1)
- net WD02: now also U13.13 (Q2)
- net WD03: now also U13.11 (Q3)
- net WD04: now also U14.15 (Q0)
- net WD05: now also U14.14 (Q1)
- net WD06: now also U14.13 (Q2)
- net WD07: now also U14.11 (Q3)
- net WD08: now also U15.15 (Q0)
- net WD09: now also U15.14 (Q1)
- net WD10: now also U15.13 (Q2)
- net WD11: now also U15.11 (Q3)
- net WD12: now also U16.15 (Q0)
- net WD13: now also U16.14 (Q1)
- net WD14: now also U16.13 (Q2)
- net WD15: now also U16.11 (Q3)
- net at U16.16 (~{R}): now also U13.16 (~{R}), U14.16 (~{R}), U15.16 (~{R}), U5.6 (3Y)
- net SUM3: now reaches U16.9 (Ser)
- net SUM3: now also J2.76 (Pin_76)
- net SUM2: now reaches U15.9 (Ser)
- net SUM2: now also J2.74 (Pin_74)
- net SUM1: now reaches U14.9 (Ser)
- net SUM1: now also J2.79 (Pin_79)
- net at U5.10 (5Y): now also U13.8 (PE), U14.8 (PE), U15.8 (PE), U16.8 (PE)
- new net: U13.1 (CK), U14.1 (CK), U15.1 (CK), U16.1 (CK), U5.4 (2Y)
- no-connect marks 10 -> 151
Other:
- moved on the sheet: U14, U15, U16
