File: El Classico ONLY RAM/nova_modern.kicad_sch (KiCad schematic)
At the start: 45 parts, among them J1 PORTA, J2 PORTB, SW1 SW_SPDT, U1 74LS14, U10 62256P, U11 62256P, U12 27C256, U13 7496, U14 7496, U15 7496, U16 7496, U17 74ALS00, U18 74LS241, U19 74LS241, U2 74LS14, U3 74LS14, U4 74LS14, U5 74LS14, U6 74LS148, U7 74LS148, U8 74LS148, U9 27C256

Commit message: bridge dchp/intp in/out
Connections:
- net dchp: now reaches J1.93 (Pin_93)
- net dchp: now also J1.94 (Pin_94)
- net intp: now reaches J1.95 (Pin_95)
- net intp: now also J1.96 (Pin_96)
- no-connect marks 151 -> 147
Changed lines of the file:
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@@
 	)
 	(no_connect
-		(at 43.18 215.9)
-	)
-	(no_connect
 		(at 43.18 104.14)
 	)
@@
 	)
 	(no_connect
-		(at 43.18 213.36)
-	)
-	(no_connect
 		(at 55.88 157.48)
 	)
 	(no_connect
-		(at 55.88 215.9)
-	)
-	(no_connect
 		(at 55.88 365.76)
 	)
@@
 	)
 	(no_connect
-		(at 55.88 213.36)
-	)
-	(no_connect
 		(at 55.88 297.18)
 	)
@@
 	(wire
 		(pts
+			(xy 41.91 223.52) (xy 58.42 223.52)
+		)
+		(stroke
+			(width 0)
+			(type default)
+		)
+	)
+	(wire
+		(pts
 			(xy 218.44 223.52) (xy 218.44 289.56)
 		)
@@
 	(wire
 		(pts
+			(xy 55.88 213.36) (xy 59.69 213.36)
+		)
+		(stroke
+			(width 0)
+			(type default)
+		)
+	)
+	(wire
+		(pts
 			(xy 354.33 356.87) (xy 396.24 356.87)
 		)
@@
 	(wire
 		(pts
+			(xy 58.42 223.52) (xy 58.42 215.9)
+		)
+		(stroke
+			(width 0)
+			(type default)
+		)
+	)
+	(wire
+		(pts
 			(xy 55.88 368.3) (xy 66.04 368.3)
 		)
@@
 	(wire
 		(pts
+			(xy 59.69 226.06) (xy 40.64 226.06)
+		)
+		(stroke
+			(width 0)
+			(type default)
+		)
+	)
+	(wire
+		(pts
 			(xy 33.02 358.14) (xy 43.18 358.14)
 		)
@@
 	(wire
 		(pts
+			(xy 41.91 215.9) (xy 43.18 215.9)
+		)
+		(stroke
+			(width 0)
+			(type default)
+		)
+	)
+	(wire
+		(pts
 			(xy 297.18 341.63) (xy 308.61 341.63)
 		)
@@
 	(wire
 		(pts
+			(xy 58.42 215.9) (xy 55.88 215.9)
+		)
+		(stroke
+			(width 0)
+			(type default)
+		)
+	)
+	(wire
+		(pts
 			(xy 190.5 119.38) (xy 246.38 119.38)
 		)
@@
 	(wire
 		(pts
+			(xy 41.91 215.9) (xy 41.91 223.52)
+		)
+		(stroke
+			(width 0)
+			(type default)
+		)
+	)
+	(wire
+		(pts
 			(xy 43.18 99.06) (xy 33.02 99.06)
 		)
@@
 	(wire
 		(pts
+			(xy 40.64 226.06) (xy 40.64 213.36)
+		)
+		(stroke
+			(width 0)
+			(type default)
+		)
+	)
+	(wire
+		(pts
 			(xy 374.65 267.97) (xy 374.65 256.54)
 		)
@@
 	(wire
 		(pts
+			(xy 40.64 213.36) (xy 43.18 213.36)
+		)
+		(stroke
+			(width 0)
+			(type default)
+		)
+	)
+	(wire
+		(pts
 			(xy 106.68 109.22) (xy 106.68 111.76)
 		)
@@
 	(wire
 		(pts
+			(xy 59.69 213.36) (xy 59.69 226.06)
+		)
+		(stroke
+			(width 0)
+			(type default)
+		)
+	)
+	(wire
+		(pts
 			(xy 287.02 223.52) (xy 266.7 223.52)
 		)
@@
 		)
 	)
+	(label "dchp"
+		(at 59.69 213.36 0)
+		(effects
+			(font
+				(size 1.27 1.27)
+			)
+			(justify left bottom)
+		)
+	)
 	(label "SX5"
 		(at 96.52 147.32 0)
@@
 		)
 	)
+	(label "intp"
+		(at 58.42 215.9 0)
+		(effects
+			(font
+				(size 1.27 1.27)
+			)
+			(justify left bottom)
+		)
+	)

Commit message: fix ram card B key + specific parts
Parts:
- removed U18, U19: 74LS241, Package_DIP:DIP-20_W7.62mm, symbol 74xx:74LS241
- added U18, U19: 74LS244, Package_DIP:DIP-20_W7.62mm, symbol 74xx:74LS244
- J2: footprint _library:portB_NovaMod -> _local:portB_NovaMod
- U17: value 74ALS00 -> 74ALS38
Connections:
- net GND: now also U18.10 (GND), U19.10 (GND)
- net IO00: now also U18.18 (O0a)
- net IO01: now also U18.16 (O1a)
- net IO02: now also U18.14 (O2a)
- net IO03: now also U18.12 (O3a)
- net IO04: now also U18.9 (O0b)
- net IO05: now also U18.7 (O1b)
- net IO06: now also U18.5 (O2b)
- net IO07: now also U18.3 (O3b)
- net IO08: now also U19.18 (O0a)
- net IO09: now also U19.16 (O1a)
- net IO10: now also U19.14 (O2a)
- net IO11: now also U19.12 (O3a)
- net IO12: now also U19.9 (O0b)
- net IO13: now also U19.7 (O1b)
- net IO14: now also U19.5 (O2b)
- net IO15: now also U19.3 (O3b)
- net VCC: now also U18.20 (VCC), U19.20 (VCC)
- net WD00: now also U18.2 (I0a)
- net WD01: now also U18.4 (I1a)
- net WD02: now also U18.6 (I2a)
- net WD03: now also U18.8 (I3a)
- net WD04: now also U18.11 (I0b)
- net WD05: now also U18.13 (I1b)
- net WD06: now also U18.15 (I2b)
- net WD07: now also U18.17 (I3b)
- net WD08: now also U19.2 (I0a)
- net WD09: now also U19.4 (I1a)
- net WD10: now also U19.6 (I2a)
- net WD11: now also U19.8 (I3a)
- net WD12: now also U19.11 (I0b)
- net WD13: now also U19.13 (I1b)
- net WD14: now also U19.15 (I2b)
- net WD15: now also U19.17 (I3b)
- net at U5.12 (6Y): now also U18.1 (OEa), U18.19 (OEb), U19.1 (OEa), U19.19 (OEb)
